Commit message: Use the calibrated frame in air hockey

File: air_hockey_description/urdf/air_hockey.urdf.xacro (robot description, xacro)
@@ -1,13 +1,7 @@
 <?xml version="1.0"?>
 <robot name="iiwas" xmlns:xacro="http://www.ros.org/wiki/xacro">
-    <xacro:include filename="$(find iiwas_description)/urdf/materials.xacro" />
-    <xacro:include filename="$(find iiwas_description)/urdf/iiwas_frame.urdf.xacro"/>
-    <xacro:include filename="$(find iiwas_description)/urdf/iiwa14.xacro"/>
-    <xacro:include filename="$(find iiwas_description)/urdf/util_defs.xml"/>
+    <xacro:include filename="$(find iiwas_description)/robots/iiwas_new_frame.urdf.xacro" />
     <xacro:include filename="$(find air_hockey_description)/urdf/iiwa_striker.urdf.xacro"/>
     <!-- the mass values and inertia may not be completly correct as the moment so this model should just be used as a kinematic one now-->
-    <xacro:property name="M_PI" value="3.1415926535897931"/>
-    <!-- offset values from world to robot base frame.  0.165+0.015 m is the height of the frame + half height of the plate -->
-    <xacro:property name="base_height" default="0.03"/>
     <xacro:arg name="front_base_to_back_base_x" default="3.02"/>
     <xacro:arg name="world_to_iiwas_f_x" default="0.0"/>
@@ -18,35 +12,13 @@
     <xacro:arg name="world_to_iiwas_f_yaw" default="0.0"/>
     <xacro:arg name="hardware_interface" default="PositionJointInterface"/>
-    <!-- construct the iiwas frame, all link is based on the front_base -->
-    <xacro:iiwas_frame name="iiwas_frame">
-        <front>
-            <origin xyz="$(arg world_to_iiwas_f_x) $(arg world_to_iiwas_f_y) ${$(arg world_to_iiwas_f_z) - base_height/2}"
-                    rpy="$(arg world_to_iiwas_f_roll) $(arg world_to_iiwas_f_pitch) $(arg world_to_iiwas_f_yaw)" />
-        </front>
-        <back>
-            <origin xyz="$(arg front_base_to_back_base_x) 0.0 0.0"
-                    rpy="0.0 0.0 0.0" />
-        </back>
-    </xacro:iiwas_frame>
-    <!-- spawn the robot on each of the base-->
-    <!-- iiwas front arm -->
-    <xacro:iiwa14 parent="front_base" hardware_interface="hardware_interface/$(arg hardware_interface)" robot_name="F">
-        <origin xyz="0.0 0.0 ${base_height/2}"
-                rpy="0.0 0.0 0.0"/>
-    </xacro:iiwa14>
     <xacro:striker robot_name="F" parent="F_link_ee" hardware_interface="hardware_interface/$(arg hardware_interface)">
     </xacro:striker>
-    <!-- iiwas back arm -->
-    <xacro:iiwa14 parent="back_base" hardware_interface="hardware_interface/$(arg hardware_interface)" robot_name="B">
-        <origin xyz="0.0 0.0 ${base_height/2}"
-                rpy="0.0 0.0 ${M_PI}"/>
-    </xacro:iiwa14>
     <xacro:striker robot_name="B" parent="B_link_ee" hardware_interface="hardware_interface/$(arg hardware_interface)">
     </xacro:striker>
     <!-- Load Gazebo lib and set the robot namespace -->
-    <gazebo>_
+<!--     <gazebo>_
       <plugin name="gazebo_ros_control" filename="libgazebo_ros_control.so">
-        <!--<robotNamespace>/${robot_name}</robotNamespace>-->
       </plugin>
     </gazebo>
+ -->
 </robot>
