Commit message: add iiwa striker joint

File: air_hockey_description/urdf/air_hockey.urdf (robot description, URDF)
Before this commit: robot iiwas, 33 links, 32 joints
Links:
- link B_hand_link: mass None -> 1
- link B_striker: mass None -> 1
- link F_hand_link: mass None -> 1
- link F_striker: mass None -> 1
Joints:
- joint B_striker_joint: limit effort=1000.0 velocity=1000.0 -> lower=-2.96705972839 upper=2.96705972839 effort=300 velocity=10; origin xyz=0.0 0.0 0.16 rpy=0.785398163397 0.0 -1.57079632679 -> xyz=0.0 0.0 0.16 rpy=0 -1.57079632679 -1.57079632679; type fixed -> revolute
- joint F_striker_joint: limit effort=1000.0 velocity=1000.0 -> lower=-2.96705972839 upper=2.96705972839 effort=300 velocity=10; origin xyz=0.0 0.0 0.16 rpy=0.785398163397 0.0 -1.57079632679 -> xyz=0.0 0.0 0.16 rpy=0 -1.57079632679 -1.57079632679; type fixed -> revolute

File: air_hockey_description/urdf/iiwa_striker.urdf.xacro (robot description, xacro)
@@ -13,4 +13,12 @@
     </joint>
     <link name="${robot_name}_hand_link">
+      <inertial>
+        <origin xyz="0 0 0" rpy="0 0 0" />
+        <mass value="1" />
+        <inertia
+          ixx="1.0" ixy="0.0" ixz="0.0"
+          iyy="1.0" iyz="0.0"
+          izz="1.0" />
+      </inertial>
       <visual>
         <origin xyz="0 0 0" rpy="0 0.0 ${PI/2}"/>
@@ -38,39 +46,46 @@
     </joint>
   <!--  The striker frame is here defined -->
-  <link name="${robot_name}_striker">
-    <visual>
-      <origin xyz="0 0 0" rpy="0.0 0.0 0.0"/>
-      <geometry>
-        <mesh filename="package://air_hockey_description/meshes/striker/visual/only_striker.stl"/>
-      </geometry>
-      <material name="Grey"/>
-    </visual>
-    <collision>
-      <origin xyz="0 0 0" rpy="0.0 0.0 0.0"/>
-      <geometry>
-        <mesh filename="package://air_hockey_description/meshes/striker/collision/only_striker.stl"/>
-      </geometry>
-      <material name="Grey"/>
-      <surface>
-          <bounce>
-              <restitution_coefficient>1</restitution_coefficient>
-          </bounce>
-          <contact>
-              <ode>
-                  <soft_cfm>0.1</soft_cfm>
-                  <soft_erp>0.1</soft_erp>
-                  <max_vel>1</max_vel>
-              </ode>
-          </contact>
-      </surface>
-    </collision>
-  </link>
-  <joint name="${robot_name}_ee_joint" type="fixed">
-    <parent link="${robot_name}_striker" />
-    <child link = "${robot_name}_striker_tip" />
-    <origin xyz="0.0 0.051 0.0" rpy="${PI/2} 0 ${PI}" />
-    <axis xyz="0 0 1"/>
-    <limit effort="1000.0" velocity="1000.0" />
-  </joint>
+    <link name="${robot_name}_striker">
+      <inertial>
+        <origin xyz="0 0 0" rpy="0 0 0" />
+        <mass value="1" />
+        <inertia
+                ixx="1.0" ixy="0.0" ixz="0.0"
+                iyy="1.0" iyz="0.0" izz="1.0" />
+      </inertial>
+      <visual>
+        <origin xyz="0 0 0" rpy="0.0 0.0 0.0"/>
+        <geometry>
+          <mesh filename="package://air_hockey_description/meshes/striker/visual/only_striker.stl"/>
+        </geometry>
+        <material name="Grey"/>
+      </visual>
+      <collision>
+        <origin xyz="0 0 0" rpy="0.0 0.0 0.0"/>
+        <geometry>
+          <mesh filename="package://air_hockey_description/meshes/striker/collision/only_striker.stl"/>
+        </geometry>
+        <material name="Grey"/>
+        <surface>
+            <bounce>
+                <restitution_coefficient>1</restitution_coefficient>
+            </bounce>
+            <contact>
+                <ode>
+                    <soft_cfm>0.1</soft_cfm>
+                    <soft_erp>0.1</soft_erp>
+                    <max_vel>1</max_vel>
+                </ode>
+            </contact>
+        </surface>
+      </collision>
+    </link>
+    <joint name="${robot_name}_ee_joint" type="fixed">
+      <parent link="${robot_name}_striker" />
+      <child link = "${robot_name}_striker_tip" />
+      <origin xyz="0.0 0.051 0.0" rpy="${PI/2} 0 ${PI}" />
+      <axis xyz="0 0 1"/>
+      <limit effort="1000.0" velocity="1000.0" />
+    </joint>
     <gazebo reference="${robot_name}_hand_link">
       <material>Gazebo/Grey</material>

Commit message: Add Dynamics property

File: air_hockey_description/urdf/air_hockey.urdf (robot description, URDF)
Before this commit: robot iiwas, 33 links, 32 joints
Links:
- link B_hand_link: mass 1 -> 0.1
- link B_striker: mass 1 -> 0.1
- link F_hand_link: mass 1 -> 0.1
- link F_striker: mass 1 -> 0.1
Joints:
- joint B_ee_joint: origin xyz=0.0 0.051 0.0 rpy=1.57079632679 0 3.14159265359 -> xyz=0.0 0.051 0.0 rpy=-1.57079632679 0 0
- joint B_striker_joint: origin xyz=0.0 0.0 0.16 rpy=0 -1.57079632679 -1.57079632679 -> xyz=0.0 0.0 0.16 rpy=1.57079632679 0 0
- joint F_ee_joint: origin xyz=0.0 0.051 0.0 rpy=1.57079632679 0 3.14159265359 -> xyz=0.0 0.051 0.0 rpy=-1.57079632679 0 0
- joint F_striker_joint: origin xyz=0.0 0.0 0.16 rpy=0 -1.57079632679 -1.57079632679 -> xyz=0.0 0.0 0.16 rpy=1.57079632679 0 0

File: air_hockey_description/urdf/iiwa_striker.urdf.xacro (robot description, xacro)
@@ -15,5 +15,5 @@
       <inertial>
         <origin xyz="0 0 0" rpy="0 0 0" />
-        <mass value="1" />
+        <mass value="0.1" />
         <inertia
           ixx="1.0" ixy="0.0" ixz="0.0"
@@ -39,18 +39,18 @@
       <parent link="${robot_name}_hand_link" />
       <child link = "${robot_name}_striker" />
-      <origin xyz="0.0 0.0 0.16" rpy="0 -${PI/2} -${PI/2}" />
+      <origin xyz="0.0 0.0 0.16" rpy="${PI/2} 0 0" />
       <axis xyz="0 0 1"/>
       <limit effort="300" lower="-2.96705972839" upper="2.96705972839" velocity="10"/>
       <safety_controller k_position="100" k_velocity="2" soft_lower_limit="-2.93215314335" soft_upper_limit="2.93215314335"/>
-      <dynamics damping="0.5"/>
+      <dynamics damping="0.01" friction="1"/>
     </joint>
   <!--  The striker frame is here defined -->
     <link name="${robot_name}_striker">
       <inertial>
-        <origin xyz="0 0 0" rpy="0 0 0" />
-        <mass value="1" />
+        <origin xyz="0 0.051 0" rpy="0 0 0" />
+        <mass value="0.1" />
         <inertia
-                ixx="1.0" ixy="0.0" ixz="0.0"
-                iyy="1.0" iyz="0.0" izz="1.0" />
+                ixx="0.00012" ixy="0.0" ixz="0.0"
+                iyy="0.00002" iyz="0.0" izz="0.00002" />
       </inertial>
       <visual>
@@ -69,5 +69,5 @@
         <surface>
             <bounce>
-                <restitution_coefficient>1</restitution_coefficient>
+                <restitution_coefficient>0.8</restitution_coefficient>
             </bounce>
             <contact>
@@ -84,5 +84,5 @@
       <parent link="${robot_name}_striker" />
       <child link = "${robot_name}_striker_tip" />
-      <origin xyz="0.0 0.051 0.0" rpy="${PI/2} 0 ${PI}" />
+      <origin xyz="0.0 0.051 0.0" rpy="-${PI/2} 0 0" />
       <axis xyz="0 0 1"/>
       <limit effort="1000.0" velocity="1000.0" />

Commit message: change the friction of the striker joint

File: air_hockey_description/urdf/air_hockey.urdf (robot description, URDF)
Before this commit: robot iiwas, 33 links, 32 joints
Links:
- link B_striker: mass 0.1 -> 0.0
- link B_striker_tip: mass None -> 0.1
- link F_striker: mass 0.1 -> 0.0
- link F_striker_tip: mass None -> 0.1

File: air_hockey_description/urdf/iiwa_striker.urdf.xacro (robot description, xacro)
@@ -43,14 +43,14 @@
       <limit effort="300" lower="-2.96705972839" upper="2.96705972839" velocity="10"/>
       <safety_controller k_position="100" k_velocity="2" soft_lower_limit="-2.93215314335" soft_upper_limit="2.93215314335"/>
-      <dynamics damping="0.01" friction="1"/>
+      <dynamics damping="0.01" friction="0.01"/>
     </joint>
   <!--  The striker frame is here defined -->
     <link name="${robot_name}_striker">
       <inertial>
-        <origin xyz="0 0.051 0" rpy="0 0 0" />
-        <mass value="0.1" />
+        <origin xyz="0 0.0 0" rpy="0 0 0" />
+        <mass value="0.0" />
         <inertia
-                ixx="0.00012" ixy="0.0" ixz="0.0"
-                iyy="0.00002" iyz="0.0" izz="0.00002" />
+                ixx="0.0" ixy="0.0" ixz="0.0"
+                iyy="0.0" iyz="0.0" izz="0.0" />
       </inertial>
       <visual>
@@ -88,4 +88,13 @@
       <limit effort="1000.0" velocity="1000.0" />
     </joint>
+    <link name="${robot_name}_striker_tip">
+      <inertial>
+        <origin xyz="0 0 0" rpy="0 0 0" />
+        <mass value="0.1" />
+        <inertia
+                ixx="0.00012" ixy="0.0" ixz="0.0"
+                iyy="0.00002" iyz="0.0" izz="0.00002" />
+      </inertial>
+    </link>
     <gazebo reference="${robot_name}_hand_link">
       <material>Gazebo/Grey</material>
@@ -100,5 +109,5 @@
       <selfCollide>0</selfCollide>
     </gazebo>
-    <transmission name="${robot_name}_ee_tran_1">
+    <transmission name="${robot_name}_striker_tran">
       <robotNamespace>/${robot_name}</robotNamespace>
       <type>transmission_interface/SimpleTransmission</type>
@@ -106,10 +115,9 @@
 	    <hardwareInterface>${hardware_interface}</hardwareInterface>
       </joint>
-      <actuator name="${robot_name}_ee_motor_1">
+      <actuator name="${robot_name}_striker_motor">
 	    <hardwareInterface>${hardware_interface}</hardwareInterface>
 	    <mechanicalReduction>1</mechanicalReduction>
       </actuator>
     </transmission>
-    <link name="${robot_name}_striker_tip"/>
   </xacro:macro>
 </robot>

Commit message: change the inertia of striker

File: air_hockey_description/urdf/air_hockey.urdf (robot description, URDF)
Before this commit: robot iiwas, 33 links, 32 joints
Links:
- link back_base: mass None -> 3
- link front_base: mass None -> 3
- link h_bar_back_in: mass None -> 5
- link h_bar_back_out: mass None -> 5
- link h_bar_front_in: mass None -> 5
- link h_bar_front_out: mass None -> 5
- link v_bar_left: mass None -> 8
- link v_bar_right: mass None -> 8
Joints:
- joint B_striker_joint: limit lower=-2.96705972839 upper=2.96705972839 effort=300 velocity=10 -> lower=-2.094395102 upper=2.094395102 effort=300 velocity=10
- joint F_striker_joint: limit lower=-2.96705972839 upper=2.96705972839 effort=300 velocity=10 -> lower=-2.094395102 upper=2.094395102 effort=300 velocity=10

File: air_hockey_description/urdf/iiwa_striker.urdf.xacro (robot description, xacro)
@@ -14,10 +14,10 @@
     <link name="${robot_name}_hand_link">
       <inertial>
-        <origin xyz="0 0 0" rpy="0 0 0" />
+        <origin xyz="0 0 0.0417" rpy="0 0 0" />
         <mass value="0.1" />
         <inertia
-          ixx="1.0" ixy="0.0" ixz="0.0"
-          iyy="1.0" iyz="0.0"
-          izz="1.0" />
+          ixx="0.000297" ixy="0.0" ixz="0.0"
+          iyy="0.000271" iyz="0.0000001"
+          izz="0.0000653" />
       </inertial>
       <visual>
@@ -41,6 +41,6 @@
       <origin xyz="0.0 0.0 0.16" rpy="${PI/2} 0 0" />
       <axis xyz="0 0 1"/>
-      <limit effort="300" lower="-2.96705972839" upper="2.96705972839" velocity="10"/>
-      <safety_controller k_position="100" k_velocity="2" soft_lower_limit="-2.93215314335" soft_upper_limit="2.93215314335"/>
+      <limit effort="300" lower="-2.094395102" upper="2.094395102" velocity="10"/>
+      <safety_controller k_position="100" k_velocity="2" soft_lower_limit="-2.094395102" soft_upper_limit="2.094395102"/>
       <dynamics damping="0.01" friction="0.01"/>
     </joint>
@@ -93,6 +93,6 @@
         <mass value="0.1" />
         <inertia
-                ixx="0.00012" ixy="0.0" ixz="0.0"
-                iyy="0.00002" iyz="0.0" izz="0.00002" />
+                ixx="0.0000658" ixy="0.0" ixz="0.0"
+                iyy="0.0000658" iyz="0.0" izz="0.000125" />
       </inertial>
     </link>

Commit message: tune the urdf parameter, add joint velocity limit

File: air_hockey_description/urdf/air_hockey.urdf (robot description, URDF)
Before this commit: robot iiwas, 33 links, 32 joints
Links:
- link B_link_ee: mass None -> 0.0
- link F_link_ee: mass None -> 0.0
Joints:
- joint B_EB: limit lower=-2.09439510239 upper=2.09439510239 effort=176 velocity=1.309 -> lower=-2.09439510239 upper=2.09439510239 effort=176 velocity=1.308996939
- joint B_HR: limit lower=-2.96705972839 upper=2.96705972839 effort=176 velocity=1.309 -> lower=-2.96705972839 upper=2.96705972839 effort=176 velocity=1.74532925199
- joint B_SAA: limit lower=-2.09439510239 upper=2.09439510239 effort=320 velocity=1.309 -> lower=-2.09439510239 upper=2.09439510239 effort=320 velocity=1.4835298642
- joint B_SFE: limit lower=-2.96705972839 upper=2.96705972839 effort=320 velocity=1.309 -> lower=-2.96705972839 upper=2.96705972839 effort=320 velocity=1.4835298642
- joint B_WAA: limit lower=-3.05432619099 upper=3.05432619099 effort=40 velocity=1.309 -> lower=-3.05432619099 upper=3.05432619099 effort=40 velocity=2.35619449019
- joint B_WFE: limit lower=-2.09439510239 upper=2.09439510239 effort=40 velocity=1.309 -> lower=-2.09439510239 upper=2.09439510239 effort=40 velocity=2.35619449019
- joint B_WR: limit lower=-2.96705972839 upper=2.96705972839 effort=110 velocity=1.309 -> lower=-2.96705972839 upper=2.96705972839 effort=110 velocity=2.26892802759
- joint B_striker_joint: limit lower=-2.094395102 upper=2.094395102 effort=300 velocity=10 -> lower=-2.094395102 upper=2.094395102 effort=10 velocity=10
- joint F_EB: limit lower=-2.09439510239 upper=2.09439510239 effort=176 velocity=1.309 -> lower=-2.09439510239 upper=2.09439510239 effort=176 velocity=1.308996939
- joint F_HR: limit lower=-2.96705972839 upper=2.96705972839 effort=176 velocity=1.309 -> lower=-2.96705972839 upper=2.96705972839 effort=176 velocity=1.74532925199
- joint F_SAA: limit lower=-2.09439510239 upper=2.09439510239 effort=320 velocity=1.309 -> lower=-2.09439510239 upper=2.09439510239 effort=320 velocity=1.4835298642
- joint F_SFE: limit lower=-2.96705972839 upper=2.96705972839 effort=320 velocity=1.309 -> lower=-2.96705972839 upper=2.96705972839 effort=320 velocity=1.4835298642
- joint F_WAA: limit lower=-3.05432619099 upper=3.05432619099 effort=40 velocity=1.309 -> lower=-3.05432619099 upper=3.05432619099 effort=40 velocity=2.35619449019
- joint F_WFE: limit lower=-2.09439510239 upper=2.09439510239 effort=40 velocity=1.309 -> lower=-2.09439510239 upper=2.09439510239 effort=40 velocity=2.35619449019
- joint F_WR: limit lower=-2.96705972839 upper=2.96705972839 effort=110 velocity=1.309 -> lower=-2.96705972839 upper=2.96705972839 effort=110 velocity=2.26892802759
- joint F_striker_joint: limit lower=-2.094395102 upper=2.094395102 effort=300 velocity=10 -> lower=-2.094395102 upper=2.094395102 effort=10 velocity=10

File: air_hockey_description/urdf/iiwa_striker.urdf.xacro (robot description, xacro)
@@ -41,7 +41,7 @@
       <origin xyz="0.0 0.0 0.16" rpy="${PI/2} 0 0" />
       <axis xyz="0 0 1"/>
-      <limit effort="300" lower="-2.094395102" upper="2.094395102" velocity="10"/>
+      <limit effort="10" lower="-2.094395102" upper="2.094395102" velocity="10"/>
       <safety_controller k_position="100" k_velocity="2" soft_lower_limit="-2.094395102" soft_upper_limit="2.094395102"/>
-      <dynamics damping="0.01" friction="0.01"/>
+      <dynamics damping="0.5" friction="0.5"/>
     </joint>
   <!--  The striker frame is here defined -->

Commit message: draw new end effector

File: air_hockey_description/urdf/air_hockey.urdf (robot description, URDF)
Before this commit: robot iiwas, 33 links, 32 joints
Links:
- link B_striker: geometry collision cylinder length=0.051 radius=0.048; visual mesh filename=package://air_hockey_description/meshes/striker/visual/only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
- link F_striker: geometry collision cylinder length=0.051 radius=0.048; visual mesh filename=package://air_hockey_description/meshes/striker/visual/only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

File: air_hockey_description/urdf/iiwa_striker.urdf.xacro (robot description, xacro)
@@ -55,14 +55,15 @@
       </inertial>
       <visual>
-        <origin xyz="0 0 0" rpy="0.0 0.0 0.0"/>
+        <origin xyz="0 0.0 0.0" rpy="0.0 0.0 0.0"/>
         <geometry>
-          <mesh filename="package://air_hockey_description/meshes/striker/visual/only_striker.stl"/>
+        	<mesh filename="package://air_hockey_description/meshes/striker/visual/only_striker.stl"/>
         </geometry>
         <material name="Grey"/>
       </visual>
       <collision>
-        <origin xyz="0 0 0" rpy="0.0 0.0 0.0"/>
+        <origin xyz="0 0.0255 0.0" rpy="${PI / 2} 0.0 0.0"/>
         <geometry>
-          <mesh filename="package://air_hockey_description/meshes/striker/collision/only_striker.stl"/>
+					<cylinder radius="0.048" length="0.051"/>
+          <!--<mesh filename="package://air_hockey_description/meshes/striker/collision/only_striker.stl"/>-->
         </geometry>
         <material name="Grey"/>

Commit message: change the joint name of urdf fil

File: air_hockey_description/urdf/air_hockey.urdf (robot description, URDF)
Before this commit: robot iiwas, 33 links, 32 joints
Joints:
- removed joint B_EB
- removed joint B_HR
- removed joint B_SAA
- removed joint B_SFE
- removed joint B_WAA
- removed joint B_WFE
- removed joint B_WR
- removed joint F_EB
- removed joint F_HR
- removed joint F_SAA
- removed joint F_SFE
- removed joint F_WAA
- removed joint F_WFE
- removed joint F_WR
- added joint B_joint_1: type revolute, parent B_link_0, child B_link_1, origin xyz=0 0 0.1575 rpy=0 0 0, axis 0 0 1, limit lower=-2.9670597283903604 upper=2.9670597283903604 effort=320 velocity=1.4835298641951802
- added joint B_joint_2: type revolute, parent B_link_1, child B_link_2, origin xyz=0 0 0.2025 rpy=1.5707963267948966   0 3.141592653589793, axis 0 0 1, limit lower=-2.0943951023931953 upper=2.0943951023931953 effort=320 velocity=1.4835298641951802
- added joint B_joint_3: type revolute, parent B_link_2, child B_link_3, origin xyz=0 0.2045 0 rpy=1.5707963267948966 0 3.141592653589793, axis 0 0 1, limit lower=-2.9670597283903604 upper=2.9670597283903604 effort=176 velocity=1.7453292519943295
- added joint B_joint_4: type revolute, parent B_link_3, child B_link_4, origin xyz=0 0 0.2155 rpy=1.5707963267948966 0 0, axis 0 0 1, limit lower=-2.0943951023931953 upper=2.0943951023931953 effort=176 velocity=1.3089969389957472
- added joint B_joint_5: type revolute, parent B_link_4, child B_link_5, origin xyz=0 0.1845 0 rpy=-1.5707963267948966 3.141592653589793 0, axis 0 0 1, limit lower=-2.9670597283903604 upper=2.9670597283903604 effort=110 velocity=2.2689280275926285
- added joint B_joint_6: type revolute, parent B_link_5, child B_link_6, origin xyz=0 0 0.2155 rpy=1.5707963267948966 0 0, axis 0 0 1, limit lower=-2.0943951023931953 upper=2.0943951023931953 effort=40 velocity=2.356194490192345
- added joint B_joint_7: type revolute, parent B_link_6, child B_link_7, origin xyz=0 0.081 0 rpy=-1.5707963267948966 3.141592653589793 0, axis 0 0 1, limit lower=-3.0543261909900763 upper=3.0543261909900763 effort=40 velocity=2.356194490192345
- added joint F_joint_1: type revolute, parent F_link_0, child F_link_1, origin xyz=0 0 0.1575 rpy=0 0 0, axis 0 0 1, limit lower=-2.9670597283903604 upper=2.9670597283903604 effort=320 velocity=1.4835298641951802
- added joint F_joint_2: type revolute, parent F_link_1, child F_link_2, origin xyz=0 0 0.2025 rpy=1.5707963267948966   0 3.141592653589793, axis 0 0 1, limit lower=-2.0943951023931953 upper=2.0943951023931953 effort=320 velocity=1.4835298641951802
- added joint F_joint_3: type revolute, parent F_link_2, child F_link_3, origin xyz=0 0.2045 0 rpy=1.5707963267948966 0 3.141592653589793, axis 0 0 1, limit lower=-2.9670597283903604 upper=2.9670597283903604 effort=176 velocity=1.7453292519943295
- added joint F_joint_4: type revolute, parent F_link_3, child F_link_4, origin xyz=0 0 0.2155 rpy=1.5707963267948966 0 0, axis 0 0 1, limit lower=-2.0943951023931953 upper=2.0943951023931953 effort=176 velocity=1.3089969389957472
- added joint F_joint_5: type revolute, parent F_link_4, child F_link_5, origin xyz=0 0.1845 0 rpy=-1.5707963267948966 3.141592653589793 0, axis 0 0 1, limit lower=-2.9670597283903604 upper=2.9670597283903604 effort=110 velocity=2.2689280275926285
- added joint F_joint_6: type revolute, parent F_link_5, child F_link_6, origin xyz=0 0 0.2155 rpy=1.5707963267948966 0 0, axis 0 0 1, limit lower=-2.0943951023931953 upper=2.0943951023931953 effort=40 velocity=2.356194490192345
- added joint F_joint_7: type revolute, parent F_link_6, child F_link_7, origin xyz=0 0.081 0 rpy=-1.5707963267948966 3.141592653589793 0, axis 0 0 1, limit lower=-3.0543261909900763 upper=3.0543261909900763 effort=40 velocity=2.356194490192345
- joint B_ee_joint: origin xyz=0.0 0.051 0.0 rpy=-1.57079632679 0 0 -> xyz=0.0 0.051 0.0 rpy=-1.5707963267948966 0 0
- joint B_striker_joint: origin xyz=0.0 0.0 0.16 rpy=1.57079632679 0 0 -> xyz=0.0 0.0 0.16 rpy=1.5707963267948966 0 0
- joint F_ee_joint: origin xyz=0.0 0.051 0.0 rpy=-1.57079632679 0 0 -> xyz=0.0 0.051 0.0 rpy=-1.5707963267948966 0 0
- joint F_striker_joint: origin xyz=0.0 0.0 0.16 rpy=1.57079632679 0 0 -> xyz=0.0 0.0 0.16 rpy=1.5707963267948966 0 0
- joint back_base_B_base_joint: origin xyz=0.0 0.0 0.015 rpy=0.0 0.0 3.14159265359 -> xyz=0.0 0.0 0.015 rpy=0.0 0.0 3.141592653589793
- joint back_in: origin xyz=0.0 0.0 -0.0975 rpy=0.0 0.0 1.57079632679 -> xyz=0.0 0.0 -0.0975 rpy=0.0 0.0 1.5707963267948966
- joint back_out: origin xyz=3.22 0.0 -0.0975 rpy=0.0 0.0 1.57079632679 -> xyz=3.22 0.0 -0.0975 rpy=0.0 0.0 1.5707963267948966
- joint front_in: origin xyz=0.0 0.0 -0.0975 rpy=0.0 0.0 1.57079632679 -> xyz=0.0 0.0 -0.0975 rpy=0.0 0.0 1.5707963267948966
- joint front_out: origin xyz=-0.20 0.0 -0.0975 rpy=0.0 0.0 1.57079632679 -> xyz=-0.20 0.0 -0.0975 rpy=0.0 0.0 1.5707963267948966

File: air_hockey_description/urdf/iiwa_striker.urdf.xacro (robot description, xacro)
@@ -64,5 +64,5 @@
         <origin xyz="0 0.0255 0.0" rpy="${PI / 2} 0.0 0.0"/>
         <geometry>
-					<cylinder radius="0.048" length="0.051"/>
+				<cylinder radius="0.048" length="0.051"/>
           <!--<mesh filename="package://air_hockey_description/meshes/striker/collision/only_striker.stl"/>-->
         </geometry>
