Commit message: Write New End Effector

File: air_hockey_description/urdf/air_hockey.urdf (robot description, URDF)
Before this commit: robot iiwas, 33 links, 32 joints
Links:
- removed link B_hand_link
- removed link B_striker
- removed link B_striker_tip
- removed link F_hand_link
- removed link F_striker
- removed link F_striker_tip
- added link B_striker_base, mass 0.1; collision mesh filename=package://air_hockey_description/meshes/striker_new/collisi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; visual mesh filename=package://air_hockey_description/meshes/striker_new/visual/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
- added link B_striker_joint_link, mass 0.0
- added link B_striker_mallet, mass 0.0; collision mesh filename=package://air_hockey_description/meshes/striker_new/collisi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; visual mesh filename=package://air_hockey_description/meshes/striker_new/visual/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
- added link B_striker_mallet_tip, mass 0.0
- added link F_striker_base, mass 0.1; collision mesh filename=package://air_hockey_description/meshes/striker_new/collisi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; visual mesh filename=package://air_hockey_description/meshes/striker_new/visual/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
- added link F_striker_joint_link, mass 0.0
- added link F_striker_mallet, mass 0.0; collision mesh filename=package://air_hockey_description/meshes/striker_new/collisi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; visual mesh filename=package://air_hockey_description/meshes/striker_new/visual/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
- added link F_striker_mallet_tip, mass 0.0
- link h_bar_back_in: geometry collision box size=0.12 1.56 0.165; visual box size=0.12 1.56 0.165
- link h_bar_back_out: geometry collision box size=0.08 1.56 0.165; visual box size=0.08 1.56 0.165
- link h_bar_front_in: geometry collision box size=0.12 1.56 0.165; visual box size=0.12 1.56 0.165
- link h_bar_front_out: geometry collision box size=0.08 1.56 0.165; visual box size=0.08 1.56 0.165
Joints:
- removed joint B_ee_joint
- removed joint B_striker_joint
- removed joint F_ee_joint
- removed joint F_striker_joint
- added joint B_striker_joint_1: type revolute, parent B_striker_base, child B_striker_joint_link, origin xyz=0.0 0.0 0.3455 rpy=0 0 0, axis 1 0 0, limit lower=-1.5707963267948966 upper=1.5707963267948966 effort=10 velocity=10
- added joint B_striker_joint_2: type revolute, parent B_striker_joint_link, child B_striker_mallet, origin xyz=0.0 0.0 0.0 rpy=0 0 0, axis 0 1 0, limit lower=-1.5707963267948966 upper=1.5707963267948966 effort=10 velocity=10
- added joint B_striker_mallet_fix: type fixed, parent B_striker_mallet, child B_striker_mallet_tip, origin xyz=0.0 0.0 0.0805 rpy=0 0 0, axis 1 0 0
- added joint F_striker_joint_1: type revolute, parent F_striker_base, child F_striker_joint_link, origin xyz=0.0 0.0 0.3455 rpy=0 0 0, axis 1 0 0, limit lower=-1.5707963267948966 upper=1.5707963267948966 effort=10 velocity=10
- added joint F_striker_joint_2: type revolute, parent F_striker_joint_link, child F_striker_mallet, origin xyz=0.0 0.0 0.0 rpy=0 0 0, axis 0 1 0, limit lower=-1.5707963267948966 upper=1.5707963267948966 effort=10 velocity=10
- added joint F_striker_mallet_fix: type fixed, parent F_striker_mallet, child F_striker_mallet_tip, origin xyz=0.0 0.0 0.0805 rpy=0 0 0, axis 1 0 0
- joint B_striker: child B_hand_link -> B_striker_base
- joint F_striker: child F_hand_link -> F_striker_base
- joint back_base_joint: origin xyz=3.02 0.0 0.0 rpy=0.0 0.0 0.0 -> xyz=3.22 0.61 -0.015 rpy=0.0 0.0 0.0; parent front_base -> world
- joint back_in: origin xyz=0.0 0.0 -0.0975 rpy=0.0 0.0 1.5707963267948966 -> xyz=0.0 -0.61 -0.0975 rpy=0.0 0.0 0.0
- joint back_out: origin xyz=3.22 0.0 -0.0975 rpy=0.0 0.0 1.5707963267948966 -> xyz=1.71 0.8400000000000001 0.0 rpy=0.0 0.0 0.0; parent front_base -> v_bar_right
- joint frame_right: origin xyz=1.51 -0.84 -0.0975 rpy=0.0 0.0 0.0 -> xyz=1.71 -0.8400000000000001 0.0 rpy=0.0 0.0 0.0; parent front_base -> h_bar_front_out
- joint front_base_joint: origin xyz=0.0 0.0 -0.015 rpy=0.0 0.0 0.0 -> xyz=0.2 -0.61 -0.015 rpy=0.0 0.0 0.0
- joint front_in: origin xyz=0.0 0.0 -0.0975 rpy=0.0 0.0 1.5707963267948966 -> xyz=0.0 0.61 -0.0975 rpy=0.0 0.0 0.0
- joint front_out: origin xyz=-0.20 0.0 -0.0975 rpy=0.0 0.0 1.5707963267948966 -> xyz=0.0 0.0 -0.1125 rpy=0.0 0.0 0; parent front_base -> world
- joint left: origin xyz=1.51 0.84 -0.0975 rpy=0.0 0.0 0.0 -> xyz=1.71 0.8400000000000001 0.0 rpy=0.0 0.0 3.141592653589793; parent front_base -> h_bar_front_out

File: air_hockey_description/urdf/iiwa_striker.urdf.xacro (robot description, xacro)
@@ -8,45 +8,62 @@
   <xacro:macro name="striker" params="robot_name parent hardware_interface">
     <joint name="${robot_name}_striker" type="fixed">
-      <parent link="${parent}" />
-      <child link = "${robot_name}_hand_link" />
-      <origin xyz="0.0 0.0 0.0" rpy="0 0 0" />
+		<parent link="${parent}" />
+		<child link = "${robot_name}_striker_base" />
+		<origin xyz="0.0 0.0 0.0" rpy="0 0 0" />
     </joint>
-    <link name="${robot_name}_hand_link">
-      <inertial>
-        <origin xyz="0 0 0.0417" rpy="0 0 0" />
-        <mass value="0.1" />
-        <inertia
-          ixx="0.000297" ixy="0.0" ixz="0.0"
-          iyy="0.000271" iyz="0.0000001"
-          izz="0.0000653" />
-      </inertial>
-      <visual>
-        <origin xyz="0 0 0" rpy="0 0.0 ${PI/2}"/>
-        <geometry>
-          <mesh filename="package://air_hockey_description/meshes/striker/visual/hand.stl"/>
-        </geometry>
-        <material name="Grey"/>
-      </visual>
-      <collision>
-        <origin xyz="0 0 0" rpy="0 0 ${PI/2}"/>
-        <geometry>
-          <mesh filename="package://air_hockey_description/meshes/striker/collision/hand.stl"/>
-        </geometry>
-        <material name="Grey"/>
-      </collision>
+    <link name="${robot_name}_striker_base">
+		<inertial>
+		<origin xyz="0 0 0.0417" rpy="0 0 0" />
+		<mass value="0.1" />
+		<inertia
+			ixx="0.000297" ixy="0.0" ixz="0.0"
+			iyy="0.000271" iyz="0.0000001" izz="0.0000653" />
+		</inertial>
+		<visual>
+		<origin xyz="0 0 0" rpy="0 0.0 0"/>
+		<geometry>
+		  	<mesh filename="package://air_hockey_description/meshes/striker_new/visual/gas_spring.stl"/>
+		</geometry>
+		<material name="Grey"/>
+		</visual>
+		<collision>
+		<origin xyz="0 0 0" rpy="0 0 0"/>
+		<geometry>
+		  	<mesh filename="package://air_hockey_description/meshes/striker_new/collision/gas_spring_collision.stl"/>
+		</geometry>
+		<material name="Grey"/>
+		</collision>
     </link>
-    <joint name="${robot_name}_striker_joint" type="revolute">
-      <parent link="${robot_name}_hand_link" />
-      <child link = "${robot_name}_striker" />
-      <origin xyz="0.0 0.0 0.16" rpy="${PI/2} 0 0" />
-      <axis xyz="0 0 1"/>
-      <limit effort="10" lower="-2.094395102" upper="2.094395102" velocity="10"/>
-      <safety_controller k_position="100" k_velocity="2" soft_lower_limit="-2.094395102" soft_upper_limit="2.094395102"/>
-      <dynamics damping="0.5" friction="0.5"/>
+    <joint name="${robot_name}_striker_joint_1" type="revolute">
+		<parent link="${robot_name}_striker_base" />
+		<child link = "${robot_name}_striker_joint_link" />
+		<origin xyz="0.0 0.0 0.3455" rpy="0 0 0" />
+		<axis xyz="1 0 0"/>
+		<limit effort="10" lower="-${PI/2}" upper="${PI/2}" velocity="10"/>
+		<safety_controller k_position="100" k_velocity="2" soft_lower_limit="-2.094395102" soft_upper_limit="2.094395102"/>
+		<dynamics damping="0.5" friction="0.5"/>
+    </joint>
+    <link name="${robot_name}_striker_joint_link">
+    	<inertial>
+	        <origin xyz="0 0.0 0" rpy="0 0 0" />
+	        <mass value="0.0" />
+	        <inertia
+                ixx="0.0" ixy="0.0" ixz="0.0"
+                iyy="0.0" iyz="0.0" izz="0.0" />
+      	</inertial>
+    </link>
+    <joint name="${robot_name}_striker_joint_2" type="revolute">
+		<parent link="${robot_name}_striker_joint_link" />
+		<child link = "${robot_name}_striker_mallet" />
+		<origin xyz="0.0 0.0 0.0" rpy="0 0 0" />
+		<axis xyz="0 1 0"/>
+		<limit effort="10" lower="-${PI/2}" upper="${PI/2}" velocity="10"/>
+		<safety_controller k_position="100" k_velocity="2" soft_lower_limit="-2.094395102" soft_upper_limit="2.094395102"/>
+		<dynamics damping="0.5" friction="0.5"/>
     </joint>
   <!--  The striker frame is here defined -->
-    <link name="${robot_name}_striker">
+    <link name="${robot_name}_striker_mallet">
       <inertial>
-        <origin xyz="0 0.0 0" rpy="0 0 0" />
+        <origin xyz="0 0.0 0.0805" rpy="0 0 0" />
         <mass value="0.0" />
         <inertia
@@ -55,15 +72,14 @@
       </inertial>
       <visual>
-        <origin xyz="0 0.0 0.0" rpy="0.0 0.0 0.0"/>
+        <origin xyz="0 0.0 0.0" rpy="0.0 0.0 0"/>
         <geometry>
-        	<mesh filename="package://air_hockey_description/meshes/striker/visual/only_striker.stl"/>
+        	<mesh filename="package://air_hockey_description/meshes/striker_new/visual/joint_mallet.stl"/>
         </geometry>
         <material name="Grey"/>
       </visual>
       <collision>
-        <origin xyz="0 0.0255 0.0" rpy="${PI / 2} 0.0 0.0"/>
+        <origin xyz="0 0.0 0.0" rpy="0.0 0.0 0"/>
         <geometry>
-				<cylinder radius="0.048" length="0.051"/>
-          <!--<mesh filename="package://air_hockey_description/meshes/striker/collision/only_striker.stl"/>-->
+          	<mesh filename="package://air_hockey_description/meshes/striker_new/collision/joint_mallet_collision.stl"/>
         </geometry>
         <material name="Grey"/>
@@ -82,43 +98,65 @@
       </collision>
     </link>
-    <joint name="${robot_name}_ee_joint" type="fixed">
-      <parent link="${robot_name}_striker" />
-      <child link = "${robot_name}_striker_tip" />
-      <origin xyz="0.0 0.051 0.0" rpy="-${PI/2} 0 0" />
-      <axis xyz="0 0 1"/>
-      <limit effort="1000.0" velocity="1000.0" />
+    <joint name="${robot_name}_striker_mallet_fix" type="fixed">
+		<parent link="${robot_name}_striker_mallet" />
+		<child link = "${robot_name}_striker_mallet_tip" />
+		<origin xyz="0.0 0.0 0.0805" rpy="0 0 0" />
+		<axis xyz="1 0 0"/>
     </joint>
-    <link name="${robot_name}_striker_tip">
-      <inertial>
-        <origin xyz="0 0 0" rpy="0 0 0" />
-        <mass value="0.1" />
-        <inertia
-                ixx="0.0000658" ixy="0.0" ixz="0.0"
-                iyy="0.0000658" iyz="0.0" izz="0.000125" />
-      </inertial>
+    <link name="${robot_name}_striker_mallet_tip">
+    	<inertial>
+	        <origin xyz="0 0.0 0" rpy="0 0 0" />
+	        <mass value="0.0" />
+	        <inertia
+                ixx="0.0" ixy="0.0" ixz="0.0"
+                iyy="0.0" iyz="0.0" izz="0.0" />
+      	</inertial>
     </link>
-    <gazebo reference="${robot_name}_hand_link">
-      <material>Gazebo/Grey</material>
-      <mu1>0.2</mu1>
-      <mu2>0.2</mu2>
-      <selfCollide>0</selfCollide>
+    <gazebo reference="${robot_name}_striker_base">
+			<material>Gazebo/Grey</material>
+			<mu1>0.2</mu1>
+			<mu2>0.2</mu2>
+			<selfCollide>0</selfCollide>
     </gazebo>
-    <gazebo reference="${robot_name}_striker">
-      <material>Gazebo/Grey</material>
-      <mu1>0.2</mu1>
-      <mu2>0.2</mu2>
-      <selfCollide>0</selfCollide>
+    <gazebo reference="${robot_name}_striker_joint_link">
+		<material>Gazebo/Grey</material>
+		<mu1>0.2</mu1>
+		<mu2>0.2</mu2>
+		<selfCollide>0</selfCollide>
     </gazebo>
-    <transmission name="${robot_name}_striker_tran">
-      <robotNamespace>/${robot_name}</robotNamespace>
-      <type>transmission_interface/SimpleTransmission</type>
-      <joint name="${robot_name}_striker_joint">
-	    <hardwareInterface>${hardware_interface}</hardwareInterface>
-      </joint>
-      <actuator name="${robot_name}_striker_motor">
-	    <hardwareInterface>${hardware_interface}</hardwareInterface>
-	    <mechanicalReduction>1</mechanicalReduction>
-      </actuator>
-    </transmission>
+    <gazebo reference="${robot_name}_striker_mallet">
+			<material>Gazebo/Grey</material>
+			<mu1>0.2</mu1>
+			<mu2>0.2</mu2>
+			<selfCollide>0</selfCollide>
+    </gazebo>
+    <gazebo reference="${robot_name}_striker_mallet_tip">
+			<material>Gazebo/Grey</material>
+			<mu1>0.2</mu1>
+			<mu2>0.2</mu2>
+			<selfCollide>0</selfCollide>
+    </gazebo>
+    <transmission name="${robot_name}_striker_tran_1">
+		<robotNamespace>/${robot_name}</robotNamespace>
+		<type>transmission_interface/SimpleTransmission</type>
+		<joint name="${robot_name}_striker_joint_1">
+			<hardwareInterface>${hardware_interface}</hardwareInterface>
+		</joint>
+		<actuator name="${robot_name}_striker_motor_1">
+		    <hardwareInterface>${hardware_interface}</hardwareInterface>
+		    <mechanicalReduction>1</mechanicalReduction>
+		</actuator>
+	</transmission>
+	<transmission name="${robot_name}_striker_tran_2">
+		<robotNamespace>/${robot_name}</robotNamespace>
+		<type>transmission_interface/SimpleTransmission</type>
+		<joint name="${robot_name}_striker_joint_2">
+			<hardwareInterface>${hardware_interface}</hardwareInterface>
+		</joint>
+		<actuator name="${robot_name}_striker_motor_2">
+		    <hardwareInterface>${hardware_interface}</hardwareInterface>
+		    <mechanicalReduction>1</mechanicalReduction>
+		</actuator>
+	</transmission>
   </xacro:macro>
 </robot>

Commit message: Fixed small bugs in urdf

File: air_hockey_description/urdf/air_hockey.urdf (robot description, URDF)
Before this commit: robot iiwas, 35 links, 34 joints
Links:
- link B_striker_joint_link: mass 0.0 -> 0.01
- link F_striker_joint_link: mass 0.0 -> 0.01
Joints:
- joint B_striker_joint_1: limit lower=-1.5707963267948966 upper=1.5707963267948966 effort=10 velocity=10 -> lower=-1.5707963267948966 upper=1.5707963267948966 effort=100 velocity=100
- joint B_striker_joint_2: limit lower=-1.5707963267948966 upper=1.5707963267948966 effort=10 velocity=10 -> lower=-1.5707963267948966 upper=1.5707963267948966 effort=100 velocity=100
- joint F_striker_joint_1: limit lower=-1.5707963267948966 upper=1.5707963267948966 effort=10 velocity=10 -> lower=-1.5707963267948966 upper=1.5707963267948966 effort=100 velocity=100
- joint F_striker_joint_2: limit lower=-1.5707963267948966 upper=1.5707963267948966 effort=10 velocity=10 -> lower=-1.5707963267948966 upper=1.5707963267948966 effort=100 velocity=100
- joint back_base_joint: origin xyz=3.22 0.61 -0.015 rpy=0.0 0.0 0.0 -> xyz=3.22 0.0 -0.015 rpy=0.0 0.0 0.0
- joint back_in: origin xyz=0.0 -0.61 -0.0975 rpy=0.0 0.0 0.0 -> xyz=0.0 -0.0 -0.0975 rpy=0.0 0.0 0.0
- joint front_base_joint: origin xyz=0.2 -0.61 -0.015 rpy=0.0 0.0 0.0 -> xyz=0.2 0.0 -0.015 rpy=0.0 0.0 0.0
- joint front_in: origin xyz=0.0 0.61 -0.0975 rpy=0.0 0.0 0.0 -> xyz=0.0 -0.0 -0.0975 rpy=0.0 0.0 0.0

File: air_hockey_description/urdf/iiwa_striker.urdf.xacro (robot description, xacro)
@@ -40,15 +40,15 @@
 		<origin xyz="0.0 0.0 0.3455" rpy="0 0 0" />
 		<axis xyz="1 0 0"/>
-		<limit effort="10" lower="-${PI/2}" upper="${PI/2}" velocity="10"/>
+		<limit effort="100" lower="-${PI/2}" upper="${PI/2}" velocity="100"/>
 		<safety_controller k_position="100" k_velocity="2" soft_lower_limit="-2.094395102" soft_upper_limit="2.094395102"/>
-		<dynamics damping="0.5" friction="0.5"/>
+		<dynamics damping="0.5"/>
     </joint>
     <link name="${robot_name}_striker_joint_link">
     	<inertial>
 	        <origin xyz="0 0.0 0" rpy="0 0 0" />
-	        <mass value="0.0" />
+	        <mass value="0.01" />
 	        <inertia
-                ixx="0.0" ixy="0.0" ixz="0.0"
-                iyy="0.0" iyz="0.0" izz="0.0" />
+                ixx="0.0001" ixy="0.0" ixz="0.0"
+                iyy="0.0001" iyz="0.000000" izz="0.00001" />
       	</inertial>
     </link>
@@ -58,16 +58,16 @@
 		<origin xyz="0.0 0.0 0.0" rpy="0 0 0" />
 		<axis xyz="0 1 0"/>
-		<limit effort="10" lower="-${PI/2}" upper="${PI/2}" velocity="10"/>
+		<limit effort="100" lower="-${PI/2}" upper="${PI/2}" velocity="100"/>
 		<safety_controller k_position="100" k_velocity="2" soft_lower_limit="-2.094395102" soft_upper_limit="2.094395102"/>
-		<dynamics damping="0.5" friction="0.5"/>
+		<dynamics damping="0.5"/>
     </joint>
   <!--  The striker frame is here defined -->
     <link name="${robot_name}_striker_mallet">
       <inertial>
-        <origin xyz="0 0.0 0.0805" rpy="0 0 0" />
-        <mass value="0.0" />
+        <origin xyz="0 0.0 0.0" rpy="0 0 0" />
+        <mass value="0.1" />
         <inertia
-                ixx="0.0" ixy="0.0" ixz="0.0"
-                iyy="0.0" iyz="0.0" izz="0.0" />
+                ixx="0.0001" ixy="0.0" ixz="0.0"
+                iyy="0.0001" iyz="0.0" izz="0.0001" />
       </inertial>
       <visual>
@@ -105,11 +105,9 @@
     </joint>
     <link name="${robot_name}_striker_mallet_tip">
-    	<inertial>
-	        <origin xyz="0 0.0 0" rpy="0 0 0" />
-	        <mass value="0.0" />
-	        <inertia
-                ixx="0.0" ixy="0.0" ixz="0.0"
-                iyy="0.0" iyz="0.0" izz="0.0" />
-      	</inertial>
+      <inertial>
+        <origin rpy="0 0 0" xyz="0 0 0.0"/>
+        <mass value="0.0"/>
+        <inertia ixx="0.0" ixy="0.0" ixz="0.0" iyy="0.0" iyz="0.0" izz="0.0"/>
+      </inertial>
     </link>
     <gazebo reference="${robot_name}_striker_base">
