Commit message: Add air hockey launch file and gazebo simulation
- update mesh file
- update urdf
- reconstruct the structure the launch

File: air_hockey_description/urdf/iiwa_striker.urdf.xacro (robot description, xacro)
@@ -1,160 +1,28 @@
 <?xml version="1.0"?>
-<!-- Here we define the robot, we named it "iiwa14_tool" -->
-<robot xmlns:xacro="http://www.ros.org/wiki/xacro">
-  <!-- Tool properties -->
-  <xacro:property name="tool_mass" value="0.200" />
-  <xacro:property name="tool_joint_offset" value="0.00 0.00 0.00" />
-  <xacro:property name="tool_link_offset" value="-0.16 0.0 0.0" />
-  <xacro:macro name="striker" params="robot_name parent hardware_interface">
-    <joint name="${robot_name}_striker" type="fixed">
-		<parent link="${parent}" />
-		<child link = "${robot_name}_striker_base" />
-		<origin xyz="0.0 0.0 0.0" rpy="0 0 0" />
-    </joint>
-    <link name="${robot_name}_striker_base">
-		<inertial>
-		<origin xyz="0 0 0.0417" rpy="0 0 0" />
-		<mass value="0.1" />
-		<inertia
-			ixx="0.000297" ixy="0.0" ixz="0.0"
-			iyy="0.000271" iyz="0.0000001" izz="0.0000653" />
-		</inertial>
-		<visual>
-		<origin xyz="0 0 0" rpy="0 0.0 0"/>
-		<geometry>
-		  	<mesh filename="package://air_hockey_description/meshes/striker_new/visual/gas_spring.stl"/>
-		</geometry>
-		<material name="Grey"/>
-		</visual>
-		<collision>
-		<origin xyz="0 0 0" rpy="0 0 0"/>
-		<geometry>
-		  	<mesh filename="package://air_hockey_description/meshes/striker_new/collision/gas_spring_collision.stl"/>
-		</geometry>
-		<material name="Grey"/>
-		</collision>
-    </link>
-    <joint name="${robot_name}_striker_joint_1" type="revolute">
-		<parent link="${robot_name}_striker_base" />
-		<child link = "${robot_name}_striker_joint_link" />
-		<origin xyz="0.0 0.0 0.3455" rpy="0 0 0" />
-		<axis xyz="1 0 0"/>
-		<limit effort="100" lower="-${PI/2}" upper="${PI/2}" velocity="100"/>
-		<safety_controller k_position="100" k_velocity="2" soft_lower_limit="-2.094395102" soft_upper_limit="2.094395102"/>
-		<dynamics damping="0.5"/>
-    </joint>
-    <link name="${robot_name}_striker_joint_link">
-    	<inertial>
-	        <origin xyz="0 0.0 0" rpy="0 0 0" />
-	        <mass value="0.01" />
-	        <inertia
-                ixx="0.0001" ixy="0.0" ixz="0.0"
-                iyy="0.0001" iyz="0.000000" izz="0.00001" />
-      	</inertial>
-    </link>
-    <joint name="${robot_name}_striker_joint_2" type="revolute">
-		<parent link="${robot_name}_striker_joint_link" />
-		<child link = "${robot_name}_striker_mallet" />
-		<origin xyz="0.0 0.0 0.0" rpy="0 0 0" />
-		<axis xyz="0 1 0"/>
-		<limit effort="100" lower="-${PI/2}" upper="${PI/2}" velocity="100"/>
-		<safety_controller k_position="100" k_velocity="2" soft_lower_limit="-2.094395102" soft_upper_limit="2.094395102"/>
-		<dynamics damping="0.5"/>
-    </joint>
-  <!--  The striker frame is here defined -->
-    <link name="${robot_name}_striker_mallet">
-      <inertial>
-        <origin xyz="0 0.0 0.0" rpy="0 0 0" />
-        <mass value="0.1" />
-        <inertia
-                ixx="0.0001" ixy="0.0" ixz="0.0"
-                iyy="0.0001" iyz="0.0" izz="0.0001" />
-      </inertial>
-      <visual>
-        <origin xyz="0 0.0 0.0" rpy="0.0 0.0 0"/>
-        <geometry>
-        	<mesh filename="package://air_hockey_description/meshes/striker_new/visual/joint_mallet.stl"/>
-        </geometry>
-        <material name="Grey"/>
-      </visual>
-      <collision>
-        <origin xyz="0 0.0 0.0" rpy="0.0 0.0 0"/>
-        <geometry>
-          	<mesh filename="package://air_hockey_description/meshes/striker_new/collision/joint_mallet_collision.stl"/>
-        </geometry>
-        <material name="Grey"/>
-        <surface>
-            <bounce>
-                <restitution_coefficient>0.8</restitution_coefficient>
-            </bounce>
-            <contact>
-                <ode>
-                    <soft_cfm>0.1</soft_cfm>
-                    <soft_erp>0.1</soft_erp>
-                    <max_vel>1</max_vel>
-                </ode>
-            </contact>
-        </surface>
-      </collision>
-    </link>
-    <joint name="${robot_name}_striker_mallet_fix" type="fixed">
-		<parent link="${robot_name}_striker_mallet" />
-		<child link = "${robot_name}_striker_mallet_tip" />
-		<origin xyz="0.0 0.0 0.0805" rpy="0 0 0" />
-		<axis xyz="1 0 0"/>
-    </joint>
-    <link name="${robot_name}_striker_mallet_tip">
-      <inertial>
-        <origin rpy="0 0 0" xyz="0 0 0.0"/>
-        <mass value="0.0"/>
-        <inertia ixx="0.0" ixy="0.0" ixz="0.0" iyy="0.0" iyz="0.0" izz="0.0"/>
-      </inertial>
-    </link>
-    <gazebo reference="${robot_name}_striker_base">
-			<material>Gazebo/Grey</material>
-			<mu1>0.2</mu1>
-			<mu2>0.2</mu2>
-			<selfCollide>0</selfCollide>
+<robot name="iiwa_striker" xmlns:xacro="http://www.ros.org/wiki/xacro">
+    <!-- Import Rviz colors -->
+    <xacro:include filename="$(find iiwas_description)/urdf/materials.xacro" />
+    <!--Import the lbr iiwa macro -->
+    <xacro:include filename="$(find iiwas_description)/urdf/iiwa14.xacro"/>
+    <!--Import the striker macro -->
+    <xacro:include filename="$(find air_hockey_description)/urdf/striker.xacro"/>
+    <xacro:property name="base_height" default="0.03"/>
+    <xacro:arg name="hardware_interface" default="hardware_interface/PositionJointInterface"/>
+    <xacro:arg name="robot_name" default="F"/>
+    <xacro:arg name="parent" default="front_base"/>
+    <xacro:arg name="base_rpy" default="0 0 0"/>
+    <!-- Fix to world just for testing -->
+    <link name="$(arg parent)"/>
+    <!--iiwa-->
+    <xacro:iiwa14 hardware_interface="$(arg hardware_interface)" robot_name="$(arg robot_name)" parent="$(arg parent)">
+        <origin xyz="0 0 ${base_height/2}" rpy="$(arg base_rpy)" />
+    </xacro:iiwa14>
+    <xacro:striker hardware_interface="hardware_interface/PositionJointInterface" robot_name="$(arg robot_name)"/>
+    <gazebo reference="$(arg parent)">
+        <kinematic>true</kinematic>
     </gazebo>
-    <gazebo reference="${robot_name}_striker_joint_link">
-		<material>Gazebo/Grey</material>
-		<mu1>0.2</mu1>
-		<mu2>0.2</mu2>
-		<selfCollide>0</selfCollide>
+    <gazebo>
+        <plugin name="gazebo_ros_control" filename="libgazebo_ros_control.so">
+        </plugin>
     </gazebo>
-    <gazebo reference="${robot_name}_striker_mallet">
-			<material>Gazebo/Grey</material>
-			<mu1>0.2</mu1>
-			<mu2>0.2</mu2>
-			<selfCollide>0</selfCollide>
-    </gazebo>
-    <gazebo reference="${robot_name}_striker_mallet_tip">
-			<material>Gazebo/Grey</material>
-			<mu1>0.2</mu1>
-			<mu2>0.2</mu2>
-			<selfCollide>0</selfCollide>
-    </gazebo>
-    <transmission name="${robot_name}_striker_tran_1">
-		<robotNamespace>/${robot_name}</robotNamespace>
-		<type>transmission_interface/SimpleTransmission</type>
-		<joint name="${robot_name}_striker_joint_1">
-			<hardwareInterface>${hardware_interface}</hardwareInterface>
-		</joint>
-		<actuator name="${robot_name}_striker_motor_1">
-		    <hardwareInterface>${hardware_interface}</hardwareInterface>
-		    <mechanicalReduction>1</mechanicalReduction>
-		</actuator>
-	</transmission>
-	<transmission name="${robot_name}_striker_tran_2">
-		<robotNamespace>/${robot_name}</robotNamespace>
-		<type>transmission_interface/SimpleTransmission</type>
-		<joint name="${robot_name}_striker_joint_2">
-			<hardwareInterface>${hardware_interface}</hardwareInterface>
-		</joint>
-		<actuator name="${robot_name}_striker_motor_2">
-		    <hardwareInterface>${hardware_interface}</hardwareInterface>
-		    <mechanicalReduction>1</mechanicalReduction>
-		</actuator>
-	</transmission>
-  </xacro:macro>
 </robot>

File: air_hockey_description/urdf/puck/model.urdf.xacro (robot description, xacro)
@@ -10,7 +10,7 @@
         <color rgba="1.0 0.0 0.0 1"/>
     </material>
-    <xacro:arg name="table_base_x" default="0.0"/>
-    <xacro:arg name="table_base_y" default="0.0"/>
-    <xacro:arg name="table_base_z" default="0.0"/>
+    <xacro:arg name="puck_base_x" default="0.0"/>
+    <xacro:arg name="puck_base_y" default="0.0"/>
+    <xacro:arg name="puck_base_z" default="0.0"/>
     <xacro:property name="table_base_length" value="2.14"/>
     <xacro:property name="table_base_width" value="1.22"/>
@@ -23,5 +23,6 @@
     <xacro:property name="table_rim_vertical_width" value="0.09"/>
     <xacro:property name="table_rim_vertical_height" value="0.03"/>
-    <xacro:macro name="air_hockey_table" params="base_x base_y base_z">
+    <xacro:macro name="puck" params="base_x base_y base_z">
+        <link name="world"/>
         <joint name="base_joint" type="fixed">
             <origin xyz="${base_x} ${base_y} ${base_z - table_base_height/2}" rpy="0 0 0"/>

Commit message: Use effort joint interface for universal joint
- Set PID of universal joint to 0
- Increase the inertia of the endeffector

File: air_hockey_description/urdf/iiwa_striker.urdf.xacro (robot description, xacro)
@@ -18,5 +18,5 @@
         <origin xyz="0 0 ${base_height/2}" rpy="$(arg base_rpy)" />
     </xacro:iiwa14>
-    <xacro:striker hardware_interface="hardware_interface/PositionJointInterface" robot_name="$(arg robot_name)"/>
+    <xacro:striker hardware_interface="hardware_interface/EffortJointInterface" robot_name="$(arg robot_name)"/>
     <gazebo reference="$(arg parent)">
         <kinematic>true</kinematic>

File: air_hockey_description/urdf/striker.xacro (robot description, xacro)
@@ -11,7 +11,8 @@
                 <origin xyz="0 0 0" rpy="0 0 0"/>
                 <mass value="0.1"/>
-                <inertia
-                        ixx="0.000297" ixy="0.0" ixz="0.0"
-                        iyy="0.000271" iyz="0.0000001" izz="0.0000653"/>
+<!--                <inertia ixx="0.000297" ixy="0.0" ixz="0.0"-->
+<!--                         iyy="0.000271" iyz="0.0000001" izz="0.0000653"/>-->
+                <inertia ixx="0.01" ixy="0.0" ixz="0.0"
+                         iyy="0.01" iyz="0.0" izz="0.01"/>
             </inertial>
             <visual>
@@ -38,5 +39,5 @@
             <safety_controller k_position="100" k_velocity="2" soft_lower_limit="-2.094395102"
                                soft_upper_limit="2.094395102"/>
-            <dynamics damping="0.5"/>
+            <dynamics damping="0.1"/>
         </joint>
         <link name="${robot_name}_striker_joint_link">
@@ -44,7 +45,9 @@
                 <origin xyz="0 0.0 0" rpy="0 0 0"/>
                 <mass value="0.01"/>
-                <inertia
-                        ixx="0.0001" ixy="0.0" ixz="0.0"
-                        iyy="0.0001" iyz="0.000000" izz="0.00001"/>
+<!--                <inertia-->
+<!--                        ixx="0.0001" ixy="0.0" ixz="0.0"-->
+<!--                        iyy="0.0001" iyz="0.000000" izz="0.00001"/>-->
+                <inertia ixx="0.01" ixy="0.0" ixz="0.0"
+                         iyy="0.01" iyz="0.0" izz="0.01"/>
             </inertial>
             <visual>
@@ -71,5 +74,5 @@
             <safety_controller k_position="100" k_velocity="2" soft_lower_limit="-2.094395102"
                                soft_upper_limit="2.094395102"/>
-            <dynamics damping="0.5"/>
+            <dynamics damping="0.1"/>
         </joint>
         <!--  The striker frame is here defined -->
@@ -78,7 +81,9 @@
                 <origin xyz="0 0.0 0.0" rpy="0 0 0"/>
                 <mass value="0.1"/>
-                <inertia
-                        ixx="0.0001" ixy="0.0" ixz="0.0"
-                        iyy="0.0001" iyz="0.0" izz="0.0001"/>
+<!--                <inertia-->
+<!--                        ixx="0.0001" ixy="0.0" ixz="0.0"-->
+<!--                        iyy="0.0001" iyz="0.0" izz="0.0001"/>-->
+                <inertia ixx="0.01" ixy="0.0" ixz="0.0"
+                         iyy="0.01" iyz="0.0" izz="0.01"/>
             </inertial>
             <visual>
@@ -118,6 +123,9 @@
             <inertial>
                 <origin rpy="0 0 0" xyz="0 0 0.0"/>
-                <mass value="0.0"/>
-                <inertia ixx="0.0" ixy="0.0" ixz="0.0" iyy="0.0" iyz="0.0" izz="0.0"/>
+<!--                <mass value="0.0"/>-->
+<!--                <inertia ixx="0.0" ixy="0.0" ixz="0.0" iyy="0.0" iyz="0.0" izz="0.0"/>-->
+                <mass value="0.1"/>
+                <inertia ixx="0.01" ixy="0.0" ixz="0.0"
+                         iyy="0.01" iyz="0.0" izz="0.01"/>
             </inertial>
         </link>

Commit message: Temporal Changes, Nothing works

File: air_hockey_description/urdf/iiwa_striker.urdf.xacro (robot description, xacro)
@@ -18,5 +18,5 @@
         <origin xyz="0 0 ${base_height/2}" rpy="$(arg base_rpy)" />
     </xacro:iiwa14>
-    <xacro:striker hardware_interface="hardware_interface/EffortJointInterface" robot_name="$(arg robot_name)"/>
+    <xacro:striker hardware_interface="hardware_interface/PositionJointInterface" robot_name="$(arg robot_name)"/>
     <gazebo reference="$(arg parent)">
         <kinematic>true</kinematic>

File: air_hockey_description/urdf/striker.xacro (robot description, xacro)
@@ -17,5 +17,5 @@
             </inertial>
             <visual>
-                <origin xyz="0 0 0" rpy="0 0.0 0"/>
+                <origin xyz="0 0 0" rpy="0 0.0 ${PI/2}"/>
                 <geometry>
                     <mesh filename="package://air_hockey_description/meshes/striker/visual/EE_arm.stl"/>
@@ -34,5 +34,5 @@
             <child link="${robot_name}_striker_joint_link"/>
             <origin xyz="0.0 0.0 0.515" rpy="0 0 0"/>
-            <axis xyz="0 1 0"/>
+            <axis xyz="1 0 0"/>
             <limit effort="1" lower="-${PI/2}" upper="${PI/2}" velocity="100"/>
             <safety_controller k_position="100" k_velocity="2" soft_lower_limit="-2.094395102"
@@ -52,5 +52,5 @@
             <child link="${robot_name}_striker_mallet"/>
             <origin xyz="0.0 0.0 0.0" rpy="0 0 0"/>
-            <axis xyz="1 0 0"/>
+            <axis xyz="0 1 0"/>
             <limit effort="1" lower="-${PI/2}" upper="${PI/2}" velocity="100"/>
             <safety_controller k_position="100" k_velocity="2" soft_lower_limit="-2.094395102"
@@ -67,5 +67,5 @@
             </inertial>
             <visual>
-                <origin xyz="0 0.0 0.0" rpy="0.0 0.0 0"/>
+                <origin xyz="0 0.0 0.0" rpy="0.0 0.0 ${PI/2}"/>
                 <geometry>
                     <mesh filename="package://air_hockey_description/meshes/striker/visual/EE_mallet.stl"/>
@@ -74,5 +74,5 @@
             </visual>
             <collision>
-                <origin xyz="0 0.0 0.0" rpy="0.0 0.0 0"/>
+                <origin xyz="0 0.0 0.0" rpy="0.0 0.0 ${PI/2}"/>
                 <geometry>
                     <mesh filename="package://air_hockey_description/meshes/striker/collision/EE_mallet_collision.stl"/>

Commit message: Modifications for the new controller

File: air_hockey_description/urdf/iiwa_striker.urdf.xacro (robot description, xacro)
@@ -24,4 +24,5 @@
     <gazebo>
         <plugin name="gazebo_ros_control" filename="libgazebo_ros_control.so">
+          <robotSimType>iiwas_gazebo/GravityCompensationHWSim</robotSimType>
         </plugin>
     </gazebo>

File: air_hockey_description/urdf/striker.xacro (robot description, xacro)
@@ -43,5 +43,5 @@
             <inertial>
                 <origin xyz="0 0.0 0" rpy="0 0 0"/>
-                <mass value="0.1"/>vvvvv
+                <mass value="0.1"/>
                 <inertia ixx="0.001" ixy="0.0" ixz="0.0"
                          iyy="0.001" iyz="0.0" izz="0.001"/>

Commit message: Now Iiwas robots are fixed to world

File: air_hockey_description/urdf/iiwa_striker.urdf.xacro (robot description, xacro)
@@ -7,19 +7,15 @@
     <!--Import the striker macro -->
     <xacro:include filename="$(find air_hockey_description)/urdf/striker.xacro"/>
-    <xacro:property name="base_height" default="0.03"/>
     <xacro:arg name="hardware_interface" default="hardware_interface/PositionJointInterface"/>
     <xacro:arg name="robot_name" default="F"/>
-    <xacro:arg name="parent" default="front_base"/>
+    <xacro:arg name="parent" default="world"/>
+    <xacro:arg name="base_xyz" default="0 0 0"/>
     <xacro:arg name="base_rpy" default="0 0 0"/>
-    <!-- Fix to world just for testing -->
     <link name="$(arg parent)"/>
     <!--iiwa-->
     <xacro:iiwa14 hardware_interface="$(arg hardware_interface)" robot_name="$(arg robot_name)" parent="$(arg parent)">
-        <origin xyz="0 0 ${base_height/2}" rpy="$(arg base_rpy)" />
+        <origin xyz="$(arg base_xyz)" rpy="$(arg base_rpy)" />
     </xacro:iiwa14>
     <xacro:striker hardware_interface="hardware_interface/EffortJointInterface" robot_name="$(arg robot_name)"/>
-    <gazebo reference="$(arg parent)">
-        <kinematic>true</kinematic>
-    </gazebo>
     <gazebo>
         <plugin name="gazebo_ros_control" filename="libgazebo_ros_control.so">
