Commit message: Update the plot code and urdf

File: air_hockey_description/urdf/iiwa_striker.urdf (robot description, URDF)
Before this commit: robot iiwa_striker, 14 links, 13 joints
Links:
- removed link front_base
- added link world
- link F_link_1: mass 3.947808 -> 2.356723
- link F_link_2: mass 4.502752 -> 6.000000
- link F_link_3: mass 2.455197 -> 6.00000
- link F_link_4: mass 2.611550 -> 1.224529
- link F_link_5: mass 3.410009 -> 6.00000
- link F_link_6: mass 3.387949 -> 1.410742
- link F_link_7: mass 0.354321 -> 1.00000
- link F_striker_joint_link: mass 0.01 -> 0.1
Joints:
- removed joint front_base_F_base_joint
- added joint world_F_base_joint: type fixed, parent world, child F_link_0, origin xyz=0 0 0 rpy=0 0 0
- joint F_striker_joint_1: limit lower=-1.5707963267948966 upper=1.5707963267948966 effort=1 velocity=100 -> lower=-1.5707963267948966 upper=1.5707963267948966 effort=10 velocity=3.1415926
- joint F_striker_joint_2: limit lower=-1.5707963267948966 upper=1.5707963267948966 effort=1 velocity=100 -> lower=-1.5707963267948966 upper=1.5707963267948966 effort=10 velocity=3.1415926
- joint F_striker_mallet_fix: origin xyz=0.0 0.0 0.095 rpy=0 0 0 -> xyz=0.0 0.0 0.0505 rpy=0 0 0

Commit message: Add debug options for the baseline agent
- Refactor the logic of osqp optimizer
- Change the striker urdf

File: air_hockey_description/urdf/iiwa_striker.urdf (robot description, URDF)
Before this commit: robot iiwa_striker, 14 links, 13 joints
Links:
- link F_link_1: mass 2.356723 -> 3.854820
- link F_link_2: mass 6.000000 -> 5.773797
- link F_link_3: mass 6.00000 -> 5.953188
- link F_link_4: mass 1.224529 -> 3.448720
- link F_link_5: mass 6.00000 -> 4.007168
- link F_link_6: mass 1.410742 -> 2.415840
- link F_link_7: mass 1.00000 -> 1.107339
- link F_link_ee: mass 0.0 -> 1e-6
- link F_striker_joint_link: mass 0.1 -> 0.05
- link F_striker_mallet: geometry collision cylinder length=0.04 radius=0.04815; visual mesh filename=package://air_hockey_description/meshes/striker/visual/EE_m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
- link F_striker_mallet_tip: mass 0.1 -> 0.05
Joints:
- joint F_striker_joint_1: limit lower=-1.5707963267948966 upper=1.5707963267948966 effort=10 velocity=3.1415926 -> lower=-1.5707963267948966 upper=1.5707963267948966 effort=1 velocity=3.1415926
- joint F_striker_joint_2: limit lower=-1.5707963267948966 upper=1.5707963267948966 effort=10 velocity=3.1415926 -> lower=-1.5707963267948966 upper=1.5707963267948966 effort=1 velocity=3.1415926
- joint F_striker_mallet_fix: origin xyz=0.0 0.0 0.0505 rpy=0 0 0 -> xyz=0.0 0.0 0.0645 rpy=0 0 0

File: air_hockey_description/urdf/striker.xacro (robot description, xacro)
@@ -4,10 +4,10 @@
         <joint name="${robot_name}_striker" type="fixed">
             <parent link="${robot_name}_link_ee"/>
-            <child link="${robot_name}_striker_base"/>
-            <origin xyz="0.0 0.0 0.0" rpy="0 0 0"/>
+            <child link="${robot_name}_striker_tip"/>
+            <origin xyz="0.0 0.0 0.515" rpy="0 0 0"/>
         </joint>
-        <link name="${robot_name}_striker_base">
+        <link name="${robot_name}_striker_tip">
             <inertial>
-                <origin xyz="0 0 0.156" rpy="0 0 0"/>
+                <origin xyz="0 0 -0.359" rpy="0 0 0"/>
                 <mass value="0.350"/>
                 <inertia ixx="0.001" ixy="0.0" ixz="0.0"
@@ -15,5 +15,5 @@
             </inertial>
             <visual>
-                <origin xyz="0 0 0" rpy="0 0.0 0"/>
+                <origin xyz="0 0 -0.515" rpy="0 0.0 0"/>
                 <geometry>
                     <mesh filename="package://air_hockey_description/meshes/striker/visual/EE_arm.stl"/>
@@ -22,5 +22,5 @@
             </visual>
             <collision>
-                <origin xyz="0 0 0" rpy="0 0 0"/>
+                <origin xyz="0 0 -0.515" rpy="0 0 0"/>
                 <geometry>
                     <mesh filename="package://air_hockey_description/meshes/striker/collision/EE_arm_collision.stl"/>
@@ -29,7 +29,7 @@
         </link>
         <joint name="${robot_name}_striker_joint_1" type="revolute">
-            <parent link="${robot_name}_striker_base"/>
+            <parent link="${robot_name}_striker_tip"/>
             <child link="${robot_name}_striker_joint_link"/>
-            <origin xyz="0.0 0.0 0.515" rpy="0 0 0"/>
+            <origin xyz="0.0 0.0 0.0" rpy="0 0 0"/>
             <axis xyz="0 1 0"/>
             <limit effort="1" lower="-${PI/2}" upper="${PI/2}" velocity="3.1415926"/>
@@ -93,5 +93,5 @@
             </inertial>
         </link>
-        <gazebo reference="${robot_name}_striker_base">
+        <gazebo reference="${robot_name}_striker_tip">
             <collision>
                 <surface>

Commit message: Refactor the baseline_agent

File: air_hockey_description/urdf/iiwa_striker.urdf (robot description, URDF)
Before this commit: robot iiwa_striker, 14 links, 13 joints
Links:
- removed link F_striker_base
- removed link F_striker_joint_link
- removed link F_striker_mallet
- removed link F_striker_mallet_tip
- added link F_striker_tip, mass 0.350; collision mesh filename=package://air_hockey_description/meshes/striker/collision/E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; visual mesh filename=package://air_hockey_description/meshes/striker/visual/EE_a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
Joints:
- removed joint F_striker_joint_1
- removed joint F_striker_joint_2
- removed joint F_striker_mallet_fix
- joint F_striker: child F_striker_base -> F_striker_tip; origin xyz=0.0 0.0 0.0 rpy=0 0 0 -> xyz=0.0 0.0 0.515 rpy=0 0 0

File: air_hockey_description/urdf/iiwa_striker.urdf.xacro (robot description, xacro)
@@ -13,4 +13,5 @@
     <xacro:arg name="base_rpy" default="0 0 0"/>
     <xacro:arg name="dynamics_parameter" default="identified"/>
+    <xacro:arg name="contain_universal_joint" default="true"/>
     <link name="$(arg parent)"/>
     <!--iiwa-->
@@ -19,5 +20,6 @@
         <origin xyz="$(arg base_xyz)" rpy="$(arg base_rpy)" />
     </xacro:iiwa14>
-    <xacro:striker hardware_interface="hardware_interface/EffortJointInterface" robot_name="$(arg robot_name)"/>
+    <xacro:striker hardware_interface="hardware_interface/EffortJointInterface" robot_name="$(arg robot_name)"
+                   contain_universal_joint="$(arg contain_universal_joint)"/>
     <gazebo>
         <plugin name="gazebo_ros_control" filename="libgazebo_ros_control.so">

File: air_hockey_description/urdf/striker.xacro (robot description, xacro)
@@ -1,5 +1,5 @@
 <?xml version="1.0"?>
 <robot xmlns:xacro="http://www.ros.org/wiki/xacro">
-    <xacro:macro name="striker" params="robot_name hardware_interface">
+    <xacro:macro name="striker" params="robot_name hardware_interface contain_universal_joint">
         <joint name="${robot_name}_striker" type="fixed">
             <parent link="${robot_name}_link_ee"/>
@@ -28,4 +28,5 @@
             </collision>
         </link>
+        <xacro:if value="${contain_universal_joint}">
         <joint name="${robot_name}_striker_joint_1" type="revolute">
             <parent link="${robot_name}_striker_tip"/>
@@ -185,4 +186,5 @@
             </plugin>
         </gazebo>
+        </xacro:if>
     </xacro:macro>
 </robot>
