Commit message: Use iiwas_control in air_hockey package

File: air_hockey_description/urdf/striker.xacro (robot description, xacro)
@@ -38,5 +38,5 @@
             <safety_controller k_position="100" k_velocity="2" soft_lower_limit="-2.094395102"
                                soft_upper_limit="2.094395102"/>
-            <dynamics damping="0.3"/>
+            <dynamics damping="0.01"/>
         </joint>
         <link name="${robot_name}_striker_joint_link">
@@ -56,5 +56,5 @@
             <safety_controller k_position="100" k_velocity="2" soft_lower_limit="-2.094395102"
                                soft_upper_limit="2.094395102"/>
-            <dynamics damping="0.3"/>
+            <dynamics damping="0.01"/>
         </joint>
         <link name="${robot_name}_striker_mallet">

Commit message: Finish the Universal Joint Plugin

File: air_hockey_description/urdf/striker.xacro (robot description, xacro)
@@ -17,5 +17,5 @@
             </inertial>
             <visual>
-                <origin xyz="0 0 0" rpy="0 0.0 ${PI/2}"/>
+                <origin xyz="0 0 0" rpy="0 0.0 0"/>
                 <geometry>
                     <mesh filename="package://air_hockey_description/meshes/striker/visual/EE_arm.stl"/>
@@ -34,5 +34,5 @@
             <child link="${robot_name}_striker_joint_link"/>
             <origin xyz="0.0 0.0 0.515" rpy="0 0 0"/>
-            <axis xyz="1 0 0"/>
+            <axis xyz="0 1 0"/>
             <limit effort="1" lower="-${PI/2}" upper="${PI/2}" velocity="100"/>
             <safety_controller k_position="100" k_velocity="2" soft_lower_limit="-2.094395102"
@@ -52,5 +52,5 @@
             <child link="${robot_name}_striker_mallet"/>
             <origin xyz="0.0 0.0 0.0" rpy="0 0 0"/>
-            <axis xyz="0 1 0"/>
+            <axis xyz="1 0 0"/>
             <limit effort="1" lower="-${PI/2}" upper="${PI/2}" velocity="100"/>
             <safety_controller k_position="100" k_velocity="2" soft_lower_limit="-2.094395102"
@@ -67,5 +67,5 @@
             </inertial>
             <visual>
-                <origin xyz="0 0.0 0.0" rpy="0.0 0.0 ${PI/2}"/>
+                <origin xyz="0 0.0 0.0" rpy="0.0 0.0 0"/>
                 <geometry>
                     <mesh filename="package://air_hockey_description/meshes/striker/visual/EE_mallet.stl"/>
@@ -74,5 +74,5 @@
             </visual>
             <collision>
-                <origin xyz="0 0.0 0.0" rpy="0.0 0.0 ${PI/2}"/>
+                <origin xyz="0 0.0 0.0" rpy="0.0 0.0 0"/>
                 <geometry>
                     <mesh filename="package://air_hockey_description/meshes/striker/collision/EE_mallet_collision.stl"/>

Commit message: Tune the universal joint controller parameter

File: air_hockey_description/urdf/striker.xacro (robot description, xacro)
@@ -35,5 +35,5 @@
             <origin xyz="0.0 0.0 0.515" rpy="0 0 0"/>
             <axis xyz="0 1 0"/>
-            <limit effort="1" lower="-${PI/2}" upper="${PI/2}" velocity="100"/>
+            <limit effort="100" lower="-${PI/2}" upper="${PI/2}" velocity="100"/>
             <safety_controller k_position="100" k_velocity="2" soft_lower_limit="-2.094395102"
                                soft_upper_limit="2.094395102"/>
@@ -53,5 +53,5 @@
             <origin xyz="0.0 0.0 0.0" rpy="0 0 0"/>
             <axis xyz="1 0 0"/>
-            <limit effort="1" lower="-${PI/2}" upper="${PI/2}" velocity="100"/>
+            <limit effort="100" lower="-${PI/2}" upper="${PI/2}" velocity="100"/>
             <safety_controller k_position="100" k_velocity="2" soft_lower_limit="-2.094395102"
                                soft_upper_limit="2.094395102"/>

Commit message: Modify the striker xacro to disable the universal joint

File: air_hockey_description/urdf/striker.xacro (robot description, xacro)
@@ -35,5 +35,5 @@
             <origin xyz="0.0 0.0 0.515" rpy="0 0 0"/>
             <axis xyz="0 1 0"/>
-            <limit effort="100" lower="-${PI/2}" upper="${PI/2}" velocity="100"/>
+            <limit effort="100" lower="-${PI/2}" upper="${PI/2}" velocity="3.1415926"/>
             <safety_controller k_position="100" k_velocity="2" soft_lower_limit="-2.094395102"
                                soft_upper_limit="2.094395102"/>
@@ -53,5 +53,5 @@
             <origin xyz="0.0 0.0 0.0" rpy="0 0 0"/>
             <axis xyz="1 0 0"/>
-            <limit effort="100" lower="-${PI/2}" upper="${PI/2}" velocity="100"/>
+            <limit effort="100" lower="-${PI/2}" upper="${PI/2}" velocity="3.1415926"/>
             <safety_controller k_position="100" k_velocity="2" soft_lower_limit="-2.094395102"
                                soft_upper_limit="2.094395102"/>
@@ -129,26 +129,26 @@
             <preserveFixedJoint>1</preserveFixedJoint>
         </gazebo>
-        <transmission name="${robot_name}_striker_tran_1">
-            <robotNamespace>/${robot_name}</robotNamespace>
-            <type>transmission_interface/SimpleTransmission</type>
-            <joint name="${robot_name}_striker_joint_1">
-                <hardwareInterface>${hardware_interface}</hardwareInterface>
-            </joint>
-            <actuator name="${robot_name}_striker_motor_1">
-                <hardwareInterface>${hardware_interface}</hardwareInterface>
-                <mechanicalReduction>1</mechanicalReduction>
-            </actuator>
-        </transmission>
-        <transmission name="${robot_name}_striker_tran_2">
-            <robotNamespace>/${robot_name}</robotNamespace>
-            <type>transmission_interface/SimpleTransmission</type>
-            <joint name="${robot_name}_striker_joint_2">
-                <hardwareInterface>${hardware_interface}</hardwareInterface>
-            </joint>
-            <actuator name="${robot_name}_striker_motor_2">
-                <hardwareInterface>${hardware_interface}</hardwareInterface>
-                <mechanicalReduction>1</mechanicalReduction>
-            </actuator>
-        </transmission>
+<!--        <transmission name="${robot_name}_striker_tran_1">-->
+<!--            <robotNamespace>/${robot_name}</robotNamespace>-->
+<!--            <type>transmission_interface/SimpleTransmission</type>-->
+<!--            <joint name="${robot_name}_striker_joint_1">-->
+<!--                <hardwareInterface>${hardware_interface}</hardwareInterface>-->
+<!--            </joint>-->
+<!--            <actuator name="${robot_name}_striker_motor_1">-->
+<!--                <hardwareInterface>${hardware_interface}</hardwareInterface>-->
+<!--                <mechanicalReduction>1</mechanicalReduction>-->
+<!--            </actuator>-->
+<!--        </transmission>-->
+<!--        <transmission name="${robot_name}_striker_tran_2">-->
+<!--            <robotNamespace>/${robot_name}</robotNamespace>-->
+<!--            <type>transmission_interface/SimpleTransmission</type>-->
+<!--            <joint name="${robot_name}_striker_joint_2">-->
+<!--                <hardwareInterface>${hardware_interface}</hardwareInterface>-->
+<!--            </joint>-->
+<!--            <actuator name="${robot_name}_striker_motor_2">-->
+<!--                <hardwareInterface>${hardware_interface}</hardwareInterface>-->
+<!--                <mechanicalReduction>1</mechanicalReduction>-->
+<!--            </actuator>-->
+<!--        </transmission>-->
         <gazebo>
             <plugin name="univsersal_joint_plugin" filename="libuniversal_joint_plugin.so">

Commit message: Modify the anchor optimizer in velocity domain

File: air_hockey_description/urdf/striker.xacro (robot description, xacro)
@@ -35,5 +35,5 @@
             <origin xyz="0.0 0.0 0.515" rpy="0 0 0"/>
             <axis xyz="0 1 0"/>
-            <limit effort="100" lower="-${PI/2}" upper="${PI/2}" velocity="3.1415926"/>
+            <limit effort="10" lower="-${PI/2}" upper="${PI/2}" velocity="3.1415926"/>
             <safety_controller k_position="100" k_velocity="2" soft_lower_limit="-2.094395102"
                                soft_upper_limit="2.094395102"/>
@@ -53,5 +53,5 @@
             <origin xyz="0.0 0.0 0.0" rpy="0 0 0"/>
             <axis xyz="1 0 0"/>
-            <limit effort="100" lower="-${PI/2}" upper="${PI/2}" velocity="3.1415926"/>
+            <limit effort="10" lower="-${PI/2}" upper="${PI/2}" velocity="3.1415926"/>
             <safety_controller k_position="100" k_velocity="2" soft_lower_limit="-2.094395102"
                                soft_upper_limit="2.094395102"/>

Commit message: Use new mallet design

File: air_hockey_description/urdf/striker.xacro (robot description, xacro)
@@ -69,5 +69,6 @@
                 <origin xyz="0 0.0 0.0" rpy="0.0 0.0 0"/>
                 <geometry>
-                    <mesh filename="package://air_hockey_description/meshes/striker/visual/EE_mallet.stl"/>
+<!--                    <mesh filename="package://air_hockey_description/meshes/striker/visual/EE_mallet.stl"/>-->
+                    <mesh filename="package://air_hockey_description/meshes/striker/visual/EE_mallet_short.stl"/>
                 </geometry>
                 <material name="LightGrey"/>
@@ -76,5 +77,6 @@
                 <origin xyz="0 0.0 0.0" rpy="0.0 0.0 0"/>
                 <geometry>
-                    <mesh filename="package://air_hockey_description/meshes/striker/collision/EE_mallet_collision.stl"/>
+<!--                    <mesh filename="package://air_hockey_description/meshes/striker/collision/EE_mallet_collision.stl"/>-->
+                    <mesh filename="package://air_hockey_description/meshes/striker/collision/EE_mallet_short_collision.stl"/>
                 </geometry>
             </collision>
@@ -83,5 +85,6 @@
             <parent link="${robot_name}_striker_mallet"/>
             <child link="${robot_name}_striker_mallet_tip"/>
-            <origin xyz="0.0 0.0 0.095" rpy="0 0 0"/>
+<!--            <origin xyz="0.0 0.0 0.095" rpy="0 0 0"/>-->
+            <origin xyz="0.0 0.0 0.0505" rpy="0 0 0"/>
             <axis xyz="1 0 0"/>
         </joint>

Commit message: Add promp in script

File: air_hockey_description/urdf/striker.xacro (robot description, xacro)
@@ -13,6 +13,6 @@
 <!--                <inertia ixx="0.000297" ixy="0.0" ixz="0.0"-->
 <!--                         iyy="0.000271" iyz="0.0" izz="0.0000653"/>-->
-                <inertia ixx="0.005" ixy="0.0" ixz="0.0"
-                         iyy="0.005" iyz="0.0" izz="0.001"/>
+                <inertia ixx="0.0005" ixy="0.0" ixz="0.0"
+                         iyy="0.0005" iyz="0.0" izz="0.0001"/>
             </inertial>
             <visual>
@@ -44,6 +44,6 @@
                 <origin xyz="0 0.0 0" rpy="0 0 0"/>
                 <mass value="0.1"/>
-                <inertia ixx="0.001" ixy="0.0" ixz="0.0"
-                         iyy="0.001" iyz="0.0" izz="0.001"/>
+                <inertia ixx="0.0001" ixy="0.0" ixz="0.0"
+                         iyy="0.0001" iyz="0.0" izz="0.0001"/>
             </inertial>
         </link>

Commit message: Add air_hockey_pybullet package
- fixed minor issues in striker urdf

File: air_hockey_description/urdf/striker.xacro (robot description, xacro)
@@ -38,5 +38,5 @@
             <safety_controller k_position="100" k_velocity="2" soft_lower_limit="-2.094395102"
                                soft_upper_limit="2.094395102"/>
-            <dynamics damping="0.01"/>
+            <dynamics damping="0.2"/>
         </joint>
         <link name="${robot_name}_striker_joint_link">
@@ -56,9 +56,9 @@
             <safety_controller k_position="100" k_velocity="2" soft_lower_limit="-2.094395102"
                                soft_upper_limit="2.094395102"/>
-            <dynamics damping="0.01"/>
+            <dynamics damping="0.2"/>
         </joint>
         <link name="${robot_name}_striker_mallet">
             <inertial>
-                <origin xyz="0 0.0 0.078" rpy="0 0 0"/>
+                <origin xyz="0 0.0 0.0505" rpy="0 0 0"/>
                 <mass value="0.183"/>
                 <inertia

Commit message: Removing the damping from urdf

File: air_hockey_description/urdf/striker.xacro (robot description, xacro)
@@ -35,8 +35,8 @@
             <origin xyz="0.0 0.0 0.515" rpy="0 0 0"/>
             <axis xyz="0 1 0"/>
-            <limit effort="10" lower="-${PI/2}" upper="${PI/2}" velocity="3.1415926"/>
+            <limit effort="1" lower="-${PI/2}" upper="${PI/2}" velocity="3.1415926"/>
             <safety_controller k_position="100" k_velocity="2" soft_lower_limit="-2.094395102"
                                soft_upper_limit="2.094395102"/>
-            <dynamics damping="0.2"/>
+            <dynamics damping="0.0"/>
         </joint>
         <link name="${robot_name}_striker_joint_link">
@@ -53,8 +53,8 @@
             <origin xyz="0.0 0.0 0.0" rpy="0 0 0"/>
             <axis xyz="1 0 0"/>
-            <limit effort="10" lower="-${PI/2}" upper="${PI/2}" velocity="3.1415926"/>
+            <limit effort="1" lower="-${PI/2}" upper="${PI/2}" velocity="3.1415926"/>
             <safety_controller k_position="100" k_velocity="2" soft_lower_limit="-2.094395102"
                                soft_upper_limit="2.094395102"/>
-            <dynamics damping="0.2"/>
+            <dynamics damping="0.0"/>
         </joint>
         <link name="${robot_name}_striker_mallet">

Commit message: Update the setup for epfl parameter

File: air_hockey_description/urdf/striker.xacro (robot description, xacro)
@@ -11,8 +11,6 @@
                 <origin xyz="0 0 0.156" rpy="0 0 0"/>
                 <mass value="0.350"/>
-<!--                <inertia ixx="0.000297" ixy="0.0" ixz="0.0"-->
-<!--                         iyy="0.000271" iyz="0.0" izz="0.0000653"/>-->
-                <inertia ixx="0.0005" ixy="0.0" ixz="0.0"
-                         iyy="0.0005" iyz="0.0" izz="0.0001"/>
+                <inertia ixx="0.001" ixy="0.0" ixz="0.0"
+                         iyy="0.001" iyz="0.0" izz="0.001"/>
             </inertial>
             <visual>
@@ -36,14 +34,14 @@
             <axis xyz="0 1 0"/>
             <limit effort="1" lower="-${PI/2}" upper="${PI/2}" velocity="3.1415926"/>
-            <safety_controller k_position="100" k_velocity="2" soft_lower_limit="-2.094395102"
+            <safety_controller k_position="100" k_velocity="10" soft_lower_limit="-2.094395102"
                                soft_upper_limit="2.094395102"/>
-            <dynamics damping="0.0"/>
+            <dynamics damping="0.1"/>
         </joint>
         <link name="${robot_name}_striker_joint_link">
             <inertial>
                 <origin xyz="0 0.0 0" rpy="0 0 0"/>
-                <mass value="0.1"/>
-                <inertia ixx="0.0001" ixy="0.0" ixz="0.0"
-                         iyy="0.0001" iyz="0.0" izz="0.0001"/>
+                <mass value="0.05"/>
+                <inertia ixx="0.001" ixy="0.0" ixz="0.0"
+                         iyy="0.001" iyz="0.0" izz="0.001"/>
             </inertial>
         </link>
@@ -54,7 +52,7 @@
             <axis xyz="1 0 0"/>
             <limit effort="1" lower="-${PI/2}" upper="${PI/2}" velocity="3.1415926"/>
-            <safety_controller k_position="100" k_velocity="2" soft_lower_limit="-2.094395102"
+            <safety_controller k_position="100" k_velocity="10" soft_lower_limit="-2.094395102"
                                soft_upper_limit="2.094395102"/>
-            <dynamics damping="0.0"/>
+            <dynamics damping="0.1"/>
         </joint>
         <link name="${robot_name}_striker_mallet">
@@ -63,11 +61,10 @@
                 <mass value="0.183"/>
                 <inertia
-                        ixx="0.0001" ixy="0.0" ixz="0.0"
-                        iyy="0.0001" iyz="0.0" izz="0.0001"/>
+                        ixx="0.01" ixy="0.0" ixz="0.0"
+                        iyy="0.01" iyz="0.0" izz="0.01"/>
             </inertial>
             <visual>
                 <origin xyz="0 0.0 0.0" rpy="0.0 0.0 0"/>
                 <geometry>
-<!--                    <mesh filename="package://air_hockey_description/meshes/striker/visual/EE_mallet.stl"/>-->
                     <mesh filename="package://air_hockey_description/meshes/striker/visual/EE_mallet_short.stl"/>
                 </geometry>
@@ -77,5 +74,4 @@
                 <origin xyz="0 0.0 0.0" rpy="0.0 0.0 0"/>
                 <geometry>
-<!--                    <mesh filename="package://air_hockey_description/meshes/striker/collision/EE_mallet_collision.stl"/>-->
                     <mesh filename="package://air_hockey_description/meshes/striker/collision/EE_mallet_short_collision.stl"/>
                 </geometry>
@@ -85,5 +81,4 @@
             <parent link="${robot_name}_striker_mallet"/>
             <child link="${robot_name}_striker_mallet_tip"/>
-<!--            <origin xyz="0.0 0.0 0.095" rpy="0 0 0"/>-->
             <origin xyz="0.0 0.0 0.0505" rpy="0 0 0"/>
             <axis xyz="1 0 0"/>
@@ -93,19 +88,49 @@
             <inertial>
                 <origin rpy="0 0 0" xyz="0 0 0.0"/>
-                <mass value="0.1"/>
-                <inertia ixx="0.0001" ixy="0.0" ixz="0.0"
-                         iyy="0.0001" iyz="0.0" izz="0.0001"/>
+                <mass value="0.05"/>
+                <inertia ixx="0.001" ixy="0.0" ixz="0.0"
+                         iyy="0.001" iyz="0.0" izz="0.001"/>
             </inertial>
         </link>
         <gazebo reference="${robot_name}_striker_base">
+            <collision>
+                <surface>
+                    <bounce>
+                        <restitution_coefficient>1.0</restitution_coefficient>
+                        <threshold>0.0</threshold>
+                    </bounce>
+                    <contact>
+                        <collide_bitmask>0x02</collide_bitmask>
+                        <ode>
+                            <kp>1e9</kp>
+                            <max_vel>10</max_vel>
+                        </ode>
+                    </contact>
+                </surface>
+            </collision>
             <material>Gazebo/Grey</material>
-            <mu1>0.2</mu1>
-            <mu2>0.2</mu2>
+            <mu1>1.0</mu1>
+            <mu2>1.0</mu2>
             <selfCollide>0</selfCollide>
         </gazebo>
         <gazebo reference="${robot_name}_striker_joint_link">
+            <collision>
+                <surface>
+                    <bounce>
+                        <restitution_coefficient>1.0</restitution_coefficient>
+                        <threshold>0.0</threshold>
+                    </bounce>
+                    <contact>
+                        <collide_bitmask>0x02</collide_bitmask>
+                        <ode>
+                            <kp>1e9</kp>
+                            <max_vel>10</max_vel>
+                        </ode>
+                    </contact>
+                </surface>
+            </collision>
             <material>Gazebo/Grey</material>
-            <mu1>0.2</mu1>
-            <mu2>0.2</mu2>
+            <mu1>1.0</mu1>
+            <mu2>1.0</mu2>
             <selfCollide>0</selfCollide>
         </gazebo>

Commit message: Remove publisher in plugin

File: air_hockey_description/urdf/striker.xacro (robot description, xacro)
@@ -159,26 +159,26 @@
             <preserveFixedJoint>1</preserveFixedJoint>
         </gazebo>
-<!--        <transmission name="${robot_name}_striker_tran_1">-->
-<!--            <robotNamespace>/${robot_name}</robotNamespace>-->
-<!--            <type>transmission_interface/SimpleTransmission</type>-->
-<!--            <joint name="${robot_name}_striker_joint_1">-->
-<!--                <hardwareInterface>${hardware_interface}</hardwareInterface>-->
-<!--            </joint>-->
-<!--            <actuator name="${robot_name}_striker_motor_1">-->
-<!--                <hardwareInterface>${hardware_interface}</hardwareInterface>-->
-<!--                <mechanicalReduction>1</mechanicalReduction>-->
-<!--            </actuator>-->
-<!--        </transmission>-->
-<!--        <transmission name="${robot_name}_striker_tran_2">-->
-<!--            <robotNamespace>/${robot_name}</robotNamespace>-->
-<!--            <type>transmission_interface/SimpleTransmission</type>-->
-<!--            <joint name="${robot_name}_striker_joint_2">-->
-<!--                <hardwareInterface>${hardware_interface}</hardwareInterface>-->
-<!--            </joint>-->
-<!--            <actuator name="${robot_name}_striker_motor_2">-->
-<!--                <hardwareInterface>${hardware_interface}</hardwareInterface>-->
-<!--                <mechanicalReduction>1</mechanicalReduction>-->
-<!--            </actuator>-->
-<!--        </transmission>-->
+        <transmission name="${robot_name}_striker_tran_1">
+            <robotNamespace>/${robot_name}</robotNamespace>
+            <type>transmission_interface/SimpleTransmission</type>
+            <joint name="${robot_name}_striker_joint_1">
+                <hardwareInterface>${hardware_interface}</hardwareInterface>
+            </joint>
+            <actuator name="${robot_name}_striker_motor_1">
+                <hardwareInterface>${hardware_interface}</hardwareInterface>
+                <mechanicalReduction>1</mechanicalReduction>
+            </actuator>
+        </transmission>
+        <transmission name="${robot_name}_striker_tran_2">
+            <robotNamespace>/${robot_name}</robotNamespace>
+            <type>transmission_interface/SimpleTransmission</type>
+            <joint name="${robot_name}_striker_joint_2">
+                <hardwareInterface>${hardware_interface}</hardwareInterface>
+            </joint>
+            <actuator name="${robot_name}_striker_motor_2">
+                <hardwareInterface>${hardware_interface}</hardwareInterface>
+                <mechanicalReduction>1</mechanicalReduction>
+            </actuator>
+        </transmission>
         <gazebo>
             <plugin name="univsersal_joint_plugin" filename="libuniversal_joint_plugin.so">
