Commit message: Update the end-effector of the air hockey

File: air_hockey_description/urdf/striker.xacro (robot description, xacro)
@@ -58,5 +58,5 @@
         <link name="${robot_name}_striker_mallet">
             <inertial>
-                <origin xyz="0 0.0 0.0505" rpy="0 0 0"/>
+                <origin xyz="0 0.0 0.0645" rpy="0 0 0"/>
                 <mass value="0.183"/>
                 <inertia
@@ -67,12 +67,12 @@
                 <origin xyz="0 0.0 0.0" rpy="0.0 0.0 0"/>
                 <geometry>
-                    <mesh filename="package://air_hockey_description/meshes/striker/visual/EE_mallet_short.stl"/>
+                    <mesh filename="package://air_hockey_description/meshes/striker/visual/EE_mallet_foam.stl"/>
                 </geometry>
                 <material name="LightGrey"/>
             </visual>
             <collision>
-                <origin xyz="0 0.0 0.0" rpy="0.0 0.0 0"/>
+                <origin xyz="0 0.0 0.0455" rpy="0.0 0.0 0"/>
                 <geometry>
-                    <mesh filename="package://air_hockey_description/meshes/striker/collision/EE_mallet_short_collision.stl"/>
+                    <cylinder radius="0.04815" length="0.04"/>
                 </geometry>
             </collision>
@@ -81,5 +81,5 @@
             <parent link="${robot_name}_striker_mallet"/>
             <child link="${robot_name}_striker_mallet_tip"/>
-            <origin xyz="0.0 0.0 0.0505" rpy="0 0 0"/>
+            <origin xyz="0.0 0.0 0.0645" rpy="0 0 0"/>
             <axis xyz="1 0 0"/>
         </joint>

Commit message: Update the simulation

File: air_hockey_description/urdf/striker.xacro (robot description, xacro)
@@ -36,5 +36,5 @@
             <safety_controller k_position="100" k_velocity="10" soft_lower_limit="-2.094395102"
                                soft_upper_limit="2.094395102"/>
-            <dynamics damping="0.1"/>
+            <dynamics damping="0.05"/>
         </joint>
         <link name="${robot_name}_striker_joint_link">
@@ -54,5 +54,5 @@
             <safety_controller k_position="100" k_velocity="10" soft_lower_limit="-2.094395102"
                                soft_upper_limit="2.094395102"/>
-            <dynamics damping="0.1"/>
+            <dynamics damping="0.05"/>
         </joint>
         <link name="${robot_name}_striker_mallet">

Commit message: Update the trajectory optimization

File: air_hockey_description/urdf/striker.xacro (robot description, xacro)
@@ -1,4 +1,5 @@
 <?xml version="1.0"?>
 <robot xmlns:xacro="http://www.ros.org/wiki/xacro">
+    <xacro:property name="collide_bitmask" value="0x02"/>
     <xacro:macro name="striker" params="robot_name hardware_interface contain_universal_joint">
         <joint name="${robot_name}_striker" type="fixed">
@@ -102,5 +103,5 @@
                     </bounce>
                     <contact>
-                        <collide_bitmask>0x02</collide_bitmask>
+                        <collide_bitmask>${collide_bitmask}</collide_bitmask>
                         <ode>
                             <kp>1e9</kp>
@@ -123,5 +124,5 @@
                     </bounce>
                     <contact>
-                        <collide_bitmask>0x02</collide_bitmask>
+                        <collide_bitmask>${collide_bitmask}</collide_bitmask>
                         <ode>
                             <kp>1e9</kp>
@@ -144,5 +145,5 @@
                     </bounce>
                     <contact>
-                        <collide_bitmask>0x02</collide_bitmask>
+                        <collide_bitmask>${collide_bitmask}</collide_bitmask>
                         <ode>
                             <kp>1e9</kp>

Commit message: Remove the safe controller

File: air_hockey_description/urdf/striker.xacro (robot description, xacro)
@@ -35,7 +35,5 @@
             <origin xyz="0.0 0.0 0.0" rpy="0 0 0"/>
             <axis xyz="0 1 0"/>
-            <limit effort="1" lower="-${PI/2}" upper="${PI/2}" velocity="3.1415926"/>
-            <safety_controller k_position="100" k_velocity="10" soft_lower_limit="-2.094395102"
-                               soft_upper_limit="2.094395102"/>
+            <limit effort="1" lower="-${PI/2}" upper="${PI/2}"/>
             <dynamics damping="0.05"/>
         </joint>
@@ -53,7 +51,5 @@
             <origin xyz="0.0 0.0 0.0" rpy="0 0 0"/>
             <axis xyz="1 0 0"/>
-            <limit effort="1" lower="-${PI/2}" upper="${PI/2}" velocity="3.1415926"/>
-            <safety_controller k_position="100" k_velocity="10" soft_lower_limit="-2.094395102"
-                               soft_upper_limit="2.094395102"/>
+            <limit effort="1" lower="-${PI/2}" upper="${PI/2}"/>
             <dynamics damping="0.05"/>
         </joint>

Commit message: Fixed velocity limits bug

File: air_hockey_description/urdf/striker.xacro (robot description, xacro)
@@ -35,5 +35,5 @@
             <origin xyz="0.0 0.0 0.0" rpy="0 0 0"/>
             <axis xyz="0 1 0"/>
-            <limit effort="1" lower="-${PI/2}" upper="${PI/2}"/>
+            <limit effort="1" lower="-${PI/2}" upper="${PI/2}" velocity="3.1415926"/>
             <dynamics damping="0.05"/>
         </joint>
@@ -51,5 +51,5 @@
             <origin xyz="0.0 0.0 0.0" rpy="0 0 0"/>
             <axis xyz="1 0 0"/>
-            <limit effort="1" lower="-${PI/2}" upper="${PI/2}"/>
+            <limit effort="1" lower="-${PI/2}" upper="${PI/2}" velocity="3.1415926"/>
             <dynamics damping="0.05"/>
         </joint>
