Commit message: Add gazebo plugin of puck TF publisher
- remove old striker mesh file
- add gazebo plugin

File: air_hockey_description/urdf/puck/model.urdf.xacro (robot description, xacro)
@@ -29,5 +29,5 @@
                     <cylinder radius="${puck_radius}" length="${puck_height}"/>
                 </geometry>
-                <material name="Red"/>
+                <material name="red"/>
             </visual>
             <collision>
@@ -68,4 +68,8 @@
             <material>Gazebo/Red</material>
         </gazebo>
+        <gazebo>
+            <plugin name="puck_tf_plugin" filename="libpuck_tf_plugin.so">
+            </plugin>
+        </gazebo>
     </xacro:macro>
     <xacro:puck/>

Commit message: Use the try collision model, increase the workspace

File: air_hockey_description/urdf/puck/model.urdf.xacro (robot description, xacro)
@@ -32,7 +32,7 @@
             </visual>
             <collision>
-                <origin xyz="0 0 0.05" rpy="0 0 0"/>
+                <origin xyz="0 0 0.0" rpy="0 0 0"/>
                 <geometry>
-                    <cylinder radius="${puck_radius}" length="${puck_height + 0.1}"/>
+                    <cylinder radius="${puck_radius}" length="${puck_height}"/>
                 </geometry>
             </collision>

Commit message: Add pulgin for universal joint

File: air_hockey_description/urdf/puck/model.urdf.xacro (robot description, xacro)
@@ -69,4 +69,5 @@
         </gazebo>
         <gazebo>
+            <updateRate>100.0</updateRate>
             <plugin name="puck_tf_plugin" filename="libpuck_tf_plugin.so">
             </plugin>

File: air_hockey_description/urdf/striker.xacro (robot description, xacro)
@@ -12,5 +12,5 @@
                 <mass value="0.350"/>
 <!--                <inertia ixx="0.000297" ixy="0.0" ixz="0.0"-->
-<!--                         iyy="0.000271" iyz="0.0000001" izz="0.0000653"/>-->
+<!--                         iyy="0.000271" iyz="0.0" izz="0.0000653"/>-->
                 <inertia ixx="0.005" ixy="0.0" ixz="0.0"
                          iyy="0.005" iyz="0.0" izz="0.001"/>
@@ -65,6 +65,4 @@
                         ixx="0.0001" ixy="0.0" ixz="0.0"
                         iyy="0.0001" iyz="0.0" izz="0.0001"/>
-<!--                <inertia ixx="0.01" ixy="0.0" ixz="0.0"-->
-<!--                         iyy="0.01" iyz="0.0" izz="0.01"/>-->
             </inertial>
             <visual>
@@ -95,7 +93,4 @@
                 <inertia ixx="0.0001" ixy="0.0" ixz="0.0"
                          iyy="0.0001" iyz="0.0" izz="0.0001"/>
-<!--                <mass value="0.1"/>-->
-<!--                <inertia ixx="0.01" ixy="0.0" ixz="0.0"-->
-<!--                         iyy="0.01" iyz="0.0" izz="0.01"/>-->
             </inertial>
         </link>
@@ -156,4 +151,8 @@
             </actuator>
         </transmission>
+        <gazebo>
+            <plugin name="univsersal_joint_plugin" filename="libuniversal_joint_plugin.so">
+            </plugin>
+        </gazebo>
     </xacro:macro>
 </robot>

Commit message: Add some physics parameter to stablize the simulation

File: air_hockey_description/urdf/puck/model.urdf.xacro (robot description, xacro)
@@ -41,5 +41,5 @@
                 <lateral_friction value="${lateral_friction}"/>
                 <rolling_friction value="0.0"/>
-                <spinning_friction value="0.0"/>
+                <spinning_friction value="0.02"/>
             </contact>
         </link>
@@ -49,9 +49,12 @@
                     <bounce>
                         <restitution_coefficient>${restitution}</restitution_coefficient>
-                        <threshold>0.0</threshold>
+                        <threshold>0.01</threshold>
                     </bounce>
                     <friction>
                         <!-- For Gazebo Must contain tag ode, mu, mu2, check https://github.com/osrf/sdformat/issues/31 -->
                         <!-- https://github.com/osrf/gazebo/blob/gazebo11/gazebo/physics/bullet/BulletSurfaceParams.cc -->
+                        <torsional>
+                            <surface_radius>${puck_radius}</surface_radius>
+                        </torsional>
                         <ode>
                             <mu>${lateral_friction}</mu>
@@ -61,5 +64,6 @@
                     <contact>
                         <ode>
-                            <max_vel>100</max_vel>
+                            <kp>1e9</kp>
+                            <max_vel>1</max_vel>
                         </ode>
                     </contact>

File: air_hockey_description/urdf/striker.xacro (robot description, xacro)
@@ -43,7 +43,7 @@
             <inertial>
                 <origin xyz="0 0.0 0" rpy="0 0 0"/>
-                <mass value="0.01"/>
-                <inertia ixx="0.01" ixy="0.0" ixz="0.0"
-                         iyy="0.01" iyz="0.0" izz="0.01"/>
+                <mass value="0.1"/>vvvvv
+                <inertia ixx="0.001" ixy="0.0" ixz="0.0"
+                         iyy="0.001" iyz="0.0" izz="0.001"/>
             </inertial>
         </link>

Commit message: Add tactics repel
- Reset the logic of cut, prepare and ready

File: air_hockey_description/urdf/puck/model.urdf.xacro (robot description, xacro)
@@ -32,5 +32,5 @@
                 <origin xyz="0 0 0.0" rpy="0 0 0"/>
                 <mass value="0.01"/>
-                <inertia ixx="0.01" ixy="0" ixz="0" iyy="0.01" iyz="0" izz="5e-6"/>
+                <inertia ixx="0.001" ixy="0" ixz="0" iyy="0.001" iyz="0" izz="5e-6"/>
             </inertial>
             <visual>

Commit message: Update puck urdf

File: air_hockey_description/urdf/puck/model.urdf.xacro (robot description, xacro)
@@ -23,4 +23,52 @@
                                      lateral_friction spinning_friction linear_vel_decay angular_vel_decay">
         <link name="${puck_name}"/>
+        <joint name="{puck_name}_joint_weight_1" type="fixed">
+            <origin xyz="${puck_radius} 0 ${puck_height/2}" rpy="0 0 0"/>
+            <parent link="${puck_name}"/>
+            <child link="${puck_name}_link_weight_1"/>
+        </joint>
+        <link name="${puck_name}_link_weight_1">
+            <inertial>
+                <origin xyz="0 0 0.0" rpy="0 0 0"/>
+                <mass value="0.002"/>
+                <inertia ixx="0.00001" ixy="0" ixz="0" iyy="0.00001" iyz="0" izz="5e-6"/>
+            </inertial>
+        </link>
+        <joint name="{puck_name}_joint_weight_2" type="fixed">
+            <origin xyz="-${puck_radius} 0 ${puck_height/2}" rpy="0 0 0"/>
+            <parent link="${puck_name}"/>
+            <child link="${puck_name}_link_weight_2"/>
+        </joint>
+        <link name="${puck_name}_link_weight_2">
+            <inertial>
+                <origin xyz="0 0 0.0" rpy="0 0 0"/>
+                <mass value="0.002"/>
+                <inertia ixx="0.00001" ixy="0" ixz="0" iyy="0.00001" iyz="0" izz="5e-6"/>
+            </inertial>
+        </link>
+        <joint name="{puck_name}_joint_weight_3" type="fixed">
+            <origin xyz="0 ${puck_radius} ${puck_height/2}" rpy="0 0 0"/>
+            <parent link="${puck_name}"/>
+            <child link="${puck_name}_link_weight_3"/>
+        </joint>
+        <link name="${puck_name}_link_weight_3">
+            <inertial>
+                <origin xyz="0 0 0.0" rpy="0 0 0"/>
+                <mass value="0.002"/>
+                <inertia ixx="0.00001" ixy="0" ixz="0" iyy="0.00001" iyz="0" izz="5e-6"/>
+            </inertial>
+        </link>
+        <joint name="{puck_name}_joint_weight_4" type="fixed">
+            <origin xyz="0 -${puck_radius} ${puck_height/2}" rpy="0 0 0"/>
+            <parent link="${puck_name}"/>
+            <child link="${puck_name}_link_weight_4"/>
+        </joint>
+        <link name="${puck_name}_link_weight_4">
+            <inertial>
+                <origin xyz="0 0 0.0" rpy="0 0 0"/>
+                <mass value="0.002"/>
+                <inertia ixx="0.00001" ixy="0" ixz="0" iyy="0.00001" iyz="0" izz="5e-6"/>
+            </inertial>
+        </link>
         <joint name="{puck_name}_joint" type="fixed">
             <origin xyz="0 0 ${puck_height/2}" rpy="0 0 0"/>
@@ -31,5 +79,5 @@
             <inertial>
                 <origin xyz="0 0 0.0" rpy="0 0 0"/>
-                <mass value="0.01"/>
+                <mass value="0.002"/>
                 <inertia ixx="0.001" ixy="0" ixz="0" iyy="0.001" iyz="0" izz="5e-6"/>
             </inertial>
