Commit message: add sdf file for launch table and puck
- Update the mesh file of striker

File: air_hockey_description/urdf/air_hockey_table/model.urdf.xacro (robot description, xacro)
@@ -36,5 +36,5 @@
                 <inertia ixx="1" ixy="0" ixz="0" iyy="1" iyz="0" izz="1"/>
             </inertial>
-            <visual name="visual">
+            <visual>
                 <origin xyz="0 0 0.0" rpy="0 0 0"/>
                 <geometry>
@@ -43,5 +43,5 @@
                 <material name="white"/>
             </visual>
-            <collision name="collision">
+            <collision>
                 <origin xyz="0 0 0.0" rpy="0 0 0"/>
                 <geometry>
@@ -54,7 +54,9 @@
                     </bounce>
                     <friction>
-                        <ode>
-                            <mu>0</mu>
-                            <mu2>0</mu2>
+                        <!-- For Gazebo Must contain tag ode, mu, mu2, check https://github.com/osrf/sdformat/issues/31 -->
+                        <!-- https://github.com/osrf/gazebo/blob/gazebo11/gazebo/physics/bullet/BulletSurfaceParams.cc -->
+                        <ode>
+                            <mu>1.0</mu>
+                            <mu2>1.0</mu2>
                         </ode>
                     </friction>
@@ -74,4 +76,5 @@
             <parent link="t_base"/>
             <child link="t_down_rim_l"/>
+            <preserveFixedJoint>true</preserveFixedJoint>
         </joint>
         <link name="t_down_rim_l">
@@ -80,5 +83,5 @@
                 <inertia ixx="1" ixy="0" ixz="0" iyy="1" iyz="0" izz="1"/>
             </inertial>
-            <visual name="visual">
+            <visual>
                 <geometry>
                     <box size="${table_rim_horizon_length} ${table_rim_horizon_width} ${table_rim_horizon_height}"/>
@@ -86,5 +89,5 @@
                 <material name="grey"/>
             </visual>
-            <collision name="collision">
+            <collision>
                 <origin xyz="0.0 0.0 0.0"/>
                 <geometry>
@@ -97,7 +100,9 @@
                     </bounce>
                     <friction>
-                        <ode>
-                            <mu>0</mu>
-                            <mu2>0</mu2>
+                        <!-- For Gazebo Must contain tag ode, mu, mu2, check https://github.com/osrf/sdformat/issues/31 -->
+                        <!-- https://github.com/osrf/gazebo/blob/gazebo11/gazebo/physics/bullet/BulletSurfaceParams.cc -->
+                        <ode>
+                            <mu>1.0</mu>
+                            <mu2>1.0</mu2>
                         </ode>
                     </friction>
@@ -117,4 +122,5 @@
             <parent link="t_base"/>
             <child link="t_down_rim_r"/>
+            <preserveFixedJoint>true</preserveFixedJoint>
         </joint>
         <link name="t_down_rim_r">
@@ -123,5 +129,5 @@
                 <inertia ixx="1" ixy="0" ixz="0" iyy="1" iyz="0" izz="1"/>
             </inertial>
-            <visual name="visual">
+            <visual>
                 <geometry>
                     <box size="${table_rim_horizon_length} ${table_rim_horizon_width} ${table_rim_horizon_height}"/>
@@ -129,5 +135,5 @@
                 <material name="grey"/>
             </visual>
-            <collision name="collision">
+            <collision>
                 <origin xyz="0.0 0.0 0.0"/>
                 <geometry>
@@ -140,7 +146,9 @@
                     </bounce>
                     <friction>
-                        <ode>
-                            <mu>0</mu>
-                            <mu2>0</mu2>
+                        <!-- For Gazebo Must contain tag ode, mu, mu2, check https://github.com/osrf/sdformat/issues/31 -->
+                        <!-- https://github.com/osrf/gazebo/blob/gazebo11/gazebo/physics/bullet/BulletSurfaceParams.cc -->
+                        <ode>
+                            <mu>1.0</mu>
+                            <mu2>1.0</mu2>
                         </ode>
                     </friction>
@@ -160,4 +168,5 @@
             <parent link="t_base"/>
             <child link="t_down_rim_top"/>
+            <preserveFixedJoint>true</preserveFixedJoint>
         </joint>
         <link name="t_down_rim_top">
@@ -166,5 +175,5 @@
                 <inertia ixx="1" ixy="0" ixz="0" iyy="1" iyz="0" izz="1"/>
             </inertial>
-            <visual name="visual">
+            <visual>
                 <geometry>
                     <box size="${table_rim_horizon_length} ${table_base_width - 2 * table_rim_vertical_width} ${table_rim_horizon_top_height}"/>
@@ -172,5 +181,5 @@
                 <material name="grey"/>
             </visual>
-            <collision name="collision">
+            <collision>
                 <geometry>
                     <box size="${table_rim_horizon_length} ${table_base_width - 2 * table_rim_vertical_width} ${table_rim_horizon_top_height}"/>
@@ -182,7 +191,9 @@
                     </bounce>
                     <friction>
-                        <ode>
-                            <mu>0</mu>
-                            <mu2>0</mu2>
+                        <!-- For Gazebo Must contain tag ode, mu, mu2, check https://github.com/osrf/sdformat/issues/31 -->
+                        <!-- https://github.com/osrf/gazebo/blob/gazebo11/gazebo/physics/bullet/BulletSurfaceParams.cc -->
+                        <ode>
+                            <mu>1.0</mu>
+                            <mu2>1.0</mu2>
                         </ode>
                     </friction>
@@ -202,4 +213,5 @@
             <parent link="t_base"/>
             <child link="t_up_rim_l"/>
+            <preserveFixedJoint>true</preserveFixedJoint>
         </joint>
         <link name="t_up_rim_l">
@@ -208,5 +220,5 @@
                 <inertia ixx="1" ixy="0" ixz="0" iyy="1" iyz="0" izz="1"/>
             </inertial>
-            <visual name="visual">
+            <visual>
                 <geometry>
                     <box size="${table_rim_horizon_length} ${table_rim_horizon_width} ${table_rim_horizon_height}"/>
@@ -214,5 +226,5 @@
                 <material name="grey"/>
             </visual>
-            <collision name="collision">
+            <collision>
                 <origin xyz="0.0 0.0 0.0"/>
                 <geometry>
@@ -225,7 +237,9 @@
                     </bounce>
                     <friction>
-                        <ode>
-                            <mu>0</mu>
-                            <mu2>0</mu2>
+                        <!-- For Gazebo Must contain tag ode, mu, mu2, check https://github.com/osrf/sdformat/issues/31 -->
+                        <!-- https://github.com/osrf/gazebo/blob/gazebo11/gazebo/physics/bullet/BulletSurfaceParams.cc -->
+                        <ode>
+                            <mu>1.0</mu>
+                            <mu2>1.0</mu2>
                         </ode>
                     </friction>
@@ -245,4 +259,5 @@
             <parent link="t_base"/>
             <child link="t_up_rim_r"/>
+            <preserveFixedJoint>true</preserveFixedJoint>
         </joint>
         <link name="t_up_rim_r">
@@ -251,5 +266,5 @@
                 <inertia ixx="1" ixy="0" ixz="0" iyy="1" iyz="0" izz="1"/>
             </inertial>
-            <visual name="visual">
+            <visual>
                 <geometry>
                     <box size="${table_rim_horizon_length} ${table_rim_horizon_width} ${table_rim_horizon_height}"/>
@@ -257,5 +272,5 @@
                 <material name="grey"/>
             </visual>
-            <collision name="collision">
+            <collision>
                 <origin xyz="0.0 0.0 0.0"/>
                 <geometry>
@@ -268,7 +283,9 @@
                     </bounce>
                     <friction>
-                        <ode>
-                            <mu>0</mu>
-                            <mu2>0</mu2>
+                        <!-- For Gazebo Must contain tag ode, mu, mu2, check https://github.com/osrf/sdformat/issues/31 -->
+                        <!-- https://github.com/osrf/gazebo/blob/gazebo11/gazebo/physics/bullet/BulletSurfaceParams.cc -->
+                        <ode>
+                            <mu>1.0</mu>
+                            <mu2>1.0</mu2>
                         </ode>
                     </friction>
@@ -288,4 +305,5 @@
             <parent link="t_base"/>
             <child link="t_up_rim_top"/>
+            <preserveFixedJoint>true</preserveFixedJoint>
         </joint>
         <link name="t_up_rim_top">
@@ -294,5 +312,5 @@
                 <inertia ixx="1" ixy="0" ixz="0" iyy="1" iyz="0" izz="1"/>
             </inertial>
-            <visual name="visual">
+            <visual>
                 <geometry>
                     <box size="${table_rim_horizon_length} ${table_base_width - 2 * table_rim_vertical_width} ${table_rim_horizon_top_height}"/>
@@ -300,5 +318,5 @@
                 <material name="grey"/>
             </visual>
-            <collision name="collision">
+            <collision>
                 <geometry>
                     <box size="${table_rim_horizon_length} ${table_base_width - 2 * table_rim_vertical_width} ${table_rim_horizon_top_height}"/>
@@ -310,7 +328,9 @@
                     </bounce>
                     <friction>
-                        <ode>
-                            <mu>0</mu>
-                            <mu2>0</mu2>
+                        <!-- For Gazebo Must contain tag ode, mu, mu2, check https://github.com/osrf/sdformat/issues/31 -->
+                        <!-- https://github.com/osrf/gazebo/blob/gazebo11/gazebo/physics/bullet/BulletSurfaceParams.cc -->
+                        <ode>
+                            <mu>1.0</mu>
+                            <mu2>1.0</mu2>
                         </ode>
                     </friction>
@@ -330,4 +350,5 @@
             <parent link="t_base"/>
             <child link="t_left_rim"/>
+            <preserveFixedJoint>true</preserveFixedJoint>
         </joint>
         <link name="t_left_rim">
@@ -336,5 +357,5 @@
                 <inertia ixx="1" ixy="0" ixz="0" iyy="1" iyz="0" izz="1"/>
             </inertial>
-            <visual name="visual">
+            <visual>
                 <geometry>
                     <box size="${table_rim_vertical_length} ${table_rim_vertical_width} ${table_rim_vertical_height}"/>
@@ -342,5 +363,5 @@
                 <material name="grey"/>
             </visual>
-            <collision name="collision">
+            <collision>
                 <origin xyz="0.0 0.0 0.0"/>
                 <geometry>
@@ -353,7 +374,9 @@
                     </bounce>
                     <friction>
-                        <ode>
-                            <mu>0</mu>
-                            <mu2>0</mu2>
+                        <!-- For Gazebo Must contain tag ode, mu, mu2, check https://github.com/osrf/sdformat/issues/31 -->
+                        <!-- https://github.com/osrf/gazebo/blob/gazebo11/gazebo/physics/bullet/BulletSurfaceParams.cc -->
+                        <ode>
+                            <mu>1.0</mu>
+                            <mu2>1.0</mu2>
                         </ode>
                     </friction>
@@ -373,4 +396,5 @@
             <parent link="t_base"/>
             <child link="t_right_rim"/>
+            <preserveFixedJoint>true</preserveFixedJoint>
         </joint>
         <link name="t_right_rim">
@@ -379,5 +403,5 @@
                 <inertia ixx="1" ixy="0" ixz="0" iyy="1" iyz="0" izz="1"/>
             </inertial>
-            <visual name="visual">
+            <visual>
                 <geometry>
                     <box size="${table_rim_vertical_length} ${table_rim_vertical_width} ${table_rim_vertical_height}"/>
@@ -385,5 +409,5 @@
                 <material name="grey"/>
             </visual>
-            <collision name="collision">
+            <collision>
                 <origin xyz="0.0 0.0 0.0"/>
                 <geometry>
@@ -396,7 +420,9 @@
                     </bounce>
                     <friction>
-                        <ode>
-                            <mu>0</mu>
-                            <mu2>0</mu2>
+                        <!-- For Gazebo Must contain tag ode, mu, mu2, check https://github.com/osrf/sdformat/issues/31 -->
+                        <!-- https://github.com/osrf/gazebo/blob/gazebo11/gazebo/physics/bullet/BulletSurfaceParams.cc -->
+                        <ode>
+                            <mu>1.0</mu>
+                            <mu2>1.0</mu2>
                         </ode>
                     </friction>
