Commit message: add sdf file for launch table and puck
- Update the mesh file of striker

File: air_hockey_description/urdf/puck/model.urdf.xacro (robot description, xacro)
@@ -1,10 +1,4 @@
 <?xml version="1.0" encoding="utf-8"?>
 <robot xmlns:xacro="http://www.ros.org/wiki/xacro" name="air_hockey">
-    <material name="grey">
-        <color rgba="0.8 0.8 0.8 1"/>
-    </material>
-    <material name="white">
-        <color rgba="1.0 1.0 1.0 1"/>
-    </material>
     <material name="red">
         <color rgba="1.0 0.0 0.0 1"/>
@@ -13,403 +7,64 @@
     <xacro:arg name="puck_base_y" default="0.0"/>
     <xacro:arg name="puck_base_z" default="0.0"/>
-    <xacro:property name="table_base_length" value="2.14"/>
-    <xacro:property name="table_base_width" value="1.22"/>
-    <xacro:property name="table_base_height" value="0.11"/>
-    <xacro:property name="table_rim_horizon_length" value="0.09"/>
-    <xacro:property name="table_rim_horizon_width" value="0.395"/>
-    <xacro:property name="table_rim_horizon_height" value="0.01"/>
-    <xacro:property name="table_rim_horizon_top_height" value="0.02"/>
-    <xacro:property name="table_rim_vertical_length" value="2.14"/>
-    <xacro:property name="table_rim_vertical_width" value="0.09"/>
-    <xacro:property name="table_rim_vertical_height" value="0.03"/>
-    <xacro:macro name="puck" params="base_x base_y base_z">
-        <link name="world"/>
+    <xacro:property name="puck_radius" value="0.03165"/>
+    <xacro:property name="puck_height" value="0.0049"/>
+    <xacro:property name="restitution" value="0.8"/>
+    <xacro:property name="lateral_friction" value="0.04"/>
+    <xacro:property name="rolling_friction" value="0.8"/>
+    <xacro:property name="spinning_friction" value="0.04"/>
+    <xacro:macro name="puck">
+        <link name="root">
+        </link>
         <joint name="base_joint" type="fixed">
-            <origin xyz="${base_x} ${base_y} ${base_z - table_base_height/2}" rpy="0 0 0"/>
-            <parent link="world"/>
-            <child link="t_base"/>
+            <origin xyz="0 0 ${puck_height/2}" rpy="0 0 0"/>
+            <parent link="root"/>
+            <child link="base"/>
         </joint>
-        <link name="t_base">
+        <link name="base">
             <inertial>
                 <origin xyz="0 0 0.0" rpy="0 0 0"/>
-                <mass value="1"/>
-                <inertia ixx="1" ixy="0" ixz="0" iyy="1" iyz="0" izz="1"/>
+                <mass value="0.01"/>
+                <inertia ixx="1" ixy="0" ixz="0" iyy="1" iyz="0" izz="2e-5"/>
             </inertial>
-            <visual name="visual">
+            <visual>
                 <origin xyz="0 0 0.0" rpy="0 0 0"/>
                 <geometry>
-                    <box size="${table_base_length} ${table_base_width} ${table_base_height}"/>
+                    <cylinder radius="${puck_radius}" length="${puck_height}"/>
                 </geometry>
-                <material name="white"/>
+                <material name="red"/>
+                <material>Gazebo/Orange</material>
             </visual>
-            <collision name="collision">
+            <collision>
                 <origin xyz="0 0 0.0" rpy="0 0 0"/>
                 <geometry>
-                    <box size="${table_base_length} ${table_base_width} ${table_base_height}"/>
+                    <cylinder radius="${puck_radius}" length="${puck_height}"/>
                 </geometry>
                 <surface>
-                    <bounce>
-                        <restitution_coefficient>1.0</restitution_coefficient>
-                        <threshold>0</threshold>
-                    </bounce>
-                    <friction>
-                        <ode>
-                            <mu>0</mu>
-                            <mu2>0</mu2>
-                        </ode>
-                    </friction>
+                    <restitution_coefficient>${restitution}</restitution_coefficient>
+                    <threshold>0.01</threshold>
                 </surface>
+                <friction>
+                    <ode>
+                        <!-- For Gazebo Must contain tag ode, mu, mu2, check https://github.com/osrf/sdformat/issues/31 -->
+                        <!-- https://github.com/osrf/gazebo/blob/gazebo11/gazebo/physics/bullet/BulletSurfaceParams.cc -->
+                        <mu>${lateral_friction}</mu>
+                        <mu2>${lateral_friction}</mu2>
+                    </ode>
+                </friction>
             </collision>
             <contact>
-                <restitution value="1.0"/>
-                <lateral_friction value="1.0"/>
+                <restitution value="${restitution}"/>
+                <lateral_friction value="${lateral_friction}"/>
                 <rolling_friction value="0.0"/>
                 <spinning_friction value="0.0"/>
             </contact>
         </link>
-        <joint name="base_down_rim_l" type="fixed">
-            <origin rpy="0.0 0.0 0.0" xyz="${(table_base_length - table_rim_horizon_length) / 2}
-                                           ${table_base_width/2 - table_rim_vertical_width - table_rim_horizon_width / 2}
-                                           ${(table_base_height + table_rim_horizon_height) / 2}"/>
-            <parent link="t_base"/>
-            <child link="t_down_rim_l"/>
-        </joint>
-        <link name="t_down_rim_l">
-            <inertial>
-                <mass value="1.0"/>
-                <inertia ixx="1" ixy="0" ixz="0" iyy="1" iyz="0" izz="1"/>
-            </inertial>
-            <visual name="visual">
-                <geometry>
-                    <box size="${table_rim_horizon_length} ${table_rim_horizon_width} ${table_rim_horizon_height}"/>
-                </geometry>
-                <material name="grey"/>
-            </visual>
-            <collision name="collision">
-                <origin xyz="0.0 0.0 0.0"/>
-                <geometry>
-                    <box size="${table_rim_horizon_length} ${table_rim_horizon_width} ${table_rim_horizon_height + 0.1}"/>
-                </geometry>
-                <surface>
-                    <bounce>
-                        <restitution_coefficient>1.0</restitution_coefficient>
-                        <threshold>0</threshold>
-                    </bounce>
-                    <friction>
-                        <ode>
-                            <mu>0</mu>
-                            <mu2>0</mu2>
-                        </ode>
-                    </friction>
-                </surface>
-            </collision>
-            <contact>
-                <restitution value="1.0"/>
-                <lateral_friction value="0.0"/>
-                <rolling_friction value="0.0"/>
-                <spinning_friction value="0.0"/>
-            </contact>
-        </link>
-        <joint name="base_down_rim_r" type="fixed">
-            <origin rpy="0.0 0.0 0.0" xyz="${(table_base_length - table_rim_horizon_length) / 2}
-                                           -${table_base_width/2 - table_rim_vertical_width - table_rim_horizon_width / 2}
-                                           ${(table_base_height + table_rim_horizon_height) / 2}"/>
-            <parent link="t_base"/>
-            <child link="t_down_rim_r"/>
-        </joint>
-        <link name="t_down_rim_r">
-            <inertial>
-                <mass value="1.0"/>
-                <inertia ixx="1" ixy="0" ixz="0" iyy="1" iyz="0" izz="1"/>
-            </inertial>
-            <visual name="visual">
-                <geometry>
-                    <box size="${table_rim_horizon_length} ${table_rim_horizon_width} ${table_rim_horizon_height}"/>
-                </geometry>
-                <material name="grey"/>
-            </visual>
-            <collision name="collision">
-                <origin xyz="0.0 0.0 0.0"/>
-                <geometry>
-                    <box size="${table_rim_horizon_length} ${table_rim_horizon_width} ${table_rim_horizon_height + 0.1}"/>
-                </geometry>
-                <surface>
-                    <bounce>
-                        <restitution_coefficient>1.0</restitution_coefficient>
-                        <threshold>0</threshold>
-                    </bounce>
-                    <friction>
-                        <ode>
-                            <mu>0</mu>
-                            <mu2>0</mu2>
-                        </ode>
-                    </friction>
-                </surface>
-            </collision>
-            <contact>
-                <restitution value="1.0"/>
-                <lateral_friction value="0.0"/>
-                <rolling_friction value="0.0"/>
-                <spinning_friction value="0.0"/>
-            </contact>
-        </link>
-        <joint name="base_down_rim_top" type="fixed">
-            <origin rpy="0.0 0.0 0.0" xyz="${(table_base_length - table_rim_horizon_length) / 2}
-                                           0.0
-                                           ${(table_base_height + table_rim_horizon_top_height) / 2 + table_rim_horizon_height}"/>
-            <parent link="t_base"/>
-            <child link="t_down_rim_top"/>
-        </joint>
-        <link name="t_down_rim_top">
-            <inertial>
-                <mass value="1.0"/>
-                <inertia ixx="1" ixy="0" ixz="0" iyy="1" iyz="0" izz="1"/>
-            </inertial>
-            <visual name="visual">
-                <geometry>
-                    <box size="${table_rim_horizon_length} ${table_base_width - 2 * table_rim_vertical_width} ${table_rim_horizon_top_height}"/>
-                </geometry>
-                <material name="grey"/>
-            </visual>
-            <collision name="collision">
-                <geometry>
-                    <box size="${table_rim_horizon_length} ${table_base_width - 2 * table_rim_vertical_width} ${table_rim_horizon_top_height}"/>
-                </geometry>
-                <surface>
-                    <bounce>
-                        <restitution_coefficient>1.0</restitution_coefficient>
-                        <threshold>0</threshold>
-                    </bounce>
-                    <friction>
-                        <ode>
-                            <mu>0</mu>
-                            <mu2>0</mu2>
-                        </ode>
-                    </friction>
-                </surface>
-            </collision>
-            <contact>
-                <restitution value="1.0"/>
-                <lateral_friction value="0.0"/>
-                <rolling_friction value="0.0"/>
-                <spinning_friction value="0.0"/>
-            </contact>
-        </link>
-        <joint name="base_up_rim_l" type="fixed">
-            <origin rpy="0.0 0.0 0.0" xyz="-${(table_base_length - table_rim_horizon_length) / 2}
-                                           ${table_base_width/2 - table_rim_vertical_width - table_rim_horizon_width / 2}
-                                           ${(table_base_height + table_rim_horizon_height) / 2}"/>
-            <parent link="t_base"/>
-            <child link="t_up_rim_l"/>
-        </joint>
-        <link name="t_up_rim_l">
-            <inertial>
-                <mass value="1.0"/>
-                <inertia ixx="1" ixy="0" ixz="0" iyy="1" iyz="0" izz="1"/>
-            </inertial>
-            <visual name="visual">
-                <geometry>
-                    <box size="${table_rim_horizon_length} ${table_rim_horizon_width} ${table_rim_horizon_height}"/>
-                </geometry>
-                <material name="grey"/>
-            </visual>
-            <collision name="collision">
-                <origin xyz="0.0 0.0 0.0"/>
-                <geometry>
-                    <box size="${table_rim_horizon_length} ${table_rim_horizon_width} ${table_rim_horizon_height + 0.1}"/>
-                </geometry>
-                <surface>
-                    <bounce>
-                        <restitution_coefficient>1.0</restitution_coefficient>
-                        <threshold>0</threshold>
-                    </bounce>
-                    <friction>
-                        <ode>
-                            <mu>0</mu>
-                            <mu2>0</mu2>
-                        </ode>
-                    </friction>
-                </surface>
-            </collision>
-            <contact>
-                <restitution value="1.0"/>
-                <lateral_friction value="0.0"/>
-                <rolling_friction value="0.0"/>
-                <spinning_friction value="0.0"/>
-            </contact>
-        </link>
-        <joint name="base_up_rim_r" type="fixed">
-            <origin rpy="0.0 0.0 0.0" xyz="-${(table_base_length - table_rim_horizon_length) / 2}
-                                           -${table_base_width/2 - table_rim_vertical_width - table_rim_horizon_width / 2}
-                                           ${(table_base_height + table_rim_horizon_height) / 2}"/>
-            <parent link="t_base"/>
-            <child link="t_up_rim_r"/>
-        </joint>
-        <link name="t_up_rim_r">
-            <inertial>
-                <mass value="1.0"/>
-                <inertia ixx="1" ixy="0" ixz="0" iyy="1" iyz="0" izz="1"/>
-            </inertial>
-            <visual name="visual">
-                <geometry>
-                    <box size="${table_rim_horizon_length} ${table_rim_horizon_width} ${table_rim_horizon_height}"/>
-                </geometry>
-                <material name="grey"/>
-            </visual>
-            <collision name="collision">
-                <origin xyz="0.0 0.0 0.0"/>
-                <geometry>
-                    <box size="${table_rim_horizon_length} ${table_rim_horizon_width} ${table_rim_horizon_height + 0.1}"/>
-                </geometry>
-                <surface>
-                    <bounce>
-                        <restitution_coefficient>1.0</restitution_coefficient>
-                        <threshold>0</threshold>
-                    </bounce>
-                    <friction>
-                        <ode>
-                            <mu>0</mu>
-                            <mu2>0</mu2>
-                        </ode>
-                    </friction>
-                </surface>
-            </collision>
-            <contact>
-                <restitution value="1.0"/>
-                <lateral_friction value="0.0"/>
-                <rolling_friction value="0.0"/>
-                <spinning_friction value="0.0"/>
-            </contact>
-        </link>
-        <joint name="base_up_rim_top" type="fixed">
-            <origin rpy="0.0 0.0 0.0" xyz="-${(table_base_length - table_rim_horizon_length) / 2}
-                                           0.0
-                                           ${(table_base_height + table_rim_horizon_top_height) / 2 + table_rim_horizon_height}"/>
-            <parent link="t_base"/>
-            <child link="t_up_rim_top"/>
-        </joint>
-        <link name="t_up_rim_top">
-            <inertial>
-                <mass value="1.0"/>
-                <inertia ixx="1" ixy="0" ixz="0" iyy="1" iyz="0" izz="1"/>
-            </inertial>
-            <visual name="visual">
-                <geometry>
-                    <box size="${table_rim_horizon_length} ${table_base_width - 2 * table_rim_vertical_width} ${table_rim_horizon_top_height}"/>
-                </geometry>
-                <material name="grey"/>
-            </visual>
-            <collision name="collision">
-                <geometry>
-                    <box size="${table_rim_horizon_length} ${table_base_width - 2 * table_rim_vertical_width} ${table_rim_horizon_top_height}"/>
-                </geometry>
-                <surface>
-                    <bounce>
-                        <restitution_coefficient>1.0</restitution_coefficient>
-                        <threshold>0</threshold>
-                    </bounce>
-                    <friction>
-                        <ode>
-                            <mu>0</mu>
-                            <mu2>0</mu2>
-                        </ode>
-                    </friction>
-                </surface>
-            </collision>
-            <contact>
-                <restitution value="1.0"/>
-                <lateral_friction value="0.0"/>
-                <rolling_friction value="0.0"/>
-                <spinning_friction value="0.0"/>
-            </contact>
-        </link>
-        <joint name="base_left_rim" type="fixed">
-            <origin rpy="0.0 0.0 0.0" xyz="0.0
-                                           ${(table_base_width - table_rim_vertical_width) / 2}
-                                           ${(table_base_height + table_rim_vertical_height) / 2}"/>
-            <parent link="t_base"/>
-            <child link="t_left_rim"/>
-        </joint>
-        <link name="t_left_rim">
-            <inertial>
-                <mass value="1.0"/>
-                <inertia ixx="1" ixy="0" ixz="0" iyy="1" iyz="0" izz="1"/>
-            </inertial>
-            <visual name="visual">
-                <geometry>
-                    <box size="${table_rim_vertical_length} ${table_rim_vertical_width} ${table_rim_vertical_height}"/>
-                </geometry>
-                <material name="grey"/>
-            </visual>
-            <collision name="collision">
-                <origin xyz="0.0 0.0 0.0"/>
-                <geometry>
-                    <box size="${table_rim_vertical_length} ${table_rim_vertical_width} ${table_rim_vertical_height + 0.1}"/>
-                </geometry>
-                <surface>
-                    <bounce>
-                        <restitution_coefficient>1.0</restitution_coefficient>
-                        <threshold>0</threshold>
-                    </bounce>
-                    <friction>
-                        <ode>
-                            <mu>0</mu>
-                            <mu2>0</mu2>
-                        </ode>
-                    </friction>
-                </surface>
-            </collision>
-            <contact>
-                <restitution value="1.0"/>
-                <lateral_friction value="0.0"/>
-                <rolling_friction value="0.0"/>
-                <spinning_friction value="0.0"/>
-            </contact>
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
File: air_hockey_description/urdf/striker.xacro (robot description, xacro)
@@ -9,10 +9,10 @@
         <link name="${robot_name}_striker_base">
             <inertial>
-                <origin xyz="0 0 0" rpy="0 0 0"/>
-                <mass value="0.1"/>
+                <origin xyz="0 0 0.156" rpy="0 0 0"/>
+                <mass value="0.350"/>
 <!--                <inertia ixx="0.000297" ixy="0.0" ixz="0.0"-->
 <!--                         iyy="0.000271" iyz="0.0000001" izz="0.0000653"/>-->
-                <inertia ixx="0.01" ixy="0.0" ixz="0.0"
-                         iyy="0.01" iyz="0.0" izz="0.01"/>
+                <inertia ixx="0.005" ixy="0.0" ixz="0.0"
+                         iyy="0.005" iyz="0.0" izz="0.001"/>
             </inertial>
             <visual>
@@ -51,18 +51,18 @@
                          iyy="0.01" iyz="0.0" izz="0.01"/>
             </inertial>
-            <visual>
-                <origin xyz="0 0 0" rpy="0 0.0 0"/>
-                <geometry>
-                    <mesh filename="package://air_hockey_description/meshes/striker/visual/EE_joint.stl"/>
-                </geometry>
-                <material name="White"/>
-            </visual>
-            <collision>
-                <origin xyz="0 0 0" rpy="0 0 0"/>
-                <geometry>
-                    <mesh filename="package://air_hockey_description/meshes/striker/collision/EE_joint_collision.stl"/>
-                </geometry>
-                <material name="White"/>
-            </collision>
+<!--            <visual>-->
+<!--                <origin xyz="0 0 0" rpy="0 0.0 0"/>-->
+<!--                <geometry>-->
+<!--                    <mesh filename="package://air_hockey_description/meshes/striker/visual/EE_joint.stl"/>-->
+<!--                </geometry>-->
+<!--                <material name="White"/>-->
+<!--            </visual>-->
+<!--            <collision>-->
+<!--                <origin xyz="0 0 0" rpy="0 0 0"/>-->
+<!--                <geometry>-->
+<!--                    <mesh filename="package://air_hockey_description/meshes/striker/collision/EE_joint_collision.stl"/>-->
+<!--                </geometry>-->
+<!--                <material name="White"/>-->
+<!--            </collision>-->
         </link>
         <joint name="${robot_name}_striker_joint_2" type="revolute">
@@ -79,11 +79,11 @@
         <link name="${robot_name}_striker_mallet">
             <inertial>
-                <origin xyz="0 0.0 0.0" rpy="0 0 0"/>
-                <mass value="0.1"/>
-<!--                <inertia-->
-<!--                        ixx="0.0001" ixy="0.0" ixz="0.0"-->
-<!--                        iyy="0.0001" iyz="0.0" izz="0.0001"/>-->
-                <inertia ixx="0.01" ixy="0.0" ixz="0.0"
-                         iyy="0.01" iyz="0.0" izz="0.01"/>
+                <origin xyz="0 0.0 0.078" rpy="0 0 0"/>
+                <mass value="0.183"/>
+                <inertia
+                        ixx="0.0001" ixy="0.0" ixz="0.0"
+                        iyy="0.0001" iyz="0.0" izz="0.0001"/>
+<!--                <inertia ixx="0.01" ixy="0.0" ixz="0.0"-->
+<!--                         iyy="0.01" iyz="0.0" izz="0.01"/>-->
             </inertial>
             <visual>
@@ -123,9 +123,10 @@
             <inertial>
                 <origin rpy="0 0 0" xyz="0 0 0.0"/>
-<!--                <mass value="0.0"/>-->
-<!--                <inertia ixx="0.0" ixy="0.0" ixz="0.0" iyy="0.0" iyz="0.0" izz="0.0"/>-->
                 <mass value="0.1"/>
-                <inertia ixx="0.01" ixy="0.0" ixz="0.0"
-                         iyy="0.01" iyz="0.0" izz="0.01"/>
+                <inertia ixx="0.0001" ixy="0.0" ixz="0.0"
+                         iyy="0.0001" iyz="0.0" izz="0.0001"/>
+<!--                <mass value="0.1"/>-->
+<!--                <inertia ixx="0.01" ixy="0.0" ixz="0.0"-->
+<!--                         iyy="0.01" iyz="0.0" izz="0.01"/>-->
             </inertial>
         </link>
