Commit message: Update the pose and puck position

File: air_hockey_description/urdf/air_hockey_table/model.urdf.xacro (robot description, xacro)
@@ -10,7 +10,7 @@
         <color rgba="1.0 0.0 0.0 1"/>
     </material>
-    <xacro:arg name="table_base_x" default="0.0"/>
-    <xacro:arg name="table_base_y" default="0.0"/>
-    <xacro:arg name="table_base_z" default="0.0"/>
+    <xacro:arg name="table_surface_x" default="0.0"/>
+    <xacro:arg name="table_surface_y" default="0.0"/>
+    <xacro:arg name="table_surface_z" default="0.0"/>
     <xacro:property name="table_base_length" value="2.14"/>
     <xacro:property name="table_base_width" value="1.22"/>
@@ -23,8 +23,8 @@
     <xacro:property name="table_rim_vertical_width" value="0.09"/>
     <xacro:property name="table_rim_vertical_height" value="0.03"/>
-    <xacro:macro name="air_hockey_table" params="base_x base_y base_z">
+    <xacro:macro name="air_hockey_table" params="surface_x surface_y surface_z">
         <link name="world"/>
         <joint name="base_joint" type="fixed">
-            <origin xyz="${base_x} ${base_y} ${base_z - table_base_height/2}" rpy="0 0 0"/>
+            <origin xyz="${surface_x} ${surface_y} ${surface_z - table_base_height/2}" rpy="0 0 0"/>
             <parent link="world"/>
             <child link="t_base"/>
@@ -438,4 +438,4 @@
         <static>1</static>
     </xacro:macro>
-    <xacro:air_hockey_table base_x="$(arg table_base_x)" base_y="$(arg table_base_y)" base_z="$(arg table_base_z)"/>
+    <xacro:air_hockey_table surface_x="$(arg table_surface_x)" surface_y="$(arg table_surface_y)" surface_z="$(arg table_surface_z)"/>
 </robot>

File: air_hockey_description/urdf/striker.xacro (robot description, xacro)
@@ -101,7 +101,5 @@
                 <material name="White"/>
                 <surface>
-                    <bounce>
-                        <restitution_coefficient>0.8</restitution_coefficient>
-                    </bounce>
+                    <bounce restitution_coefficient="1.0" threshold="0.01"/>
                     <contact>
                         <ode>
