Commit message: Use urdf.xacro to launch the description

File: air_hockey_description/urdf/air_hockey_table/model.urdf.xacro (robot description, xacro)
@@ -1,4 +1,4 @@
 <?xml version="1.0" encoding="utf-8"?>
-<robot xmlns:xacro="http://www.ros.org/wiki/xacro" name="air_hockey">
+<robot name="air_hockey_table" xmlns:xacro="http://www.ros.org/wiki/xacro">
     <material name="grey">
         <color rgba="0.8 0.8 0.8 1"/>
@@ -48,18 +48,4 @@
                     <box size="${table_base_length} ${table_base_width} ${table_base_height}"/>
                 </geometry>
-                <surface>
-                    <bounce>
-                        <restitution_coefficient>1.0</restitution_coefficient>
-                        <threshold>0</threshold>
-                    </bounce>
-                    <friction>
-                        <!-- For Gazebo Must contain tag ode, mu, mu2, check https://github.com/osrf/sdformat/issues/31 -->
-                        <!-- https://github.com/osrf/gazebo/blob/gazebo11/gazebo/physics/bullet/BulletSurfaceParams.cc -->
-                        <ode>
-                            <mu>1.0</mu>
-                            <mu2>1.0</mu2>
-                        </ode>
-                    </friction>
-                </surface>
             </collision>
             <contact>
@@ -94,18 +80,4 @@
                     <box size="${table_rim_horizon_length} ${table_rim_horizon_width} ${table_rim_horizon_height + 0.1}"/>
                 </geometry>
-                <surface>
-                    <bounce>
-                        <restitution_coefficient>1.0</restitution_coefficient>
-                        <threshold>0</threshold>
-                    </bounce>
-                    <friction>
-                        <!-- For Gazebo Must contain tag ode, mu, mu2, check https://github.com/osrf/sdformat/issues/31 -->
-                        <!-- https://github.com/osrf/gazebo/blob/gazebo11/gazebo/physics/bullet/BulletSurfaceParams.cc -->
-                        <ode>
-                            <mu>1.0</mu>
-                            <mu2>1.0</mu2>
-                        </ode>
-                    </friction>
-                </surface>
             </collision>
             <contact>
@@ -140,18 +112,4 @@
                     <box size="${table_rim_horizon_length} ${table_rim_horizon_width} ${table_rim_horizon_height + 0.1}"/>
                 </geometry>
-                <surface>
-                    <bounce>
-                        <restitution_coefficient>1.0</restitution_coefficient>
-                        <threshold>0</threshold>
-                    </bounce>
-                    <friction>
-                        <!-- For Gazebo Must contain tag ode, mu, mu2, check https://github.com/osrf/sdformat/issues/31 -->
-                        <!-- https://github.com/osrf/gazebo/blob/gazebo11/gazebo/physics/bullet/BulletSurfaceParams.cc -->
-                        <ode>
-                            <mu>1.0</mu>
-                            <mu2>1.0</mu2>
-                        </ode>
-                    </friction>
-                </surface>
             </collision>
             <contact>
@@ -185,18 +143,4 @@
                     <box size="${table_rim_horizon_length} ${table_base_width - 2 * table_rim_vertical_width} ${table_rim_horizon_top_height}"/>
                 </geometry>
-                <surface>
-                    <bounce>
-                        <restitution_coefficient>1.0</restitution_coefficient>
-                        <threshold>0</threshold>
-                    </bounce>
-                    <friction>
-                        <!-- For Gazebo Must contain tag ode, mu, mu2, check https://github.com/osrf/sdformat/issues/31 -->
-                        <!-- https://github.com/osrf/gazebo/blob/gazebo11/gazebo/physics/bullet/BulletSurfaceParams.cc -->
-                        <ode>
-                            <mu>1.0</mu>
-                            <mu2>1.0</mu2>
-                        </ode>
-                    </friction>
-                </surface>
             </collision>
             <contact>
@@ -231,18 +175,4 @@
                     <box size="${table_rim_horizon_length} ${table_rim_horizon_width} ${table_rim_horizon_height + 0.1}"/>
                 </geometry>
-                <surface>
-                    <bounce>
-                        <restitution_coefficient>1.0</restitution_coefficient>
-                        <threshold>0</threshold>
-                    </bounce>
-                    <friction>
-                        <!-- For Gazebo Must contain tag ode, mu, mu2, check https://github.com/osrf/sdformat/issues/31 -->
-                        <!-- https://github.com/osrf/gazebo/blob/gazebo11/gazebo/physics/bullet/BulletSurfaceParams.cc -->
-                        <ode>
-                            <mu>1.0</mu>
-                            <mu2>1.0</mu2>
-                        </ode>
-                    </friction>
-                </surface>
             </collision>
             <contact>
@@ -277,18 +207,4 @@
                     <box size="${table_rim_horizon_length} ${table_rim_horizon_width} ${table_rim_horizon_height + 0.1}"/>
                 </geometry>
-                <surface>
-                    <bounce>
-                        <restitution_coefficient>1.0</restitution_coefficient>
-                        <threshold>0</threshold>
-                    </bounce>
-                    <friction>
-                        <!-- For Gazebo Must contain tag ode, mu, mu2, check https://github.com/osrf/sdformat/issues/31 -->
-                        <!-- https://github.com/osrf/gazebo/blob/gazebo11/gazebo/physics/bullet/BulletSurfaceParams.cc -->
-                        <ode>
-                            <mu>1.0</mu>
-                            <mu2>1.0</mu2>
-                        </ode>
-                    </friction>
-                </surface>
             </collision>
             <contact>
@@ -318,23 +234,4 @@
                 <material name="grey"/>
             </visual>
-            <collision>
-                <geometry>
-                    <box size="${table_rim_horizon_length} ${table_base_width - 2 * table_rim_vertical_width} ${table_rim_horizon_top_height}"/>
-                </geometry>
-                <surface>
-                    <bounce>
-                        <restitution_coefficient>1.0</restitution_coefficient>
-                        <threshold>0</threshold>
-                    </bounce>
-                    <friction>
-                        <!-- For Gazebo Must contain tag ode, mu, mu2, check https://github.com/osrf/sdformat/issues/31 -->
-                        <!-- https://github.com/osrf/gazebo/blob/gazebo11/gazebo/physics/bullet/BulletSurfaceParams.cc -->
-                        <ode>
-                            <mu>1.0</mu>
-                            <mu2>1.0</mu2>
-                        </ode>
-                    </friction>
-                </surface>
-            </collision>
             <contact>
                 <restitution value="1.0"/>
@@ -368,18 +265,4 @@
                     <box size="${table_rim_vertical_length} ${table_rim_vertical_width} ${table_rim_vertical_height + 0.1}"/>
                 </geometry>
-                <surface>
-                    <bounce>
-                        <restitution_coefficient>1.0</restitution_coefficient>
-                        <threshold>0</threshold>
-                    </bounce>
-                    <friction>
-                        <!-- For Gazebo Must contain tag ode, mu, mu2, check https://github.com/osrf/sdformat/issues/31 -->
-                        <!-- https://github.com/osrf/gazebo/blob/gazebo11/gazebo/physics/bullet/BulletSurfaceParams.cc -->
-                        <ode>
-                            <mu>1.0</mu>
-                            <mu2>1.0</mu2>
-                        </ode>
-                    </friction>
-                </surface>
             </collision>
             <contact>
@@ -414,26 +297,252 @@
                     <box size="${table_rim_vertical_length} ${table_rim_vertical_width} ${table_rim_vertical_height + 0.1}"/>
                 </geometry>
-                <surface>
-                    <bounce>
-                        <restitution_coefficient>1.0</restitution_coefficient>
-                        <threshold>0</threshold>
-                    </bounce>
-                    <friction>
-                        <!-- For Gazebo Must contain tag ode, mu, mu2, check https://github.com/osrf/sdformat/issues/31 -->
-                        <!-- https://github.com/osrf/gazebo/blob/gazebo11/gazebo/physics/bullet/BulletSurfaceParams.cc -->
-                        <ode>
-                            <mu>1.0</mu>
-                            <mu2>1.0</mu2>
-                        </ode>
-                    </friction>
-                </surface>
-            </collision>
-            <contact>
-                <restitution value="1.0"/>
-                <lateral_friction value="0.0"/>
-                <rolling_friction value="0.0"/>
-                <spinning_friction value="0.0"/>
-            </contact>
-        </link>
+            </collision>
+            <contact>
+                <restitution value="1.0"/>
+                <lateral_friction value="0.0"/>
+                <rolling_friction value="0.0"/>
+                <spinning_friction value="0.0"/>
+            </contact>
+        </link>
+        <gazebo reference="t_base">
+            <collision>
+                <surface>
+                    <bounce>
+                        <restitution_coefficient>1.0</restitution_coefficient>
+                        <threshold>0</threshold>
+                    </bounce>
+                    <friction>
+                        <!-- For Gazebo Must contain tag ode, mu, mu2, check https://github.com/osrf/sdformat/issues/31 -->
+                        <!-- https://github.com/osrf/gazebo/blob/gazebo11/gazebo/physics/bullet/BulletSurfaceParams.cc -->
+                        <ode>
+                            <mu>0.04</mu>
+                            <mu2>0.04</mu2>
+                        </ode>
+                    </friction>
+                    <contact>
+                        <ode>
+                            <max_vel>10</max_vel>
+                        </ode>
+                    </contact>
+                </surface>
+            </collision>
+            <material>Gazebo/White</material>
+        </gazebo>
+        <gazebo reference="base_down_rim_l">
+            <preserveFixedJoint>1</preserveFixedJoint>
+        </gazebo>
+        <gazebo reference="t_down_rim_l">
+            <collision>
+                <surface>
+                    <bounce>
+                        <restitution_coefficient>1.0</restitution_coefficient>
+                        <threshold>0</threshold>
+                    </bounce>
+                    <friction>
+                        <!-- For Gazebo Must contain tag ode, mu, mu2, check https://github.com/osrf/sdformat/issues/31 -->
+                        <!-- https://github.com/osrf/gazebo/blob/gazebo11/gazebo/physics/bullet/BulletSurfaceParams.cc -->
+                        <ode>
+                            <mu>0.04</mu>
+                            <mu2>0.04</mu2>
+                        </ode>
+                    </friction>
+                    <contact>
+                        <ode>
+                            <max_vel>10</max_vel>
+                        </ode>
+                    </contact>
+                </surface>
+            </collision>
+            <material>Gazebo/Grey</material>
+        </gazebo>
+        <gazebo reference="base_down_rim_r">
+            <preserveFixedJoint>1</preserveFixedJoint>
+        </gazebo>
+        <gazebo reference="t_down_rim_r">
+            <collision>
+                <surface>
+                    <bounce>
+                        <restitution_coefficient>1.0</restitution_coefficient>
+                        <threshold>0</threshold>
+                    </bounce>
+                    <friction>
+                        <!-- For Gazebo Must contain tag ode, mu, mu2, check https://github.com/osrf/sdformat/issues/31 -->
+                        <!-- https://github.com/osrf/gazebo/blob/gazebo11/gazebo/physics/bullet/BulletSurfaceParams.cc -->
+                        <ode>
+                            <mu>0.04</mu>
+                            <mu2>0.04</mu2>
+                        </ode>
+                    </friction>
+                    <contact>
+                        <ode>
+                            <max_vel>10</max_vel>
+                        </ode>
+                    </contact>
+                </surface>
+            </collision>
+            <material>Gazebo/Grey</material>
+        </gazebo>
+        <gazebo reference="base_down_rim_top">
+            <preserveFixedJoint>1</preserveFixedJoint>
+        </gazebo>
+        <gazebo reference="t_down_rim_top">
+            <collision>
+                <surface>
+                    <bounce>
+                        <restitution_coefficient>1.0</restitution_coefficient>
+                        <threshold>0</threshold>
+                    </bounce>
+                    <friction>
+                        <!-- For Gazebo Must contain tag ode, mu, mu2, check https://github.com/osrf/sdformat/issues/31 -->
+                        <!-- https://github.com/osrf/gazebo/blob/gazebo11/gazebo/physics/bullet/BulletSurfaceParams.cc -->
+                        <ode>
+                            <mu>0.04</mu>
+                            <mu2>0.04</mu2>
+                        </ode>
+                    </friction>
+                    <contact>
+                        <ode>
+                            <max_vel>10</max_vel>
+                        </ode>
+                    </contact>
+                </surface>
+            </collision>
+            <material>Gazebo/Grey</material>
+        </gazebo>
+        <gazebo reference="base_up_rim_l">
+            <preserveFixedJoint>1</preserveFixedJoint>
+        </gazebo>
+        <gazebo reference="t_up_rim_l">
+            <collision>
+                <surface>
+                    <bounce>
+                        <restitution_coefficient>1.0</restitution_coefficient>
+                        <threshold>0</threshold>
+                    </bounce>
+                    <friction>
+                        <!-- For Gazebo Must contain tag ode, mu, mu2, check https://github.com/osrf/sdformat/issues/31 -->
+                        <!-- https://github.com/osrf/gazebo/blob/gazebo11/gazebo/physics/bullet/BulletSurfaceParams.cc -->
+                        <ode>
+                            <mu>0.04</mu>
+                            <mu2>0.04</mu2>
+                        </ode>
+                    </friction>
+                    <contact>
+                        <ode>
+                            <max_vel>10</max_vel>
+                        </ode>
+                    </contact>
+                </surface>
+            </collision>
+            <material>Gazebo/Grey</material>
+        </gazebo>
+        <gazebo reference="base_up_rim_r">
+            <preserveFixedJoint>1</preserveFixedJoint>
+        </gazebo>
+        <gazebo reference="t_up_rim_r">
+            <collision>
+                <surface>
+                    <bounce>
+                        <restitution_coefficient>1.0</restitution_coefficient>
+                        <threshold>0</threshold>
+                    </bounce>
+                    <friction>
+                        <!-- For Gazebo Must contain tag ode, mu, mu2, check https://github.com/osrf/sdformat/issues/31 -->
+                        <!-- https://github.com/osrf/gazebo/blob/gazebo11/gazebo/physics/bullet/BulletSurfaceParams.cc -->
+                        <ode>
+                            <mu>0.04</mu>
+                            <mu2>0.04</mu2>
+                        </ode>
+                    </friction>
+                    <contact>
+                        <ode>
+                            <max_vel>10</max_vel>
+                        </ode>
+                    </contact>
+                </surface>
+            </collision>
+            <material>Gazebo/Grey</material>
+        </gazebo>
+        <gazebo reference="base_up_rim_top">
+            <preserveFixedJoint>1</preserveFixedJoint>
+        </gazebo>
+        <gazebo reference="t_up_rim_top">
+            <collision>
+                <surface>
+                    <bounce>
+                        <restitution_coefficient>1.0</restitution_coefficient>
+                        <threshold>0</threshold>
+                    </bounce>
+                    <friction>
+                        <!-- For Gazebo Must contain tag ode, mu, mu2, check https://github.com/osrf/sdformat/issues/31 -->
+                        <!-- https://github.com/osrf/gazebo/blob/gazebo11/gazebo/physics/bullet/BulletSurfaceParams.cc -->
+                        <ode>
+                            <mu>0.04</mu>
+                            <mu2>0.04</mu2>
+                        </ode>
+                    </friction>
+                    <contact>
+                        <ode>
+                            <max_vel>10</max_vel>
+                        </ode>
+                    </contact>
+                </surface>
+            </collision>
+            <material>Gazebo/Grey</material>
+        </gazebo>
+        <gazebo reference="base_left_rim">
+            <preserveFixedJoint>1</preserveFixedJoint>
+        </gazebo>
+        <gazebo reference="t_left_rim">
+            <collision>
+                <surface>
+                    <bounce>
+                        <restitution_coefficient>1.0</restitution_coefficient>
+                        <threshold>0</threshold>
+                    </bounce>
+                    <friction>
+                        <!-- For Gazebo Must contain tag ode, mu, mu2, check https://github.com/osrf/sdformat/issues/31 -->
+                        <!-- https://github.com/osrf/gazebo/blob/gazebo11/gazebo/physics/bullet/BulletSurfaceParams.cc -->
+                        <ode>
+                            <mu>0.04</mu>
+                            <mu2>0.04</mu2>
+                        </ode>
+                    </friction>
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
File: air_hockey_description/urdf/puck/model.urdf.xacro (robot description, xacro)
@@ -1,25 +1,22 @@
 <?xml version="1.0" encoding="utf-8"?>
-<robot xmlns:xacro="http://www.ros.org/wiki/xacro" name="air_hockey">
+<robot name="puck" xmlns:xacro="http://www.ros.org/wiki/xacro" >
     <material name="red">
         <color rgba="1.0 0.0 0.0 1"/>
     </material>
-    <xacro:arg name="puck_base_x" default="0.0"/>
-    <xacro:arg name="puck_base_y" default="0.0"/>
-    <xacro:arg name="puck_base_z" default="0.0"/>
     <xacro:property name="puck_radius" value="0.03165"/>
     <xacro:property name="puck_height" value="0.0049"/>
     <xacro:property name="restitution" value="0.8"/>
-    <xacro:property name="lateral_friction" value="0.04"/>
+    <xacro:property name="lateral_friction" value="0.02"/>
     <xacro:property name="rolling_friction" value="0.8"/>
     <xacro:property name="spinning_friction" value="0.04"/>
     <xacro:macro name="puck">
-        <link name="root">
+        <link name="base">
         </link>
         <joint name="base_joint" type="fixed">
             <origin xyz="0 0 ${puck_height/2}" rpy="0 0 0"/>
-            <parent link="root"/>
-            <child link="base"/>
+            <parent link="base"/>
+            <child link="link"/>
         </joint>
-        <link name="base">
+        <link name="link">
             <inertial>
                 <origin xyz="0 0 0.0" rpy="0 0 0"/>
@@ -32,24 +29,11 @@
                     <cylinder radius="${puck_radius}" length="${puck_height}"/>
                 </geometry>
-                <material name="red"/>
-                <material>Gazebo/Orange</material>
+                <material name="Red"/>
             </visual>
             <collision>
-                <origin xyz="0 0 0.0" rpy="0 0 0"/>
+                <origin xyz="0 0 0.05" rpy="0 0 0"/>
                 <geometry>
-                    <cylinder radius="${puck_radius}" length="${puck_height}"/>
+                    <cylinder radius="${puck_radius}" length="${puck_height + 0.1}"/>
                 </geometry>
-                <surface>
-                    <restitution_coefficient>${restitution}</restitution_coefficient>
-                    <threshold>0.01</threshold>
-                </surface>
-                <friction>
-                    <ode>
-                        <!-- For Gazebo Must contain tag ode, mu, mu2, check https://github.com/osrf/sdformat/issues/31 -->
-                        <!-- https://github.com/osrf/gazebo/blob/gazebo11/gazebo/physics/bullet/BulletSurfaceParams.cc -->
-                        <mu>${lateral_friction}</mu>
-                        <mu2>${lateral_friction}</mu2>
-                    </ode>
-                </friction>
             </collision>
             <contact>
@@ -60,8 +44,26 @@
             </contact>
         </link>
-        <gazebo reference="base">
-<!--            <mu1>${lateral_friction}</mu1>-->
-<!--            <mu2>${lateral_friction}</mu2>-->
-            <maxVel value="10.0"/>
+        <gazebo reference="link">
+            <collision>
+                <surface>
+                    <bounce>
+                        <restitution_coefficient>${restitution}</restitution_coefficient>
+                        <threshold>0.0</threshold>
+                    </bounce>
+                    <friction>
+                        <!-- For Gazebo Must contain tag ode, mu, mu2, check https://github.com/osrf/sdformat/issues/31 -->
+                        <!-- https://github.com/osrf/gazebo/blob/gazebo11/gazebo/physics/bullet/BulletSurfaceParams.cc -->
+                        <ode>
+                            <mu>${lateral_friction}</mu>
+                            <mu2>${lateral_friction}</mu2>
+                        </ode>
+                    </friction>
+                    <contact>
+                        <ode>
+                            <max_vel>100</max_vel>
+                        </ode>
+                    </contact>
+                </surface>
+            </collision>
             <material>Gazebo/Red</material>
         </gazebo>
