Commit message: Use urdf.xacro to launch the description

File: air_hockey_description/urdf/striker.xacro (robot description, xacro)
@@ -21,5 +21,5 @@
                     <mesh filename="package://air_hockey_description/meshes/striker/visual/EE_arm.stl"/>
                 </geometry>
-                <material name="White"/>
+                <material name="LightGrey"/>
             </visual>
             <collision>
@@ -28,5 +28,4 @@
                     <mesh filename="package://air_hockey_description/meshes/striker/collision/EE_arm_collision.stl"/>
                 </geometry>
-                <material name="White"/>
             </collision>
         </link>
@@ -39,5 +38,5 @@
             <safety_controller k_position="100" k_velocity="2" soft_lower_limit="-2.094395102"
                                soft_upper_limit="2.094395102"/>
-            <dynamics damping="0.1"/>
+            <dynamics damping="0.3"/>
         </joint>
         <link name="${robot_name}_striker_joint_link">
@@ -45,24 +44,7 @@
                 <origin xyz="0 0.0 0" rpy="0 0 0"/>
                 <mass value="0.01"/>
-<!--                <inertia-->
-<!--                        ixx="0.0001" ixy="0.0" ixz="0.0"-->
-<!--                        iyy="0.0001" iyz="0.000000" izz="0.00001"/>-->
                 <inertia ixx="0.01" ixy="0.0" ixz="0.0"
                          iyy="0.01" iyz="0.0" izz="0.01"/>
             </inertial>
-<!--            <visual>-->
-<!--                <origin xyz="0 0 0" rpy="0 0.0 0"/>-->
-<!--                <geometry>-->
-<!--                    <mesh filename="package://air_hockey_description/meshes/striker/visual/EE_joint.stl"/>-->
-<!--                </geometry>-->
-<!--                <material name="White"/>-->
-<!--            </visual>-->
-<!--            <collision>-->
-<!--                <origin xyz="0 0 0" rpy="0 0 0"/>-->
-<!--                <geometry>-->
-<!--                    <mesh filename="package://air_hockey_description/meshes/striker/collision/EE_joint_collision.stl"/>-->
-<!--                </geometry>-->
-<!--                <material name="White"/>-->
-<!--            </collision>-->
         </link>
         <joint name="${robot_name}_striker_joint_2" type="revolute">
@@ -74,7 +56,6 @@
             <safety_controller k_position="100" k_velocity="2" soft_lower_limit="-2.094395102"
                                soft_upper_limit="2.094395102"/>
-            <dynamics damping="0.1"/>
+            <dynamics damping="0.3"/>
         </joint>
-        <!--  The striker frame is here defined -->
         <link name="${robot_name}_striker_mallet">
             <inertial>
@@ -92,5 +73,5 @@
                     <mesh filename="package://air_hockey_description/meshes/striker/visual/EE_mallet.stl"/>
                 </geometry>
-                <material name="White"/>
+                <material name="LightGrey"/>
             </visual>
             <collision>
@@ -99,15 +80,4 @@
                     <mesh filename="package://air_hockey_description/meshes/striker/collision/EE_mallet_collision.stl"/>
                 </geometry>
-                <material name="White"/>
-                <surface>
-                    <bounce restitution_coefficient="1.0" threshold="0.01"/>
-                    <contact>
-                        <ode>
-                            <soft_cfm>0.1</soft_cfm>
-                            <soft_erp>0.1</soft_erp>
-                            <max_vel>1</max_vel>
-                        </ode>
-                    </contact>
-                </surface>
             </collision>
         </link>
@@ -118,4 +88,5 @@
             <axis xyz="1 0 0"/>
         </joint>
+        <!--  The striker frame is here defined -->
         <link name="${robot_name}_striker_mallet_tip">
             <inertial>
@@ -142,14 +113,24 @@
         </gazebo>
         <gazebo reference="${robot_name}_striker_mallet">
+            <collision>
+                <surface>
+                    <bounce>
+                        <restitution_coefficient>1.0</restitution_coefficient>
+                        <threshold>0.0</threshold>
+                    </bounce>
+                    <contact>
+                        <ode>
+                            <max_vel>100</max_vel>
+                        </ode>
+                    </contact>
+                </surface>
+            </collision>
             <material>Gazebo/Grey</material>
-            <mu1>0.2</mu1>
-            <mu2>0.2</mu2>
+            <mu1>1.0</mu1>
+            <mu2>1.0</mu2>
             <selfCollide>0</selfCollide>
         </gazebo>
-        <gazebo reference="${robot_name}_striker_mallet_tip">
-            <material>Gazebo/Grey</material>
-            <mu1>0.2</mu1>
-            <mu2>0.2</mu2>
-            <selfCollide>0</selfCollide>
+        <gazebo reference="${robot_name}_striker_mallet_fix">
+            <preserveFixedJoint>1</preserveFixedJoint>
         </gazebo>
         <transmission name="${robot_name}_striker_tran_1">

Commit message: Add static tf publisher of table, remove collision model of undesired edge

File: air_hockey_description/urdf/air_hockey_table/model.urdf.xacro (robot description, xacro)
@@ -139,9 +139,9 @@
                 <material name="grey"/>
             </visual>
-            <collision>
-                <geometry>
-                    <box size="${table_rim_horizon_length} ${table_base_width - 2 * table_rim_vertical_width} ${table_rim_horizon_top_height}"/>
-                </geometry>
-            </collision>
+<!--            <collision>-->
+<!--                <geometry>-->
+<!--                    <box size="${table_rim_horizon_length} ${table_base_width - 2 * table_rim_vertical_width} ${table_rim_horizon_top_height}"/>-->
+<!--                </geometry>-->
+<!--            </collision>-->
             <contact>
                 <restitution value="1.0"/>
@@ -387,25 +387,25 @@
         </gazebo>
         <gazebo reference="t_down_rim_top">
-            <collision>
-                <surface>
-                    <bounce>
-                        <restitution_coefficient>1.0</restitution_coefficient>
-                        <threshold>0</threshold>
-                    </bounce>
-                    <friction>
-                        <!-- For Gazebo Must contain tag ode, mu, mu2, check https://github.com/osrf/sdformat/issues/31 -->
-                        <!-- https://github.com/osrf/gazebo/blob/gazebo11/gazebo/physics/bullet/BulletSurfaceParams.cc -->
-                        <ode>
-                            <mu>0.04</mu>
-                            <mu2>0.04</mu2>
-                        </ode>
-                    </friction>
-                    <contact>
-                        <ode>
-                            <max_vel>10</max_vel>
-                        </ode>
-                    </contact>
-                </surface>
-            </collision>
+<!--            <collision>-->
+<!--                <surface>-->
+<!--                    <bounce>-->
+<!--                        <restitution_coefficient>1.0</restitution_coefficient>-->
+<!--                        <threshold>0</threshold>-->
+<!--                    </bounce>-->
+<!--                    <friction>-->
+<!--                        &lt;!&ndash; For Gazebo Must contain tag ode, mu, mu2, check https://github.com/osrf/sdformat/issues/31 &ndash;&gt;-->
+<!--                        &lt;!&ndash; https://github.com/osrf/gazebo/blob/gazebo11/gazebo/physics/bullet/BulletSurfaceParams.cc &ndash;&gt;-->
+<!--                        <ode>-->
+<!--                            <mu>0.04</mu>-->
+<!--                            <mu2>0.04</mu2>-->
+<!--                        </ode>-->
+<!--                    </friction>-->
+<!--                    <contact>-->
+<!--                        <ode>-->
+<!--                            <max_vel>10</max_vel>-->
+<!--                        </ode>-->
+<!--                    </contact>-->
+<!--                </surface>-->
+<!--            </collision>-->
             <material>Gazebo/Grey</material>
         </gazebo>
@@ -468,25 +468,25 @@
         </gazebo>
         <gazebo reference="t_up_rim_top">
-            <collision>
-                <surface>
-                    <bounce>
-                        <restitution_coefficient>1.0</restitution_coefficient>
-                        <threshold>0</threshold>
-                    </bounce>
-                    <friction>
-                        <!-- For Gazebo Must contain tag ode, mu, mu2, check https://github.com/osrf/sdformat/issues/31 -->
-                        <!-- https://github.com/osrf/gazebo/blob/gazebo11/gazebo/physics/bullet/BulletSurfaceParams.cc -->
-                        <ode>
-                            <mu>0.04</mu>
-                            <mu2>0.04</mu2>
-                        </ode>
-                    </friction>
-                    <contact>
-                        <ode>
-                            <max_vel>10</max_vel>
-                        </ode>
-                    </contact>
-                </surface>
-            </collision>
+<!--            <collision>-->
+<!--                <surface>-->
+<!--                    <bounce>-->
+<!--                        <restitution_coefficient>1.0</restitution_coefficient>-->
+<!--                        <threshold>0</threshold>-->
+<!--                    </bounce>-->
+<!--                    <friction>-->
+<!--                        &lt;!&ndash; For Gazebo Must contain tag ode, mu, mu2, check https://github.com/osrf/sdformat/issues/31 &ndash;&gt;-->
+<!--                        &lt;!&ndash; https://github.com/osrf/gazebo/blob/gazebo11/gazebo/physics/bullet/BulletSurfaceParams.cc &ndash;&gt;-->
+<!--                        <ode>-->
+<!--                            <mu>0.04</mu>-->
+<!--                            <mu2>0.04</mu2>-->
+<!--                        </ode>-->
+<!--                    </friction>-->
+<!--                    <contact>-->
+<!--                        <ode>-->
+<!--                            <max_vel>10</max_vel>-->
+<!--                        </ode>-->
+<!--                    </contact>-->
+<!--                </surface>-->
+<!--            </collision>-->
             <material>Gazebo/Grey</material>
         </gazebo>

Commit message: Add bringup launch file
- refactor the urdf xacro: now the table and puck model is aligned with tf

File: air_hockey_description/urdf/air_hockey_table/model.urdf.xacro (robot description, xacro)
@@ -10,7 +10,5 @@
         <color rgba="1.0 0.0 0.0 1"/>
     </material>
-    <xacro:arg name="table_surface_x" default="0.0"/>
-    <xacro:arg name="table_surface_y" default="0.0"/>
-    <xacro:arg name="table_surface_z" default="0.0"/>
+    <xacro:arg name="parent" default="world"/>
     <xacro:property name="table_base_length" value="2.14"/>
     <xacro:property name="table_base_width" value="1.22"/>
@@ -23,9 +21,9 @@
     <xacro:property name="table_rim_vertical_width" value="0.09"/>
     <xacro:property name="table_rim_vertical_height" value="0.03"/>
-    <xacro:macro name="air_hockey_table" params="surface_x surface_y surface_z">
-        <link name="world"/>
+    <xacro:macro name="air_hockey_table" params="parent">
+        <link name="${parent}"/>
         <joint name="base_joint" type="fixed">
-            <origin xyz="${surface_x} ${surface_y} ${surface_z - table_base_height/2}" rpy="0 0 0"/>
-            <parent link="world"/>
+            <origin xyz="0 0 ${-table_base_height/2}" rpy="0 0 0"/>
+            <parent link="${parent}"/>
             <child link="t_base"/>
         </joint>
@@ -545,6 +543,8 @@
             <material>Gazebo/Grey</material>
         </gazebo>
-        <static>1</static>
+        <gazebo>
+            <static>true</static>
+        </gazebo>
     </xacro:macro>
-    <xacro:air_hockey_table surface_x="$(arg table_surface_x)" surface_y="$(arg table_surface_y)" surface_z="$(arg table_surface_z)"/>
+    <xacro:air_hockey_table parent="$(arg parent)"/>
 </robot>

File: air_hockey_description/urdf/puck/model.urdf.xacro (robot description, xacro)
@@ -4,4 +4,5 @@
         <color rgba="1.0 0.0 0.0 1"/>
     </material>
+    <xacro:arg name="parent" default="world"/>
     <xacro:property name="puck_radius" value="0.03165"/>
     <xacro:property name="puck_height" value="0.0049"/>
@@ -10,10 +11,9 @@
     <xacro:property name="rolling_friction" value="0.8"/>
     <xacro:property name="spinning_friction" value="0.04"/>
-    <xacro:macro name="puck">
-        <link name="base">
-        </link>
+    <xacro:macro name="puck" params="parent">
+        <link name="${parent}"/>
         <joint name="base_joint" type="fixed">
             <origin xyz="0 0 ${puck_height/2}" rpy="0 0 0"/>
-            <parent link="base"/>
+            <parent link="${parent}"/>
             <child link="link"/>
         </joint>
@@ -73,4 +73,4 @@
         </gazebo>
     </xacro:macro>
-    <xacro:puck/>
+    <xacro:puck parent="$(arg parent)"/>
 </robot>

Commit message: Add reference frame of Home and Away
- Puck tracker based on the player perspective frame

File: air_hockey_description/urdf/air_hockey_table/model.urdf.xacro (robot description, xacro)
@@ -11,4 +11,5 @@
     </material>
     <xacro:arg name="parent" default="world"/>
+    <xacro:property name="M_PI" value="3.1415926535897931"/>
     <xacro:property name="table_base_length" value="2.14"/>
     <xacro:property name="table_base_width" value="1.22"/>
@@ -54,4 +55,16 @@
             </contact>
         </link>
+        <joint name="base_home_joint" type="fixed">
+            <origin xyz="-${table_base_length / 2 - table_rim_horizon_length} 0 0" rpy="0 0 0"/>
+            <parent link="${parent}"/>
+            <child link="TableHome"/>
+        </joint>
+        <link name="TableHome"/>
+        <joint name="base_away_joint" type="fixed">
+            <origin xyz="${table_base_length / 2 - table_rim_horizon_length} 0 0" rpy="0 0 ${M_PI}"/>
+            <parent link="${parent}"/>
+            <child link="TableAway"/>
+        </joint>
+        <link name="TableAway"/>
         <joint name="base_down_rim_l" type="fixed">
             <origin rpy="0.0 0.0 0.0" xyz="${(table_base_length - table_rim_horizon_length) / 2}

Commit message: Change the parameter of table dimensions
- add option of controller
- increase the motion time for safety

File: air_hockey_description/urdf/air_hockey_table/model.urdf.xacro (robot description, xacro)
@@ -12,12 +12,12 @@
     <xacro:arg name="parent" default="world"/>
     <xacro:property name="M_PI" value="3.1415926535897931"/>
-    <xacro:property name="table_base_length" value="2.14"/>
-    <xacro:property name="table_base_width" value="1.22"/>
+    <xacro:property name="table_base_length" value="2.136"/>
+    <xacro:property name="table_base_width" value="1.222"/>
     <xacro:property name="table_base_height" value="0.11"/>
     <xacro:property name="table_rim_horizon_length" value="0.09"/>
-    <xacro:property name="table_rim_horizon_width" value="0.395"/>
+    <xacro:property name="table_rim_horizon_width" value="0.396"/>
     <xacro:property name="table_rim_horizon_height" value="0.01"/>
     <xacro:property name="table_rim_horizon_top_height" value="0.02"/>
-    <xacro:property name="table_rim_vertical_length" value="2.14"/>
+    <xacro:property name="table_rim_vertical_length" value="2.136"/>
     <xacro:property name="table_rim_vertical_width" value="0.09"/>
     <xacro:property name="table_rim_vertical_height" value="0.03"/>

Commit message: Add collision bitmask

File: air_hockey_description/urdf/air_hockey_table/model.urdf.xacro (robot description, xacro)
@@ -22,4 +22,5 @@
     <xacro:property name="table_rim_vertical_width" value="0.09"/>
     <xacro:property name="table_rim_vertical_height" value="0.03"/>
+    <xacro:property name="collide_bitmask" value="0x01"/>
     <xacro:macro name="air_hockey_table" params="parent">
         <link name="${parent}"/>
@@ -332,4 +333,5 @@
                     </friction>
                     <contact>
+                        <collide_bitmask>0x01</collide_bitmask>
                         <ode>
                             <max_vel>10</max_vel>
@@ -359,4 +361,5 @@
                     </friction>
                     <contact>
+                        <collide_bitmask>0x01</collide_bitmask>
                         <ode>
                             <max_vel>10</max_vel>
@@ -386,4 +389,5 @@
                     </friction>
                     <contact>
+                        <collide_bitmask>0x01</collide_bitmask>
                         <ode>
                             <max_vel>10</max_vel>
@@ -440,4 +444,5 @@
                     </friction>
                     <contact>
+                        <collide_bitmask>0x01</collide_bitmask>
                         <ode>
                             <max_vel>10</max_vel>
@@ -467,4 +472,5 @@
                     </friction>
                     <contact>
+                        <collide_bitmask>0x01</collide_bitmask>
                         <ode>
                             <max_vel>10</max_vel>
@@ -521,4 +527,5 @@
                     </friction>
                     <contact>
+                        <collide_bitmask>0x01</collide_bitmask>
                         <ode>
                             <max_vel>10</max_vel>
@@ -548,4 +555,5 @@
                     </friction>
                     <contact>
+                        <collide_bitmask>0x01</collide_bitmask>
                         <ode>
                             <max_vel>10</max_vel>

File: air_hockey_description/urdf/puck/model.urdf.xacro (robot description, xacro)
@@ -63,4 +63,5 @@
                     </friction>
                     <contact>
+                        <collide_bitmask>0x03</collide_bitmask>
                         <ode>
                             <kp>1e9</kp>

File: air_hockey_description/urdf/striker.xacro (robot description, xacro)
@@ -115,4 +115,5 @@
                     </bounce>
                     <contact>
+                        <collide_bitmask>0x02</collide_bitmask>
                         <ode>
                             <kp>1e9</kp>
