Commit message: Add arguments for puck collision model
- collision model name should same as parent's name

File: air_hockey_description/urdf/air_hockey_table/model.urdf.xacro (robot description, xacro)
@@ -11,4 +11,5 @@
     </material>
     <xacro:arg name="parent" default="world"/>
+    <xacro:arg name="collide_bitmask" default="0x01"/>
     <xacro:property name="M_PI" value="3.1415926535897931"/>
     <xacro:property name="table_base_length" value="2.136"/>
@@ -22,6 +23,5 @@
     <xacro:property name="table_rim_vertical_width" value="0.09"/>
     <xacro:property name="table_rim_vertical_height" value="0.03"/>
-    <xacro:property name="collide_bitmask" value="0x01"/>
-    <xacro:macro name="air_hockey_table" params="parent">
+    <xacro:macro name="air_hockey_table" params="parent collide_bitmask">
         <link name="${parent}"/>
         <joint name="base_joint" type="fixed">
@@ -333,5 +333,5 @@
                     </friction>
                     <contact>
-                        <collide_bitmask>0x01</collide_bitmask>
+                        <collide_bitmask>${collide_bitmask}</collide_bitmask>
                         <ode>
                             <max_vel>10</max_vel>
@@ -361,5 +361,5 @@
                     </friction>
                     <contact>
-                        <collide_bitmask>0x01</collide_bitmask>
+                        <collide_bitmask>${collide_bitmask}</collide_bitmask>
                         <ode>
                             <max_vel>10</max_vel>
@@ -389,5 +389,5 @@
                     </friction>
                     <contact>
-                        <collide_bitmask>0x01</collide_bitmask>
+                        <collide_bitmask>${collide_bitmask}</collide_bitmask>
                         <ode>
                             <max_vel>10</max_vel>
@@ -444,5 +444,5 @@
                     </friction>
                     <contact>
-                        <collide_bitmask>0x01</collide_bitmask>
+                        <collide_bitmask>${collide_bitmask}</collide_bitmask>
                         <ode>
                             <max_vel>10</max_vel>
@@ -472,5 +472,5 @@
                     </friction>
                     <contact>
-                        <collide_bitmask>0x01</collide_bitmask>
+                        <collide_bitmask>${collide_bitmask}</collide_bitmask>
                         <ode>
                             <max_vel>10</max_vel>
@@ -527,5 +527,5 @@
                     </friction>
                     <contact>
-                        <collide_bitmask>0x01</collide_bitmask>
+                        <collide_bitmask>${collide_bitmask}</collide_bitmask>
                         <ode>
                             <max_vel>10</max_vel>
@@ -555,5 +555,5 @@
                     </friction>
                     <contact>
-                        <collide_bitmask>0x01</collide_bitmask>
+                        <collide_bitmask>${collide_bitmask}</collide_bitmask>
                         <ode>
                             <max_vel>10</max_vel>
@@ -568,4 +568,4 @@
         </gazebo>
     </xacro:macro>
-    <xacro:air_hockey_table parent="$(arg parent)"/>
+    <xacro:air_hockey_table parent="$(arg parent)" collide_bitmask="$(arg collide_bitmask)"/>
 </robot>

File: air_hockey_description/urdf/puck/model.urdf (robot description, URDF)
Before this commit: robot puck, 2 links, 1 joints
Links:
- removed link link
- removed link world
- added link Puck
- added link Puck_link, mass 0.01; collision cylinder length=0.0049 radius=0.03165; visual cylinder length=0.0049 radius=0.03165
Joints:
- removed joint base_joint
- added joint {puck_name}_joint: type fixed, parent Puck, child Puck_link, origin xyz=0 0 0.00245 rpy=0 0 0

File: air_hockey_description/urdf/puck/model.urdf.xacro (robot description, xacro)
@@ -1,8 +1,17 @@
 <?xml version="1.0" encoding="utf-8"?>
 <robot name="puck" xmlns:xacro="http://www.ros.org/wiki/xacro" >
-    <material name="red">
+    <material name="Red">
         <color rgba="1.0 0.0 0.0 1"/>
     </material>
-    <xacro:arg name="parent" default="world"/>
+    <material name="Green">
+        <color rgba="0.0 1.0 0.0 1"/>
+    </material>
+    <material name="Blue">
+        <color rgba="0.0 0.0 1.0 1"/>
+    </material>
+    <xacro:arg name="puck_name" default="Puck"/>
+    <xacro:arg name="parent" default="Puck"/>
+    <xacro:arg name="color" default="Red"/>
+    <xacro:arg name="collide_bitmask" default="0x03"/>
     <xacro:property name="puck_radius" value="0.03165"/>
     <xacro:property name="puck_height" value="0.0049"/>
@@ -11,12 +20,12 @@
     <xacro:property name="rolling_friction" value="0.8"/>
     <xacro:property name="spinning_friction" value="0.04"/>
-    <xacro:macro name="puck" params="parent">
+    <xacro:macro name="puck" params="puck_name parent color collide_bitmask">
         <link name="${parent}"/>
-        <joint name="base_joint" type="fixed">
+        <joint name="{puck_name}_joint" type="fixed">
             <origin xyz="0 0 ${puck_height/2}" rpy="0 0 0"/>
             <parent link="${parent}"/>
-            <child link="link"/>
+            <child link="${puck_name}_link"/>
         </joint>
-        <link name="link">
+        <link name="${puck_name}_link">
             <inertial>
                 <origin xyz="0 0 0.0" rpy="0 0 0"/>
@@ -29,5 +38,5 @@
                     <cylinder radius="${puck_radius}" length="${puck_height}"/>
                 </geometry>
-                <material name="red"/>
+                <material name="${color}"/>
             </visual>
             <collision>
@@ -44,5 +53,5 @@
             </contact>
         </link>
-        <gazebo reference="link">
+        <gazebo reference="${parent}">
             <collision>
                 <surface>
@@ -63,5 +72,5 @@
                     </friction>
                     <contact>
-                        <collide_bitmask>0x03</collide_bitmask>
+                        <collide_bitmask>${collide_bitmask}</collide_bitmask>
                         <ode>
                             <kp>1e9</kp>
@@ -79,4 +88,4 @@
         </gazebo>
     </xacro:macro>
-    <xacro:puck parent="$(arg parent)"/>
+    <xacro:puck puck_name="$(arg puck_name)" parent="$(arg parent)" collide_bitmask="$(arg collide_bitmask)" color="$(arg color)"/>
 </robot>

Commit message: Add argument for physics paramter

File: air_hockey_description/urdf/air_hockey_table/model.urdf.xacro (robot description, xacro)
@@ -12,4 +12,5 @@
     <xacro:arg name="parent" default="world"/>
     <xacro:arg name="collide_bitmask" default="0x01"/>
+    <xacro:arg name="restitution" default="1.0"/>
     <xacro:property name="M_PI" value="3.1415926535897931"/>
     <xacro:property name="table_base_length" value="2.136"/>
@@ -23,5 +24,5 @@
     <xacro:property name="table_rim_vertical_width" value="0.09"/>
     <xacro:property name="table_rim_vertical_height" value="0.03"/>
-    <xacro:macro name="air_hockey_table" params="parent collide_bitmask">
+    <xacro:macro name="air_hockey_table" params="parent collide_bitmask restitution">
         <link name="${parent}"/>
         <joint name="base_joint" type="fixed">
@@ -50,5 +51,5 @@
             </collision>
             <contact>
-                <restitution value="1.0"/>
+                <restitution value="${restitution}"/>
                 <lateral_friction value="1.0"/>
                 <rolling_friction value="0.0"/>
@@ -94,5 +95,5 @@
             </collision>
             <contact>
-                <restitution value="1.0"/>
+                <restitution value="${restitution}"/>
                 <lateral_friction value="0.0"/>
                 <rolling_friction value="0.0"/>
@@ -126,5 +127,5 @@
             </collision>
             <contact>
-                <restitution value="1.0"/>
+                <restitution value="${restitution}"/>
                 <lateral_friction value="0.0"/>
                 <rolling_friction value="0.0"/>
@@ -157,5 +158,5 @@
 <!--            </collision>-->
             <contact>
-                <restitution value="1.0"/>
+                <restitution value="${restitution}"/>
                 <lateral_friction value="0.0"/>
                 <rolling_friction value="0.0"/>
@@ -189,5 +190,5 @@
             </collision>
             <contact>
-                <restitution value="1.0"/>
+                <restitution value="${restitution}"/>
                 <lateral_friction value="0.0"/>
                 <rolling_friction value="0.0"/>
@@ -221,5 +222,5 @@
             </collision>
             <contact>
-                <restitution value="1.0"/>
+                <restitution value="${restitution}"/>
                 <lateral_friction value="0.0"/>
                 <rolling_friction value="0.0"/>
@@ -247,5 +248,5 @@
             </visual>
             <contact>
-                <restitution value="1.0"/>
+                <restitution value="${restitution}"/>
                 <lateral_friction value="0.0"/>
                 <rolling_friction value="0.0"/>
@@ -279,5 +280,5 @@
             </collision>
             <contact>
-                <restitution value="1.0"/>
+                <restitution value="${restitution}"/>
                 <lateral_friction value="0.0"/>
                 <rolling_friction value="0.0"/>
@@ -311,5 +312,5 @@
             </collision>
             <contact>
-                <restitution value="1.0"/>
+                <restitution value="${restitution}"/>
                 <lateral_friction value="0.0"/>
                 <rolling_friction value="0.0"/>
@@ -321,5 +322,5 @@
                 <surface>
                     <bounce>
-                        <restitution_coefficient>1.0</restitution_coefficient>
+                        <restitution_coefficient>${restitution}</restitution_coefficient>
                         <threshold>0</threshold>
                     </bounce>
@@ -349,5 +350,5 @@
                 <surface>
                     <bounce>
-                        <restitution_coefficient>1.0</restitution_coefficient>
+                        <restitution_coefficient>${restitution}</restitution_coefficient>
                         <threshold>0</threshold>
                     </bounce>
@@ -377,5 +378,5 @@
                 <surface>
                     <bounce>
-                        <restitution_coefficient>1.0</restitution_coefficient>
+                        <restitution_coefficient>${restitution}</restitution_coefficient>
                         <threshold>0</threshold>
                     </bounce>
@@ -405,5 +406,5 @@
 <!--                <surface>-->
 <!--                    <bounce>-->
-<!--                        <restitution_coefficient>1.0</restitution_coefficient>-->
+<!--                        <restitution_coefficient>${restitution}</restitution_coefficient>-->
 <!--                        <threshold>0</threshold>-->
 <!--                    </bounce>-->
@@ -432,5 +433,5 @@
                 <surface>
                     <bounce>
-                        <restitution_coefficient>1.0</restitution_coefficient>
+                        <restitution_coefficient>${restitution}</restitution_coefficient>
                         <threshold>0</threshold>
                     </bounce>
@@ -460,5 +461,5 @@
                 <surface>
                     <bounce>
-                        <restitution_coefficient>1.0</restitution_coefficient>
+                        <restitution_coefficient>${restitution}</restitution_coefficient>
                         <threshold>0</threshold>
                     </bounce>
@@ -488,5 +489,5 @@
 <!--                <surface>-->
 <!--                    <bounce>-->
-<!--                        <restitution_coefficient>1.0</restitution_coefficient>-->
+<!--                        <restitution_coefficient>${restitution}</restitution_coefficient>-->
 <!--                        <threshold>0</threshold>-->
 <!--                    </bounce>-->
@@ -515,5 +516,5 @@
                 <surface>
                     <bounce>
-                        <restitution_coefficient>1.0</restitution_coefficient>
+                        <restitution_coefficient>${restitution}</restitution_coefficient>
                         <threshold>0</threshold>
                     </bounce>
@@ -543,5 +544,5 @@
                 <surface>
                     <bounce>
-                        <restitution_coefficient>1.0</restitution_coefficient>
+                        <restitution_coefficient>${restitution}</restitution_coefficient>
                         <threshold>0</threshold>
                     </bounce>
@@ -568,4 +569,6 @@
         </gazebo>
     </xacro:macro>
-    <xacro:air_hockey_table parent="$(arg parent)" collide_bitmask="$(arg collide_bitmask)"/>
+    <xacro:air_hockey_table parent="$(arg parent)"
+                            collide_bitmask="$(arg collide_bitmask)"
+                            restitution="$(arg restitution)"/>
 </robot>

File: air_hockey_description/urdf/puck/model.urdf.xacro (robot description, xacro)
@@ -11,18 +11,17 @@
     </material>
     <xacro:arg name="puck_name" default="Puck"/>
-    <xacro:arg name="parent" default="Puck"/>
     <xacro:arg name="color" default="Red"/>
     <xacro:arg name="collide_bitmask" default="0x03"/>
+    <xacro:arg name="restitution" default="0.8"/>
+    <xacro:arg name="lateral_friction" default="0.02"/>
+    <xacro:arg name="rolling_friction" default="0.8"/>
+    <xacro:arg name="spinning_friction" default="0.04"/>
     <xacro:property name="puck_radius" value="0.03165"/>
     <xacro:property name="puck_height" value="0.0049"/>
-    <xacro:property name="restitution" value="0.8"/>
-    <xacro:property name="lateral_friction" value="0.02"/>
-    <xacro:property name="rolling_friction" value="0.8"/>
-    <xacro:property name="spinning_friction" value="0.04"/>
-    <xacro:macro name="puck" params="puck_name parent color collide_bitmask">
-        <link name="${parent}"/>
+    <xacro:macro name="puck" params="puck_name color collide_bitmask restitution lateral_friction rolling_friction spinning_friction">
+        <link name="${puck_name}"/>
         <joint name="{puck_name}_joint" type="fixed">
             <origin xyz="0 0 ${puck_height/2}" rpy="0 0 0"/>
-            <parent link="${parent}"/>
+            <parent link="${puck_name}"/>
             <child link="${puck_name}_link"/>
         </joint>
@@ -47,11 +46,11 @@
             </collision>
             <contact>
-                <restitution value="${restitution}"/>
+                <restitution value="$(arg restitution)"/>
                 <lateral_friction value="${lateral_friction}"/>
                 <rolling_friction value="0.0"/>
-                <spinning_friction value="0.02"/>
+                <spinning_friction value="${spinning_friction}"/>
             </contact>
         </link>
-        <gazebo reference="${parent}">
+        <gazebo reference="${puck_name}">
             <collision>
                 <surface>
@@ -64,4 +63,6 @@
                         <!-- https://github.com/osrf/gazebo/blob/gazebo11/gazebo/physics/bullet/BulletSurfaceParams.cc -->
                         <torsional>
+                            <coefficient>${spinning_friction}</coefficient>
+                            <use_patch_radius>false</use_patch_radius>
                             <surface_radius>${puck_radius}</surface_radius>
                         </torsional>
@@ -88,4 +89,10 @@
         </gazebo>
     </xacro:macro>
-    <xacro:puck puck_name="$(arg puck_name)" parent="$(arg parent)" collide_bitmask="$(arg collide_bitmask)" color="$(arg color)"/>
+    <xacro:puck puck_name="$(arg puck_name)"
+                collide_bitmask="$(arg collide_bitmask)"
+                color="$(arg color)"
+                restitution="$(arg restitution)"
+                lateral_friction="$(arg lateral_friction)"
+                rolling_friction="$(arg rolling_friction)"
+                spinning_friction="$(arg spinning_friction)"/>
 </robot>
