Commit message: Add arugments of physics parameter in xacro

File: air_hockey_description/urdf/air_hockey_table/model.urdf.xacro (robot description, xacro)
@@ -12,5 +12,8 @@
     <xacro:arg name="parent" default="world"/>
     <xacro:arg name="collide_bitmask" default="0x01"/>
-    <xacro:arg name="restitution" default="1.0"/>
+    <xacro:arg name="restitution" default="0.68"/>
+    <xacro:arg name="lateral_friction" default="1.0"/>
+    <xacro:arg name="rolling_friction" default="1.0"/>
+    <xacro:arg name="spinning_friction" default="1.0"/>
     <xacro:property name="M_PI" value="3.1415926535897931"/>
     <xacro:property name="table_base_length" value="2.136"/>
@@ -24,5 +27,6 @@
     <xacro:property name="table_rim_vertical_width" value="0.09"/>
     <xacro:property name="table_rim_vertical_height" value="0.03"/>
-    <xacro:macro name="air_hockey_table" params="parent collide_bitmask restitution">
+    <xacro:macro name="air_hockey_table" params="parent collide_bitmask restitution
+                                                 lateral_friction rolling_friction spinning_friction">
         <link name="${parent}"/>
         <joint name="base_joint" type="fixed">
@@ -329,6 +333,6 @@
                         <!-- https://github.com/osrf/gazebo/blob/gazebo11/gazebo/physics/bullet/BulletSurfaceParams.cc -->
                         <ode>
-                            <mu>0.04</mu>
-                            <mu2>0.04</mu2>
+                            <mu>${lateral_friction}</mu>
+                            <mu2>${lateral_friction}</mu2>
                         </ode>
                     </friction>
@@ -357,6 +361,6 @@
                         <!-- https://github.com/osrf/gazebo/blob/gazebo11/gazebo/physics/bullet/BulletSurfaceParams.cc -->
                         <ode>
-                            <mu>0.04</mu>
-                            <mu2>0.04</mu2>
+                            <mu>${lateral_friction}</mu>
+                            <mu2>${lateral_friction}</mu2>
                         </ode>
                     </friction>
@@ -385,6 +389,6 @@
                         <!-- https://github.com/osrf/gazebo/blob/gazebo11/gazebo/physics/bullet/BulletSurfaceParams.cc -->
                         <ode>
-                            <mu>0.04</mu>
-                            <mu2>0.04</mu2>
+                            <mu>${lateral_friction}</mu>
+                            <mu2>${lateral_friction}</mu2>
                         </ode>
                     </friction>
@@ -413,6 +417,6 @@
 <!--                        &lt;!&ndash; https://github.com/osrf/gazebo/blob/gazebo11/gazebo/physics/bullet/BulletSurfaceParams.cc &ndash;&gt;-->
 <!--                        <ode>-->
-<!--                            <mu>0.04</mu>-->
-<!--                            <mu2>0.04</mu2>-->
+<!--                            <mu>${lateral_friction}</mu>-->
+<!--                            <mu2>${lateral_friction}</mu2>-->
 <!--                        </ode>-->
 <!--                    </friction>-->
@@ -440,6 +444,6 @@
                         <!-- https://github.com/osrf/gazebo/blob/gazebo11/gazebo/physics/bullet/BulletSurfaceParams.cc -->
                         <ode>
-                            <mu>0.04</mu>
-                            <mu2>0.04</mu2>
+                            <mu>${lateral_friction}</mu>
+                            <mu2>${lateral_friction}</mu2>
                         </ode>
                     </friction>
@@ -468,6 +472,6 @@
                         <!-- https://github.com/osrf/gazebo/blob/gazebo11/gazebo/physics/bullet/BulletSurfaceParams.cc -->
                         <ode>
-                            <mu>0.04</mu>
-                            <mu2>0.04</mu2>
+                            <mu>${lateral_friction}</mu>
+                            <mu2>${lateral_friction}</mu2>
                         </ode>
                     </friction>
@@ -496,6 +500,6 @@
 <!--                        &lt;!&ndash; https://github.com/osrf/gazebo/blob/gazebo11/gazebo/physics/bullet/BulletSurfaceParams.cc &ndash;&gt;-->
 <!--                        <ode>-->
-<!--                            <mu>0.04</mu>-->
-<!--                            <mu2>0.04</mu2>-->
+<!--                            <mu>${lateral_friction}</mu>-->
+<!--                            <mu2>${lateral_friction}</mu2>-->
 <!--                        </ode>-->
 <!--                    </friction>-->
@@ -523,6 +527,6 @@
                         <!-- https://github.com/osrf/gazebo/blob/gazebo11/gazebo/physics/bullet/BulletSurfaceParams.cc -->
                         <ode>
-                            <mu>0.04</mu>
-                            <mu2>0.04</mu2>
+                            <mu>${lateral_friction}</mu>
+                            <mu2>${lateral_friction}</mu2>
                         </ode>
                     </friction>
@@ -551,6 +555,6 @@
                         <!-- https://github.com/osrf/gazebo/blob/gazebo11/gazebo/physics/bullet/BulletSurfaceParams.cc -->
                         <ode>
-                            <mu>0.04</mu>
-                            <mu2>0.04</mu2>
+                            <mu>${lateral_friction}</mu>
+                            <mu2>${lateral_friction}</mu2>
                         </ode>
                     </friction>
@@ -571,4 +575,7 @@
     <xacro:air_hockey_table parent="$(arg parent)"
                             collide_bitmask="$(arg collide_bitmask)"
-                            restitution="$(arg restitution)"/>
+                            restitution="$(arg restitution)"
+                            lateral_friction="$(arg lateral_friction)"
+                            rolling_friction="$(arg rolling_friction)"
+                            spinning_friction="$(arg spinning_friction)"/>
 </robot>

File: air_hockey_description/urdf/puck/model.urdf.xacro (robot description, xacro)
@@ -13,11 +13,12 @@
     <xacro:arg name="color" default="Red"/>
     <xacro:arg name="collide_bitmask" default="0x03"/>
-    <xacro:arg name="restitution" default="0.8"/>
-    <xacro:arg name="lateral_friction" default="0.02"/>
-    <xacro:arg name="rolling_friction" default="0.8"/>
-    <xacro:arg name="spinning_friction" default="0.04"/>
+    <xacro:arg name="restitution" default="1.0"/>
+    <xacro:arg name="lateral_friction" default="1.0"/>
+    <xacro:arg name="viscous_friction" default="1.0"/>
+    <xacro:arg name="spinning_friction" default="1.0"/>
     <xacro:property name="puck_radius" value="0.03165"/>
     <xacro:property name="puck_height" value="0.0049"/>
-    <xacro:macro name="puck" params="puck_name color collide_bitmask restitution lateral_friction rolling_friction spinning_friction">
+    <xacro:macro name="puck" params="puck_name color collide_bitmask restitution
+                                     lateral_friction viscous_friction spinning_friction">
         <link name="${puck_name}"/>
         <joint name="{puck_name}_joint" type="fixed">
@@ -57,5 +58,5 @@
                     <bounce>
                         <restitution_coefficient>${restitution}</restitution_coefficient>
-                        <threshold>0.01</threshold>
+                        <threshold>0.0</threshold>
                     </bounce>
                     <friction>
@@ -70,4 +71,6 @@
                             <mu>${lateral_friction}</mu>
                             <mu2>${lateral_friction}</mu2>
+                            <slip1>${viscous_friction}</slip1>
+                            <slip2>${viscous_friction}</slip2>
                         </ode>
                     </friction>
@@ -84,5 +87,5 @@
         </gazebo>
         <gazebo>
-            <updateRate>100.0</updateRate>
+            <updateRate>500.0</updateRate>
             <plugin name="puck_tf_plugin" filename="libpuck_tf_plugin.so">
             </plugin>
@@ -94,5 +97,5 @@
                 restitution="$(arg restitution)"
                 lateral_friction="$(arg lateral_friction)"
-                rolling_friction="$(arg rolling_friction)"
+                viscous_friction="$(arg viscous_friction)"
                 spinning_friction="$(arg spinning_friction)"/>
 </robot>

Commit message: Change the urdf

File: air_hockey_description/urdf/air_hockey_table/model.urdf.xacro (robot description, xacro)
@@ -10,10 +10,9 @@
         <color rgba="1.0 0.0 0.0 1"/>
     </material>
-    <xacro:arg name="parent" default="world"/>
+    <xacro:arg name="parent" default="Table"/>
     <xacro:arg name="collide_bitmask" default="0x01"/>
-    <xacro:arg name="restitution" default="0.68"/>
-    <xacro:arg name="lateral_friction" default="1.0"/>
-    <xacro:arg name="rolling_friction" default="1.0"/>
-    <xacro:arg name="spinning_friction" default="1.0"/>
+    <xacro:arg name="restitution" default="1.0"/>
+    <xacro:arg name="lateral_friction_rim" default="1.0"/>
+    <xacro:arg name="lateral_friction_surface" default="1.0"/>
     <xacro:property name="M_PI" value="3.1415926535897931"/>
     <xacro:property name="table_base_length" value="2.136"/>
@@ -28,5 +27,5 @@
     <xacro:property name="table_rim_vertical_height" value="0.03"/>
     <xacro:macro name="air_hockey_table" params="parent collide_bitmask restitution
-                                                 lateral_friction rolling_friction spinning_friction">
+                                                 lateral_friction_rim lateral_friction_surface">
         <link name="${parent}"/>
         <joint name="base_joint" type="fixed">
@@ -56,5 +55,5 @@
             <contact>
                 <restitution value="${restitution}"/>
-                <lateral_friction value="1.0"/>
+                <lateral_friction value="${lateral_friction_surface}"/>
                 <rolling_friction value="0.0"/>
                 <spinning_friction value="0.0"/>
@@ -100,5 +99,5 @@
             <contact>
                 <restitution value="${restitution}"/>
-                <lateral_friction value="0.0"/>
+                <lateral_friction value="${lateral_friction_rim}"/>
                 <rolling_friction value="0.0"/>
                 <spinning_friction value="0.0"/>
@@ -132,5 +131,5 @@
             <contact>
                 <restitution value="${restitution}"/>
-                <lateral_friction value="0.0"/>
+                <lateral_friction value="${lateral_friction_rim}"/>
                 <rolling_friction value="0.0"/>
                 <spinning_friction value="0.0"/>
@@ -163,5 +162,5 @@
             <contact>
                 <restitution value="${restitution}"/>
-                <lateral_friction value="0.0"/>
+                <lateral_friction value="${lateral_friction_rim}"/>
                 <rolling_friction value="0.0"/>
                 <spinning_friction value="0.0"/>
@@ -195,5 +194,5 @@
             <contact>
                 <restitution value="${restitution}"/>
-                <lateral_friction value="0.0"/>
+                <lateral_friction value="${lateral_friction_rim}"/>
                 <rolling_friction value="0.0"/>
                 <spinning_friction value="0.0"/>
@@ -227,5 +226,5 @@
             <contact>
                 <restitution value="${restitution}"/>
-                <lateral_friction value="0.0"/>
+                <lateral_friction value="${lateral_friction_rim}"/>
                 <rolling_friction value="0.0"/>
                 <spinning_friction value="0.0"/>
@@ -253,5 +252,5 @@
             <contact>
                 <restitution value="${restitution}"/>
-                <lateral_friction value="0.0"/>
+                <lateral_friction value="${lateral_friction_rim}"/>
                 <rolling_friction value="0.0"/>
                 <spinning_friction value="0.0"/>
@@ -285,5 +284,5 @@
             <contact>
                 <restitution value="${restitution}"/>
-                <lateral_friction value="0.0"/>
+                <lateral_friction value="${lateral_friction_rim}"/>
                 <rolling_friction value="0.0"/>
                 <spinning_friction value="0.0"/>
@@ -317,5 +316,5 @@
             <contact>
                 <restitution value="${restitution}"/>
-                <lateral_friction value="0.0"/>
+                <lateral_friction value="${lateral_friction_rim}"/>
                 <rolling_friction value="0.0"/>
                 <spinning_friction value="0.0"/>
@@ -333,6 +332,6 @@
                         <!-- https://github.com/osrf/gazebo/blob/gazebo11/gazebo/physics/bullet/BulletSurfaceParams.cc -->
                         <ode>
-                            <mu>${lateral_friction}</mu>
-                            <mu2>${lateral_friction}</mu2>
+                            <mu>${lateral_friction_surface}</mu>
+                            <mu2>${lateral_friction_surface}</mu2>
                         </ode>
                     </friction>
@@ -361,6 +360,6 @@
                         <!-- https://github.com/osrf/gazebo/blob/gazebo11/gazebo/physics/bullet/BulletSurfaceParams.cc -->
                         <ode>
-                            <mu>${lateral_friction}</mu>
-                            <mu2>${lateral_friction}</mu2>
+                            <mu>${lateral_friction_rim}</mu>
+                            <mu2>${lateral_friction_rim}</mu2>
                         </ode>
                     </friction>
@@ -389,6 +388,6 @@
                         <!-- https://github.com/osrf/gazebo/blob/gazebo11/gazebo/physics/bullet/BulletSurfaceParams.cc -->
                         <ode>
-                            <mu>${lateral_friction}</mu>
-                            <mu2>${lateral_friction}</mu2>
+                            <mu>${lateral_friction_rim}</mu>
+                            <mu2>${lateral_friction_rim}</mu2>
                         </ode>
                     </friction>
@@ -417,6 +416,6 @@
 <!--                        &lt;!&ndash; https://github.com/osrf/gazebo/blob/gazebo11/gazebo/physics/bullet/BulletSurfaceParams.cc &ndash;&gt;-->
 <!--                        <ode>-->
-<!--                            <mu>${lateral_friction}</mu>-->
-<!--                            <mu2>${lateral_friction}</mu2>-->
+<!--                            <mu>${lateral_friction_rim}</mu>-->
+<!--                            <mu2>${lateral_friction_rim}</mu2>-->
 <!--                        </ode>-->
 <!--                    </friction>-->
@@ -444,6 +443,6 @@
                         <!-- https://github.com/osrf/gazebo/blob/gazebo11/gazebo/physics/bullet/BulletSurfaceParams.cc -->
                         <ode>
-                            <mu>${lateral_friction}</mu>
-                            <mu2>${lateral_friction}</mu2>
+                            <mu>${lateral_friction_rim}</mu>
+                            <mu2>${lateral_friction_rim}</mu2>
                         </ode>
                     </friction>
@@ -472,6 +471,6 @@
                         <!-- https://github.com/osrf/gazebo/blob/gazebo11/gazebo/physics/bullet/BulletSurfaceParams.cc -->
                         <ode>
-                            <mu>${lateral_friction}</mu>
-                            <mu2>${lateral_friction}</mu2>
+                            <mu>${lateral_friction_rim}</mu>
+                            <mu2>${lateral_friction_rim}</mu2>
                         </ode>
                     </friction>
@@ -500,6 +499,6 @@
 <!--                        &lt;!&ndash; https://github.com/osrf/gazebo/blob/gazebo11/gazebo/physics/bullet/BulletSurfaceParams.cc &ndash;&gt;-->
 <!--                        <ode>-->
-<!--                            <mu>${lateral_friction}</mu>-->
-<!--                            <mu2>${lateral_friction}</mu2>-->
+<!--                            <mu>${lateral_friction_rim}</mu>-->
+<!--                            <mu2>${lateral_friction_rim}</mu2>-->
 <!--                        </ode>-->
 <!--                    </friction>-->
@@ -527,6 +526,6 @@
                         <!-- https://github.com/osrf/gazebo/blob/gazebo11/gazebo/physics/bullet/BulletSurfaceParams.cc -->
                         <ode>
-                            <mu>${lateral_friction}</mu>
-                            <mu2>${lateral_friction}</mu2>
+                            <mu>${lateral_friction_rim}</mu>
+                            <mu2>${lateral_friction_rim}</mu2>
                         </ode>
                     </friction>
@@ -555,6 +554,6 @@
                         <!-- https://github.com/osrf/gazebo/blob/gazebo11/gazebo/physics/bullet/BulletSurfaceParams.cc -->
                         <ode>
-                            <mu>${lateral_friction}</mu>
-                            <mu2>${lateral_friction}</mu2>
+                            <mu>${lateral_friction_rim}</mu>
+                            <mu2>${lateral_friction_rim}</mu2>
                         </ode>
                     </friction>
@@ -576,6 +575,5 @@
                             collide_bitmask="$(arg collide_bitmask)"
                             restitution="$(arg restitution)"
-                            lateral_friction="$(arg lateral_friction)"
-                            rolling_friction="$(arg rolling_friction)"
-                            spinning_friction="$(arg spinning_friction)"/>
+                            lateral_friction_rim="$(arg lateral_friction_rim)"
+                            lateral_friction_surface="$(arg lateral_friction_surface)"/>
 </robot>

File: air_hockey_description/urdf/puck/model.urdf.xacro (robot description, xacro)
@@ -15,10 +15,9 @@
     <xacro:arg name="restitution" default="1.0"/>
     <xacro:arg name="lateral_friction" default="1.0"/>
-    <xacro:arg name="viscous_friction" default="1.0"/>
     <xacro:arg name="spinning_friction" default="1.0"/>
     <xacro:property name="puck_radius" value="0.03165"/>
     <xacro:property name="puck_height" value="0.0049"/>
     <xacro:macro name="puck" params="puck_name color collide_bitmask restitution
-                                     lateral_friction viscous_friction spinning_friction">
+                                     lateral_friction spinning_friction">
         <link name="${puck_name}"/>
         <joint name="{puck_name}_joint" type="fixed">
@@ -31,5 +30,5 @@
                 <origin xyz="0 0 0.0" rpy="0 0 0"/>
                 <mass value="0.01"/>
-                <inertia ixx="1" ixy="0" ixz="0" iyy="1" iyz="0" izz="2e-5"/>
+                <inertia ixx="0.01" ixy="0" ixz="0" iyy="0.01" iyz="0" izz="5e-6"/>
             </inertial>
             <visual>
@@ -65,12 +64,10 @@
                         <torsional>
                             <coefficient>${spinning_friction}</coefficient>
-                            <use_patch_radius>false</use_patch_radius>
-                            <surface_radius>${puck_radius}</surface_radius>
+                            <use_patch_radius>true</use_patch_radius>
+                            <patch_radius>${puck_radius}</patch_radius>
                         </torsional>
                         <ode>
                             <mu>${lateral_friction}</mu>
                             <mu2>${lateral_friction}</mu2>
-                            <slip1>${viscous_friction}</slip1>
-                            <slip2>${viscous_friction}</slip2>
                         </ode>
                     </friction>
@@ -79,5 +76,5 @@
                         <ode>
                             <kp>1e9</kp>
-                            <max_vel>10</max_vel>
+                            <max_vel>20</max_vel>
                         </ode>
                     </contact>
@@ -97,5 +94,4 @@
                 restitution="$(arg restitution)"
                 lateral_friction="$(arg lateral_friction)"
-                viscous_friction="$(arg viscous_friction)"
                 spinning_friction="$(arg spinning_friction)"/>
 </robot>
