Commit message: separete restitution on longitude and latitude coefficient
- Add check for init tactics

File: air_hockey_description/urdf/air_hockey_table/model.urdf.xacro (robot description, xacro)
@@ -12,5 +12,6 @@
     <xacro:arg name="parent" default="Table"/>
     <xacro:arg name="collide_bitmask" default="0x01"/>
-    <xacro:arg name="restitution" default="1.0"/>
+    <xacro:arg name="restitution_longitude" default="1.0"/>
+    <xacro:arg name="restitution_latitude" default="1.0"/>
     <xacro:arg name="lateral_friction_rim" default="1.0"/>
     <xacro:arg name="lateral_friction_surface" default="1.0"/>
@@ -26,5 +27,5 @@
     <xacro:property name="table_rim_vertical_width" value="0.09"/>
     <xacro:property name="table_rim_vertical_height" value="0.03"/>
-    <xacro:macro name="air_hockey_table" params="parent collide_bitmask restitution
+    <xacro:macro name="air_hockey_table" params="parent collide_bitmask restitution_longitude restitution_latitude
                                                  lateral_friction_rim lateral_friction_surface">
         <link name="${parent}"/>
@@ -54,5 +55,5 @@
             </collision>
             <contact>
-                <restitution value="${restitution}"/>
+                <restitution value="${restitution_longitude}"/>
                 <lateral_friction value="${lateral_friction_surface}"/>
                 <rolling_friction value="0.0"/>
@@ -98,5 +99,5 @@
             </collision>
             <contact>
-                <restitution value="${restitution}"/>
+                <restitution value="${restitution_latitude}"/>
                 <lateral_friction value="${lateral_friction_rim}"/>
                 <rolling_friction value="0.0"/>
@@ -130,5 +131,5 @@
             </collision>
             <contact>
-                <restitution value="${restitution}"/>
+                <restitution value="${restitution_latitude}"/>
                 <lateral_friction value="${lateral_friction_rim}"/>
                 <rolling_friction value="0.0"/>
@@ -161,5 +162,5 @@
 <!--            </collision>-->
             <contact>
-                <restitution value="${restitution}"/>
+                <restitution value="${restitution_latitude}"/>
                 <lateral_friction value="${lateral_friction_rim}"/>
                 <rolling_friction value="0.0"/>
@@ -193,5 +194,5 @@
             </collision>
             <contact>
-                <restitution value="${restitution}"/>
+                <restitution value="${restitution_latitude}"/>
                 <lateral_friction value="${lateral_friction_rim}"/>
                 <rolling_friction value="0.0"/>
@@ -225,5 +226,5 @@
             </collision>
             <contact>
-                <restitution value="${restitution}"/>
+                <restitution value="${restitution_latitude}"/>
                 <lateral_friction value="${lateral_friction_rim}"/>
                 <rolling_friction value="0.0"/>
@@ -251,5 +252,5 @@
             </visual>
             <contact>
-                <restitution value="${restitution}"/>
+                <restitution value="${restitution_latitude}"/>
                 <lateral_friction value="${lateral_friction_rim}"/>
                 <rolling_friction value="0.0"/>
@@ -283,5 +284,5 @@
             </collision>
             <contact>
-                <restitution value="${restitution}"/>
+                <restitution value="${restitution_longitude}"/>
                 <lateral_friction value="${lateral_friction_rim}"/>
                 <rolling_friction value="0.0"/>
@@ -315,5 +316,5 @@
             </collision>
             <contact>
-                <restitution value="${restitution}"/>
+                <restitution value="${restitution_longitude}"/>
                 <lateral_friction value="${lateral_friction_rim}"/>
                 <rolling_friction value="0.0"/>
@@ -325,5 +326,5 @@
                 <surface>
                     <bounce>
-                        <restitution_coefficient>${restitution}</restitution_coefficient>
+                        <restitution_coefficient>${restitution_longitude}</restitution_coefficient>
                         <threshold>0</threshold>
                     </bounce>
@@ -353,5 +354,5 @@
                 <surface>
                     <bounce>
-                        <restitution_coefficient>${restitution}</restitution_coefficient>
+                        <restitution_coefficient>${restitution_latitude}</restitution_coefficient>
                         <threshold>0</threshold>
                     </bounce>
@@ -381,5 +382,5 @@
                 <surface>
                     <bounce>
-                        <restitution_coefficient>${restitution}</restitution_coefficient>
+                        <restitution_coefficient>${restitution_latitude}</restitution_coefficient>
                         <threshold>0</threshold>
                     </bounce>
@@ -409,5 +410,5 @@
 <!--                <surface>-->
 <!--                    <bounce>-->
-<!--                        <restitution_coefficient>${restitution}</restitution_coefficient>-->
+<!--                        <restitution_coefficient>${restitution_latitude}</restitution_coefficient>-->
 <!--                        <threshold>0</threshold>-->
 <!--                    </bounce>-->
@@ -436,5 +437,5 @@
                 <surface>
                     <bounce>
-                        <restitution_coefficient>${restitution}</restitution_coefficient>
+                        <restitution_coefficient>${restitution_latitude}</restitution_coefficient>
                         <threshold>0</threshold>
                     </bounce>
@@ -464,5 +465,5 @@
                 <surface>
                     <bounce>
-                        <restitution_coefficient>${restitution}</restitution_coefficient>
+                        <restitution_coefficient>${restitution_latitude}</restitution_coefficient>
                         <threshold>0</threshold>
                     </bounce>
@@ -492,5 +493,5 @@
 <!--                <surface>-->
 <!--                    <bounce>-->
-<!--                        <restitution_coefficient>${restitution}</restitution_coefficient>-->
+<!--                        <restitution_coefficient>${restitution_latitude}</restitution_coefficient>-->
 <!--                        <threshold>0</threshold>-->
 <!--                    </bounce>-->
@@ -519,5 +520,5 @@
                 <surface>
                     <bounce>
-                        <restitution_coefficient>${restitution}</restitution_coefficient>
+                        <restitution_coefficient>${restitution_longitude}</restitution_coefficient>
                         <threshold>0</threshold>
                     </bounce>
@@ -547,5 +548,5 @@
                 <surface>
                     <bounce>
-                        <restitution_coefficient>${restitution}</restitution_coefficient>
+                        <restitution_coefficient>${restitution_longitude}</restitution_coefficient>
                         <threshold>0</threshold>
                     </bounce>
@@ -574,5 +575,6 @@
     <xacro:air_hockey_table parent="$(arg parent)"
                             collide_bitmask="$(arg collide_bitmask)"
-                            restitution="$(arg restitution)"
+                            restitution_longitude="$(arg restitution_longitude)"
+                            restitution_latitude="$(arg restitution_latitude)"
                             lateral_friction_rim="$(arg lateral_friction_rim)"
                             lateral_friction_surface="$(arg lateral_friction_surface)"/>

File: air_hockey_description/urdf/puck/model.urdf.xacro (robot description, xacro)
@@ -1,4 +1,4 @@
 <?xml version="1.0" encoding="utf-8"?>
-<robot name="puck" xmlns:xacro="http://www.ros.org/wiki/xacro" >
+<robot name="puck" xmlns:xacro="http://www.ros.org/wiki/xacro">
     <material name="Red">
         <color rgba="1.0 0.0 0.0 1"/>
@@ -16,8 +16,10 @@
     <xacro:arg name="lateral_friction" default="1.0"/>
     <xacro:arg name="spinning_friction" default="1.0"/>
+    <xacro:arg name="linear_vel_decay" default="0.0001"/>
+    <xacro:arg name="angular_vel_decay" default="0.0001"/>
     <xacro:property name="puck_radius" value="0.03165"/>
     <xacro:property name="puck_height" value="0.0049"/>
     <xacro:macro name="puck" params="puck_name color collide_bitmask restitution
-                                     lateral_friction spinning_friction">
+                                     lateral_friction spinning_friction linear_vel_decay angular_vel_decay">
         <link name="${puck_name}"/>
         <joint name="{puck_name}_joint" type="fixed">
@@ -53,4 +55,8 @@
         </link>
         <gazebo reference="${puck_name}">
+            <velocity_decay>
+                <linear>${linear_vel_decay}</linear>
+                <angular>${angular_vel_decay}</angular>
+            </velocity_decay>
             <collision>
                 <surface>
@@ -94,4 +100,6 @@
                 restitution="$(arg restitution)"
                 lateral_friction="$(arg lateral_friction)"
-                spinning_friction="$(arg spinning_friction)"/>
+                spinning_friction="$(arg spinning_friction)"
+                linear_vel_decay="$(arg linear_vel_decay)"
+                angular_vel_decay="$(arg angular_vel_decay)"/>
 </robot>

Commit message: Update the debuging code

File: air_hockey_description/urdf/air_hockey_table/model.urdf.xacro (robot description, xacro)
@@ -17,6 +17,6 @@
     <xacro:arg name="lateral_friction_surface" default="0.0001"/>
     <xacro:property name="M_PI" value="3.1415926535897931"/>
-    <xacro:property name="table_base_length" value="2.136"/>
-    <xacro:property name="table_base_width" value="1.222"/>
+    <xacro:property name="table_base_length" value="2.128"/>
+    <xacro:property name="table_base_width" value="1.218"/>
     <xacro:property name="table_base_height" value="0.11"/>
     <xacro:property name="table_rim_horizon_length" value="0.09"/>
@@ -24,5 +24,5 @@
     <xacro:property name="table_rim_horizon_height" value="0.01"/>
     <xacro:property name="table_rim_horizon_top_height" value="0.02"/>
-    <xacro:property name="table_rim_vertical_length" value="2.136"/>
+    <xacro:property name="table_rim_vertical_length" value="2.128"/>
     <xacro:property name="table_rim_vertical_width" value="0.09"/>
     <xacro:property name="table_rim_vertical_height" value="0.03"/>
