Commit message: Update model parameters

File: air_hockey_description/urdf/air_hockey_table/model.urdf (robot description, URDF)
Before this commit: robot air_hockey_table, 12 links, 11 joints
Links:
- link t_base: geometry collision box size=2.128 1.218 0.11; visual box size=2.128 1.218 0.11
- link t_down_rim_top: geometry visual box size=0.09 1.038 0.02
- link t_left_rim: geometry collision box size=2.128 0.09 0.13; visual box size=2.128 0.09 0.03
- link t_right_rim: geometry collision box size=2.128 0.09 0.13; visual box size=2.128 0.09 0.03
- link t_up_rim_top: geometry visual box size=0.09 1.038 0.02
Joints:
- joint base_away_joint: origin xyz=0.9780000000000001 0 0 rpy=0 0 3.141592653589793 -> xyz=0.9740000000000001 0 0 rpy=0 0 3.141592653589793
- joint base_down_rim_l: origin xyz=1.0230000000000001                                            0.323                                            0.06 rpy=0.0 0.0 0.0 -> xyz=1.0190000000000001                                            0.321                                            0.06 rpy=0.0 0.0 0.0
- joint base_down_rim_r: origin xyz=1.0230000000000001                                            -0.323                                            0.06 rpy=0.0 0.0 0.0 -> xyz=1.0190000000000001                                            -0.321                                            0.06 rpy=0.0 0.0 0.0
- joint base_down_rim_top: origin xyz=1.0230000000000001                                            0.0                                            0.075 rpy=0.0 0.0 0.0 -> xyz=1.0190000000000001                                            0.0                                            0.075 rpy=0.0 0.0 0.0
- joint base_home_joint: origin xyz=-0.9780000000000001 0 0 rpy=0 0 0 -> xyz=-0.9740000000000001 0 0 rpy=0 0 0
- joint base_left_rim: origin xyz=0.0                                            0.566                                            0.07 rpy=0.0 0.0 0.0 -> xyz=0.0                                            0.564                                            0.07 rpy=0.0 0.0 0.0
- joint base_right_rim: origin xyz=0.0                                            -0.566                                            0.07 rpy=0.0 0.0 0.0 -> xyz=0.0                                            -0.564                                            0.07 rpy=0.0 0.0 0.0
- joint base_up_rim_l: origin xyz=-1.0230000000000001                                            0.323                                            0.06 rpy=0.0 0.0 0.0 -> xyz=-1.0190000000000001                                            0.321                                            0.06 rpy=0.0 0.0 0.0
- joint base_up_rim_r: origin xyz=-1.0230000000000001                                            -0.323                                            0.06 rpy=0.0 0.0 0.0 -> xyz=-1.0190000000000001                                            -0.321                                            0.06 rpy=0.0 0.0 0.0
- joint base_up_rim_top: origin xyz=-1.0230000000000001                                            0.0                                            0.075 rpy=0.0 0.0 0.0 -> xyz=-1.0190000000000001                                            0.0                                            0.075 rpy=0.0 0.0 0.0
